File: 4-MPPC_FARICH_Prototype/4-MPPC_FARICH_Prototype.kicad_pcb (KiCad board)
At the start: 2 copper layers, 4 parts

Commit message: .
Parts:
- added J1: 1778764, HV_Connector:PHOENIX_1778764, B.Cu at (214.8, 85.0)
- added J10: ST4-40-1.00-L-D-P-TR, FARICH:SAMTEC_ST4-40-1.00-L-D-P-TR, B.Cu at (166.3, 79.1)
- added J11: ST4-40-1.00-L-D-P-TR, FARICH:SAMTEC_ST4-40-1.00-L-D-P-TR, B.Cu at (179.1, 79.1)
- added J12: ST4-40-1.00-L-D-P-TR, FARICH:SAMTEC_ST4-40-1.00-L-D-P-TR, B.Cu at (166.3, 106.0)
- added J13: ST4-40-1.00-L-D-P-TR, FARICH:SAMTEC_ST4-40-1.00-L-D-P-TR, B.Cu at (179.1, 106.0)
- added J2: ST4-40-1.00-L-D-P-TR, FARICH:SAMTEC_ST4-40-1.00-L-D-P-TR, B.Cu at (112.7, 79.1)
- added J3: ST4-40-1.00-L-D-P-TR, FARICH:SAMTEC_ST4-40-1.00-L-D-P-TR, B.Cu at (125.5, 79.1)
- added J4: ST4-40-1.00-L-D-P-TR, FARICH:SAMTEC_ST4-40-1.00-L-D-P-TR, B.Cu at (112.7, 106.0)
- added J5: ST4-40-1.00-L-D-P-TR, FARICH:SAMTEC_ST4-40-1.00-L-D-P-TR, B.Cu at (125.5, 106.0)
- added J6: ST4-40-1.00-L-D-P-TR, FARICH:SAMTEC_ST4-40-1.00-L-D-P-TR, B.Cu at (139.5, 79.1)
- added J7: ST4-40-1.00-L-D-P-TR, FARICH:SAMTEC_ST4-40-1.00-L-D-P-TR, B.Cu at (152.3, 79.1)
- added J8: ST4-40-1.00-L-D-P-TR, FARICH:SAMTEC_ST4-40-1.00-L-D-P-TR, B.Cu at (139.5, 106.0)
- added J9: ST4-40-1.00-L-D-P-TR, FARICH:SAMTEC_ST4-40-1.00-L-D-P-TR, B.Cu at (152.3, 106.0)
- moved MPPC4 1.10 mm to (194.8, 92.2)
- moved MPPC3 0.65 mm to (162.2, 92.2)
- moved MPPC2 0.26 mm to (129.6, 92.2)
Routing:
- added copper zone on B.Cu, net GND
- added copper zone on F.Cu, net GND
- added copper zone on In1.Cu, net GND
- added copper zone on In2.Cu, net GND
- added copper zone on In3.Cu, net GND
- added copper zone on In4.Cu, net GND
- added copper zone on In5.Cu, net GND
- added copper zone on In6.Cu, net GND
Other:
- board outline added: 164.2 x 53.4 mm
- copper layers 2 -> 8
- board text added: "NOTEs: FARICH: d=12.8 (distance between two connectors in one cube) D=26.84 (distance between two cubes)"

Commit message: .
Parts:
- added H1: MountingHole, MountingHole:MountingHole_3.2mm_M3_DIN965_Pad, F.Cu at (73.2, 72.4)
- added H2: MountingHole, MountingHole:MountingHole_3.2mm_M3_DIN965_Pad, F.Cu at (73.2, 112.7)
- added H3: MountingHole, MountingHole:MountingHole_3.2mm_M3_DIN965_Pad, F.Cu at (224.7, 72.4)
- added H4: MountingHole, MountingHole:MountingHole_3.2mm_M3_DIN965_Pad, F.Cu at (224.7, 112.9)
Connections:
- J1 pad SH1: GND -> (no net)
- J1 pad SH2: GND -> (no net)
Other:
- board size 164.2 x 53.4 mm -> 164.1 x 52.9 mm

Commit message: .
Other:
- board text added: "NOTEs: FARICH: d=12.8 (distance between two connectors in one cube) D=26.84 (distance between two cubes) MPPCs: MPPC1 & MPPC2 2 pads combined MPPC3 & MPPC4 individual pads"
- board text removed: "NOTEs: FARICH: d=12.8 (distance between two connectors in one cube) D=26.84 (distance between two cubes)"
Changed lines of the file:
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@@
 	(footprint "HV_Connector:PHOENIX_1778764"
 		(layer "B.Cu")
-		(at 214.78 84.9575)
+		(at 214.78 85.007107)
 		(property "Reference" "J1"
 			(at 3.175 11.385 0)
@@
 		(layer "Edge.Cuts")
 	)
-	(gr_text "NOTEs:\n	FARICH: \n			d=12.8 (distance between two connectors in one cube)\n			D=26.84 (distance between two cubes)"
-		(at 17.21 28.61 0)
+	(gr_text "NOTEs:\n	FARICH: \n			d=12.8 (distance between two connectors in one cube)\n			D=26.84 (distance between two cubes)\n	MPPCs:\n			MPPC1 & MPPC2 2 pads combined\n			MPPC3 & MPPC4 individual pads"
+		(at 14.707107 36.207107 0)
 		(layer "F.Fab")
 		(effects
@@
 		(polygon
 			(pts
-				(xy 57.2 44.13) (xy 241.3 44.13) (xy 241.3 141.93) (xy 57.2 141.93)
+				(xy 57.2 62.13) (xy 241.3 62.13) (xy 241.3 125.43) (xy 57.2 125.43)
 			)
 		)
