File: 4-MPPC_FARICH_Prototype/4-MPPC_FARICH_Prototype.kicad_pcb (KiCad board)
At the start: 8 copper layers, 164.1 x 52.9 mm, 21 parts, among them J1 1778764, J10 ST4-40-1.00-L-D-P-TR, J11 ST4-40-1.00-L-D-P-TR, J12 ST4-40-1.00-L-D-P-TR, J13 ST4-40-1.00-L-D-P-TR, J2 ST4-40-1.00-L-D-P-TR, J3 ST4-40-1.00-L-D-P-TR, J4 ST4-40-1.00-L-D-P-TR, J5 ST4-40-1.00-L-D-P-TR, J6 ST4-40-1.00-L-D-P-TR, J7 ST4-40-1.00-L-D-P-TR, J8 ST4-40-1.00-L-D-P-TR, J9 ST4-40-1.00-L-D-P-TR

Commit message: .
Connections:
- H1 pad 1: GND -> (no net)
- H2 pad 1: GND -> (no net)
- H3 pad 1: GND -> (no net)
- H4 pad 1: GND -> (no net)
- J10 pad 01: unconnected-(J10-Pad01) -> Onboard_HV
- J10 pad 02: unconnected-(J10-Pad02) -> Onboard_HV
- J10 pad 03: unconnected-(J10-Pad03) -> Onboard_HV
- J10 pad 04: unconnected-(J10-Pad04) -> Onboard_HV
- J10 pad 05: unconnected-(J10-Pad05) -> GND
- J10 pad 06: unconnected-(J10-Pad06) -> GND
- J10 pad 15: unconnected-(J10-Pad15) -> GND
- J10 pad 16: unconnected-(J10-Pad16) -> GND
- J10 pad 17: unconnected-(J10-Pad17) -> Onboard_HV
- J10 pad 18: unconnected-(J10-Pad18) -> Onboard_HV
- J10 pad 19: unconnected-(J10-Pad19) -> Onboard_HV
- J10 pad 20: unconnected-(J10-Pad20) -> Onboard_HV
- J10 pad 21: unconnected-(J10-Pad21) -> Onboard_HV
- J10 pad 22: unconnected-(J10-Pad22) -> Onboard_HV
- J10 pad 23: unconnected-(J10-Pad23) -> Onboard_HV
- J10 pad 24: unconnected-(J10-Pad24) -> Onboard_HV
- J10 pad 25: unconnected-(J10-Pad25) -> GND
- J10 pad 26: unconnected-(J10-Pad26) -> GND
- J10 pad 35: unconnected-(J10-Pad35) -> GND
- J10 pad 36: unconnected-(J10-Pad36) -> GND
- J10 pad 37: unconnected-(J10-Pad37) -> Onboard_HV
- J10 pad 38: unconnected-(J10-Pad38) -> Onboard_HV
- J10 pad 39: unconnected-(J10-Pad39) -> Onboard_HV
- J10 pad 40: unconnected-(J10-Pad40) -> Onboard_HV
- J10 pad 41: unconnected-(J10-Pad41) -> Onboard_HV
- J10 pad 42: unconnected-(J10-Pad42) -> Onboard_HV
- J10 pad 43: unconnected-(J10-Pad43) -> Onboard_HV
- J10 pad 44: unconnected-(J10-Pad44) -> Onboard_HV
- J10 pad 45: unconnected-(J10-Pad45) -> GND
- J10 pad 46: unconnected-(J10-Pad46) -> GND
- J10 pad 55: unconnected-(J10-Pad55) -> GND
- J10 pad 56: unconnected-(J10-Pad56) -> GND
- J10 pad 57: unconnected-(J10-Pad57) -> Onboard_HV
- J10 pad 58: unconnected-(J10-Pad58) -> Onboard_HV
- J10 pad 59: unconnected-(J10-Pad59) -> Onboard_HV
- J10 pad 60: unconnected-(J10-Pad60) -> Onboard_HV
- J10 pad 61: unconnected-(J10-Pad61) -> Onboard_HV
- J10 pad 62: unconnected-(J10-Pad62) -> Onboard_HV
- J10 pad 63: unconnected-(J10-Pad63) -> Onboard_HV
- J10 pad 64: unconnected-(J10-Pad64) -> Onboard_HV
- J10 pad 65: unconnected-(J10-Pad65) -> GND
- J10 pad 66: unconnected-(J10-Pad66) -> GND
- J10 pad 75: unconnected-(J10-Pad75) -> GND
- J10 pad 76: unconnected-(J10-Pad76) -> GND
- J10 pad 77: unconnected-(J10-Pad77) -> Onboard_HV
- J10 pad 78: unconnected-(J10-Pad78) -> Onboard_HV
- J10 pad 79: unconnected-(J10-Pad79) -> Onboard_HV
- J10 pad 80: unconnected-(J10-Pad80) -> Onboard_HV
- J11 pad 01: unconnected-(J11-Pad01) -> Onboard_HV
- J11 pad 02: unconnected-(J11-Pad02) -> Onboard_HV
- J11 pad 03: unconnected-(J11-Pad03) -> Onboard_HV
- J11 pad 04: unconnected-(J11-Pad04) -> Onboard_HV
- J11 pad 05: unconnected-(J11-Pad05) -> GND
- J11 pad 06: unconnected-(J11-Pad06) -> GND
- J11 pad 15: unconnected-(J11-Pad15) -> GND
- J11 pad 16: unconnected-(J11-Pad16) -> GND
- J11 pad 17: unconnected-(J11-Pad17) -> Onboard_HV
- J11 pad 18: unconnected-(J11-Pad18) -> Onboard_HV
- J11 pad 19: unconnected-(J11-Pad19) -> Onboard_HV
- J11 pad 20: unconnected-(J11-Pad20) -> Onboard_HV
- J11 pad 21: unconnected-(J11-Pad21) -> Onboard_HV
- J11 pad 22: unconnected-(J11-Pad22) -> Onboard_HV
- J11 pad 23: unconnected-(J11-Pad23) -> Onboard_HV
- J11 pad 24: unconnected-(J11-Pad24) -> Onboard_HV
- J11 pad 25: unconnected-(J11-Pad25) -> GND
- J11 pad 26: unconnected-(J11-Pad26) -> GND
- J11 pad 35: unconnected-(J11-Pad35) -> GND
- J11 pad 36: unconnected-(J11-Pad36) -> GND
- J11 pad 37: unconnected-(J11-Pad37) -> Onboard_HV
- J11 pad 38: unconnected-(J11-Pad38) -> Onboard_HV
- J11 pad 39: unconnected-(J11-Pad39) -> Onboard_HV
- J11 pad 40: unconnected-(J11-Pad40) -> Onboard_HV
- J11 pad 41: unconnected-(J11-Pad41) -> Onboard_HV
- J11 pad 42: unconnected-(J11-Pad42) -> Onboard_HV
- J11 pad 43: unconnected-(J11-Pad43) -> Onboard_HV
- J11 pad 44: unconnected-(J11-Pad44) -> Onboard_HV
- J11 pad 45: unconnected-(J11-Pad45) -> GND
- J11 pad 46: unconnected-(J11-Pad46) -> GND
- J11 pad 55: unconnected-(J11-Pad55) -> GND
- J11 pad 56: unconnected-(J11-Pad56) -> GND
- J11 pad 57: unconnected-(J11-Pad57) -> Onboard_HV
- J11 pad 58: unconnected-(J11-Pad58) -> Onboard_HV
- J11 pad 59: unconnected-(J11-Pad59) -> Onboard_HV
- J11 pad 60: unconnected-(J11-Pad60) -> Onboard_HV
- J11 pad 61: unconnected-(J11-Pad61) -> Onboard_HV
- J11 pad 62: unconnected-(J11-Pad62) -> Onboard_HV
- J11 pad 63: unconnected-(J11-Pad63) -> Onboard_HV
- J11 pad 64: unconnected-(J11-Pad64) -> Onboard_HV
- J11 pad 65: unconnected-(J11-Pad65) -> GND
- J11 pad 66: unconnected-(J11-Pad66) -> GND
- J11 pad 75: unconnected-(J11-Pad75) -> GND
- J11 pad 76: unconnected-(J11-Pad76) -> GND
- J11 pad 77: unconnected-(J11-Pad77) -> Onboard_HV
- J11 pad 78: unconnected-(J11-Pad78) -> Onboard_HV
- J11 pad 79: unconnected-(J11-Pad79) -> Onboard_HV
- J11 pad 80: unconnected-(J11-Pad80) -> Onboard_HV
- J12 pad 01: unconnected-(J12-Pad01) -> Onboard_HV
- J12 pad 02: unconnected-(J12-Pad02) -> Onboard_HV
- J12 pad 03: unconnected-(J12-Pad03) -> Onboard_HV
- J12 pad 04: unconnected-(J12-Pad04) -> Onboard_HV
- J12 pad 05: unconnected-(J12-Pad05) -> GND
- J12 pad 06: unconnected-(J12-Pad06) -> GND
- J12 pad 15: unconnected-(J12-Pad15) -> GND
- J12 pad 16: unconnected-(J12-Pad16) -> GND
- J12 pad 17: unconnected-(J12-Pad17) -> Onboard_HV
- J12 pad 18: unconnected-(J12-Pad18) -> Onboard_HV
- J12 pad 19: unconnected-(J12-Pad19) -> Onboard_HV
- J12 pad 20: unconnected-(J12-Pad20) -> Onboard_HV
- J12 pad 21: unconnected-(J12-Pad21) -> Onboard_HV
- J12 pad 22: unconnected-(J12-Pad22) -> Onboard_HV
- J12 pad 23: unconnected-(J12-Pad23) -> Onboard_HV
- J12 pad 24: unconnected-(J12-Pad24) -> Onboard_HV
- J12 pad 25: unconnected-(J12-Pad25) -> GND
- J12 pad 26: unconnected-(J12-Pad26) -> GND
- J12 pad 35: unconnected-(J12-Pad35) -> GND
- J12 pad 36: unconnected-(J12-Pad36) -> GND
- J12 pad 37: unconnected-(J12-Pad37) -> Onboard_HV
- J12 pad 38: unconnected-(J12-Pad38) -> Onboard_HV
- J12 pad 39: unconnected-(J12-Pad39) -> Onboard_HV
- J12 pad 40: unconnected-(J12-Pad40) -> Onboard_HV
- J12 pad 41: unconnected-(J12-Pad41) -> Onboard_HV
- J12 pad 42: unconnected-(J12-Pad42) -> Onboard_HV
- J12 pad 43: unconnected-(J12-Pad43) -> Onboard_HV
- J12 pad 44: unconnected-(J12-Pad44) -> Onboard_HV
- J12 pad 45: unconnected-(J12-Pad45) -> GND
- J12 pad 46: unconnected-(J12-Pad46) -> GND
- J12 pad 55: unconnected-(J12-Pad55) -> GND
- J12 pad 56: unconnected-(J12-Pad56) -> GND
- J12 pad 57: unconnected-(J12-Pad57) -> Onboard_HV
- J12 pad 58: unconnected-(J12-Pad58) -> Onboard_HV
- J12 pad 59: unconnected-(J12-Pad59) -> Onboard_HV
- J12 pad 60: unconnected-(J12-Pad60) -> Onboard_HV
- J12 pad 61: unconnected-(J12-Pad61) -> Onboard_HV
- J12 pad 62: unconnected-(J12-Pad62) -> Onboard_HV
- J12 pad 63: unconnected-(J12-Pad63) -> Onboard_HV
- J12 pad 64: unconnected-(J12-Pad64) -> Onboard_HV
- J12 pad 65: unconnected-(J12-Pad65) -> GND
- J12 pad 66: unconnected-(J12-Pad66) -> GND
- J12 pad 75: unconnected-(J12-Pad75) -> GND
- J12 pad 76: unconnected-(J12-Pad76) -> GND
- J12 pad 77: unconnected-(J12-Pad77) -> Onboard_HV
- J12 pad 78: unconnected-(J12-Pad78) -> Onboard_HV
- J12 pad 79: unconnected-(J12-Pad79) -> Onboard_HV
- J12 pad 80: unconnected-(J12-Pad80) -> Onboard_HV
- J13 pad 01: unconnected-(J13-Pad01) -> Onboard_HV
- J13 pad 02: unconnected-(J13-Pad02) -> Onboard_HV
- J13 pad 03: unconnected-(J13-Pad03) -> Onboard_HV
- J13 pad 04: unconnected-(J13-Pad04) -> Onboard_HV
- J13 pad 05: unconnected-(J13-Pad05) -> GND
- J13 pad 06: unconnected-(J13-Pad06) -> GND
- J13 pad 15: unconnected-(J13-Pad15) -> GND
- J13 pad 16: unconnected-(J13-Pad16) -> GND
- J13 pad 17: unconnected-(J13-Pad17) -> Onboard_HV
- J13 pad 18: unconnected-(J13-Pad18) -> Onboard_HV
- J13 pad 19: unconnected-(J13-Pad19) -> Onboard_HV
- J13 pad 20: unconnected-(J13-Pad20) -> Onboard_HV
- J13 pad 21: unconnected-(J13-Pad21) -> Onboard_HV
- J13 pad 22: unconnected-(J13-Pad22) -> Onboard_HV
- J13 pad 23: unconnected-(J13-Pad23) -> Onboard_HV
- J13 pad 24: unconnected-(J13-Pad24) -> Onboard_HV
- J13 pad 25: unconnected-(J13-Pad25) -> GND
- J13 pad 26: unconnected-(J13-Pad26) -> GND
- J13 pad 35: unconnected-(J13-Pad35) -> GND
- J13 pad 36: unconnected-(J13-Pad36) -> GND
- J13 pad 37: unconnected-(J13-Pad37) -> Onboard_HV
- J13 pad 38: unconnected-(J13-Pad38) -> Onboard_HV
- J13 pad 39: unconnected-(J13-Pad39) -> Onboard_HV
- J13 pad 40: unconnected-(J13-Pad40) -> Onboard_HV
- J13 pad 41: unconnected-(J13-Pad41) -> Onboard_HV
- J13 pad 42: unconnected-(J13-Pad42) -> Onboard_HV
- J13 pad 43: unconnected-(J13-Pad43) -> Onboard_HV
- J13 pad 44: unconnected-(J13-Pad44) -> Onboard_HV
- J13 pad 45: unconnected-(J13-Pad45) -> GND
- J13 pad 46: unconnected-(J13-Pad46) -> GND
- J13 pad 55: unconnected-(J13-Pad55) -> GND
- J13 pad 56: unconnected-(J13-Pad56) -> GND
- J13 pad 57: unconnected-(J13-Pad57) -> Onboard_HV
- J13 pad 58: unconnected-(J13-Pad58) -> Onboard_HV
- J13 pad 59: unconnected-(J13-Pad59) -> Onboard_HV
- J13 pad 60: unconnected-(J13-Pad60) -> Onboard_HV
- J13 pad 61: unconnected-(J13-Pad61) -> Onboard_HV
- J13 pad 62: unconnected-(J13-Pad62) -> Onboard_HV
- J13 pad 63: unconnected-(J13-Pad63) -> Onboard_HV
- J13 pad 64: unconnected-(J13-Pad64) -> Onboard_HV
- J13 pad 65: unconnected-(J13-Pad65) -> GND
- J13 pad 66: unconnected-(J13-Pad66) -> GND
- J13 pad 75: unconnected-(J13-Pad75) -> GND
- J13 pad 76: unconnected-(J13-Pad76) -> GND
- J13 pad 77: unconnected-(J13-Pad77) -> Onboard_HV
- J13 pad 78: unconnected-(J13-Pad78) -> Onboard_HV
- J13 pad 79: unconnected-(J13-Pad79) -> Onboard_HV
- J13 pad 80: unconnected-(J13-Pad80) -> Onboard_HV
- J2 pad 01: unconnected-(J2-Pad01) -> Onboard_HV
- J2 pad 02: unconnected-(J2-Pad02) -> Onboard_HV
- J2 pad 03: unconnected-(J2-Pad03) -> Onboard_HV
- J2 pad 04: unconnected-(J2-Pad04) -> Onboard_HV
- J2 pad 05: unconnected-(J2-Pad05) -> GND
- J2 pad 06: unconnected-(J2-Pad06) -> GND
- J2 pad 15: unconnected-(J2-Pad15) -> GND
- J2 pad 16: unconnected-(J2-Pad16) -> GND
- J2 pad 17: unconnected-(J2-Pad17) -> Onboard_HV
- J2 pad 18: unconnected-(J2-Pad18) -> Onboard_HV
- J2 pad 19: unconnected-(J2-Pad19) -> Onboard_HV
- J2 pad 20: unconnected-(J2-Pad20) -> Onboard_HV
- J2 pad 21: unconnected-(J2-Pad21) -> Onboard_HV
- J2 pad 22: unconnected-(J2-Pad22) -> Onboard_HV
- J2 pad 23: unconnected-(J2-Pad23) -> Onboard_HV
- J2 pad 24: unconnected-(J2-Pad24) -> Onboard_HV
- J2 pad 25: unconnected-(J2-Pad25) -> GND
- J2 pad 26: unconnected-(J2-Pad26) -> GND
- J2 pad 35: unconnected-(J2-Pad35) -> GND
- J2 pad 36: unconnected-(J2-Pad36) -> GND
- J2 pad 37: unconnected-(J2-Pad37) -> Onboard_HV
- J2 pad 38: unconnected-(J2-Pad38) -> Onboard_HV
- J2 pad 39: unconnected-(J2-Pad39) -> Onboard_HV
- J2 pad 40: unconnected-(J2-Pad40) -> Onboard_HV
- J2 pad 41: unconnected-(J2-Pad41) -> Onboard_HV
- J2 pad 42: unconnected-(J2-Pad42) -> Onboard_HV
- J2 pad 43: unconnected-(J2-Pad43) -> Onboard_HV
- J2 pad 44: unconnected-(J2-Pad44) -> Onboard_HV
- J2 pad 45: unconnected-(J2-Pad45) -> GND
- J2 pad 46: unconnected-(J2-Pad46) -> GND
- J2 pad 55: unconnected-(J2-Pad55) -> GND
- J2 pad 56: unconnected-(J2-Pad56) -> GND
- J2 pad 57: unconnected-(J2-Pad57) -> Onboard_HV
- J2 pad 58: unconnected-(J2-Pad58) -> Onboard_HV
- J2 pad 59: unconnected-(J2-Pad59) -> Onboard_HV
- J2 pad 60: unconnected-(J2-Pad60) -> Onboard_HV
- J2 pad 61: unconnected-(J2-Pad61) -> Onboard_HV
- J2 pad 62: unconnected-(J2-Pad62) -> Onboard_HV
- J2 pad 63: unconnected-(J2-Pad63) -> Onboard_HV
- J2 pad 64: unconnected-(J2-Pad64) -> Onboard_HV
- J2 pad 65: unconnected-(J2-Pad65) -> GND
- J2 pad 66: unconnected-(J2-Pad66) -> GND
- J2 pad 75: unconnected-(J2-Pad75) -> GND
- J2 pad 76: unconnected-(J2-Pad76) -> GND
- J2 pad 77: unconnected-(J2-Pad77) -> Onboard_HV
- J2 pad 78: unconnected-(J2-Pad78) -> Onboard_HV
- J2 pad 79: unconnected-(J2-Pad79) -> Onboard_HV
- J2 pad 80: unconnected-(J2-Pad80) -> Onboard_HV
- J3 pad 01: unconnected-(J3-Pad01) -> Onboard_HV
- J3 pad 02: unconnected-(J3-Pad02) -> Onboard_HV
- J3 pad 03: unconnected-(J3-Pad03) -> Onboard_HV
- J3 pad 04: unconnected-(J3-Pad04) -> Onboard_HV
- J3 pad 05: unconnected-(J3-Pad05) -> GND
- J3 pad 06: unconnected-(J3-Pad06) -> GND
- J3 pad 15: unconnected-(J3-Pad15) -> GND
- J3 pad 16: unconnected-(J3-Pad16) -> GND
- J3 pad 17: unconnected-(J3-Pad17) -> Onboard_HV
- J3 pad 18: unconnected-(J3-Pad18) -> Onboard_HV
- J3 pad 19: unconnected-(J3-Pad19) -> Onboard_HV
- J3 pad 20: unconnected-(J3-Pad20) -> Onboard_HV
- J3 pad 21: unconnected-(J3-Pad21) -> Onboard_HV
- J3 pad 22: unconnected-(J3-Pad22) -> Onboard_HV
- J3 pad 23: unconnected-(J3-Pad23) -> Onboard_HV
- J3 pad 24: unconnected-(J3-Pad24) -> Onboard_HV
- J3 pad 25: unconnected-(J3-Pad25) -> GND
- J3 pad 26: unconnected-(J3-Pad26) -> GND
- J3 pad 35: unconnected-(J3-Pad35) -> GND
- J3 pad 36: unconnected-(J3-Pad36) -> GND
- J3 pad 37: unconnected-(J3-Pad37) -> Onboard_HV
- J3 pad 38: unconnected-(J3-Pad38) -> Onboard_HV
- J3 pad 39: unconnected-(J3-Pad39) -> Onboard_HV
- J3 pad 40: unconnected-(J3-Pad40) -> Onboard_HV
- J3 pad 41: unconnected-(J3-Pad41) -> Onboard_HV
- J3 pad 42: unconnected-(J3-Pad42) -> Onboard_HV
- J3 pad 43: unconnected-(J3-Pad43) -> Onboard_HV
- J3 pad 44: unconnected-(J3-Pad44) -> Onboard_HV
- J3 pad 45: unconnected-(J3-Pad45) -> GND
- J3 pad 46: unconnected-(J3-Pad46) -> GND
- J3 pad 55: unconnected-(J3-Pad55) -> GND
- J3 pad 56: unconnected-(J3-Pad56) -> GND
- J3 pad 57: unconnected-(J3-Pad57) -> Onboard_HV
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Routing:
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
Commit message: .
Parts:
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Connections:
- J2 pad 07: unconnected-(J2-Pad07) -> Cube_1_A-G8
- J2 pad 08: unconnected-(J2-Pad08) -> Cube_1_A-F8
- J2 pad 09: unconnected-(J2-Pad09) -> Cube_1_A-H8
- J2 pad 10: unconnected-(J2-Pad10) -> Cube_1_A-E8
- J2 pad 11: unconnected-(J2-Pad11) -> Cube_1_A-H7
- J2 pad 12: unconnected-(J2-Pad12) -> Cube_1_A-E7
- J2 pad 13: unconnected-(J2-Pad13) -> Cube_1_A-G7
- J2 pad 14: unconnected-(J2-Pad14) -> Cube_1_A-F7
- J2 pad 27: unconnected-(J2-Pad27) -> Cube_1_A-G6
- J2 pad 28: unconnected-(J2-Pad28) -> Cube_1_A-F6
- J2 pad 29: unconnected-(J2-Pad29) -> Cube_1_A-H6
- J2 pad 30: unconnected-(J2-Pad30) -> Cube_1_A-E6
- J2 pad 31: unconnected-(J2-Pad31) -> Cube_1_A-H5
- J2 pad 32: unconnected-(J2-Pad32) -> Cube_1_A-E5
- J2 pad 33: unconnected-(J2-Pad33) -> Cube_1_A-G5
- J2 pad 34: unconnected-(J2-Pad34) -> Cube_1_A-F5
- J2 pad 47: unconnected-(J2-Pad47) -> Cube_1_A-G4
- J2 pad 48: unconnected-(J2-Pad48) -> Cube_1_A-F4
- J2 pad 49: unconnected-(J2-Pad49) -> Cube_1_A-H4
- J2 pad 50: unconnected-(J2-Pad50) -> Cube_1_A-E4
- J2 pad 51: unconnected-(J2-Pad51) -> Cube_1_A-H3
- J2 pad 52: unconnected-(J2-Pad52) -> Cube_1_A-E3
- J2 pad 53: unconnected-(J2-Pad53) -> Cube_1_A-G3
- J2 pad 54: unconnected-(J2-Pad54) -> Cube_1_A-F3
- J2 pad 67: unconnected-(J2-Pad67) -> Cube_1_A-G2
- J2 pad 68: unconnected-(J2-Pad68) -> Cube_1_A-F2
- J2 pad 69: unconnected-(J2-Pad69) -> Cube_1_A-H2
- J2 pad 70: unconnected-(J2-Pad70) -> Cube_1_A-E2
- J2 pad 71: unconnected-(J2-Pad71) -> Cube_1_A-H1
- J2 pad 72: unconnected-(J2-Pad72) -> Cube_1_A-E1
- J2 pad 73: unconnected-(J2-Pad73) -> Cube_1_A-G1
- J2 pad 74: unconnected-(J2-Pad74) -> Cube_1_A-F1
- J3 pad 07: unconnected-(J3-Pad07) -> Cube_1_A-B1
- J3 pad 08: unconnected-(J3-Pad08) -> Cube_1_A-C1
- J3 pad 09: unconnected-(J3-Pad09) -> Cube_1_A-A1
- J3 pad 10: unconnected-(J3-Pad10) -> Cube_1_A-D1
- J3 pad 11: unconnected-(J3-Pad11) -> Cube_1_A-A2
- J3 pad 12: unconnected-(J3-Pad12) -> Cube_1_A-D2
- J3 pad 13: unconnected-(J3-Pad13) -> Cube_1_A-B2
- J3 pad 14: unconnected-(J3-Pad14) -> Cube_1_A-C2
- J3 pad 27: unconnected-(J3-Pad27) -> Cube_1_A-B3
- J3 pad 28: unconnected-(J3-Pad28) -> Cube_1_A-C3
- J3 pad 29: unconnected-(J3-Pad29) -> Cube_1_A-A3
- J3 pad 30: unconnected-(J3-Pad30) -> Cube_1_A-D3
- J3 pad 31: unconnected-(J3-Pad31) -> Cube_1_A-A4
- J3 pad 32: unconnected-(J3-Pad32) -> Cube_1_A-D4
- J3 pad 33: unconnected-(J3-Pad33) -> Cube_1_A-B4
- J3 pad 34: unconnected-(J3-Pad34) -> Cube_1_A-C4
- J3 pad 47: unconnected-(J3-Pad47) -> Cube_1_A-B5
- J3 pad 48: unconnected-(J3-Pad48) -> Cube_1_A-C5
- J3 pad 49: unconnected-(J3-Pad49) -> Cube_1_A-A5
- J3 pad 50: unconnected-(J3-Pad50) -> Cube_1_A-D5
- J3 pad 51: unconnected-(J3-Pad51) -> Cube_1_A-A6
- J3 pad 52: unconnected-(J3-Pad52) -> Cube_1_A-D6
- J3 pad 53: unconnected-(J3-Pad53) -> Cube_1_A-B6
- J3 pad 54: unconnected-(J3-Pad54) -> Cube_1_A-C6
- J3 pad 67: unconnected-(J3-Pad67) -> Cube_1_A-B7
- J3 pad 68: unconnected-(J3-Pad68) -> Cube_1_A-C7
- J3 pad 69: unconnected-(J3-Pad69) -> Cube_1_A-A7
- J3 pad 70: unconnected-(J3-Pad70) -> Cube_1_A-D7
- J3 pad 71: unconnected-(J3-Pad71) -> Cube_1_A-A8
- J3 pad 72: unconnected-(J3-Pad72) -> Cube_1_A-D8
- J3 pad 73: unconnected-(J3-Pad73) -> Cube_1_A-B8
- J3 pad 74: unconnected-(J3-Pad74) -> Cube_1_A-C8
- J4 pad 07: unconnected-(J4-Pad07) -> Cube_2_A-G8
- J4 pad 08: unconnected-(J4-Pad08) -> Cube_2_A-F8
- J4 pad 09: unconnected-(J4-Pad09) -> Cube_2_A-H8
- J4 pad 10: unconnected-(J4-Pad10) -> Cube_2_A-E8
- J4 pad 11: unconnected-(J4-Pad11) -> Cube_2_A-H7
- J4 pad 12: unconnected-(J4-Pad12) -> Cube_2_A-E7
- J4 pad 13: unconnected-(J4-Pad13) -> Cube_2_A-G7
- J4 pad 14: unconnected-(J4-Pad14) -> Cube_2_A-F7
- J4 pad 27: unconnected-(J4-Pad27) -> Cube_2_A-G6
- J4 pad 28: unconnected-(J4-Pad28) -> Cube_2_A-F6
- J4 pad 29: unconnected-(J4-Pad29) -> Cube_2_A-H6
- J4 pad 30: unconnected-(J4-Pad30) -> Cube_2_A-E6
- J4 pad 31: unconnected-(J4-Pad31) -> Cube_2_A-H5
- J4 pad 32: unconnected-(J4-Pad32) -> Cube_2_A-E5
- J4 pad 33: unconnected-(J4-Pad33) -> Cube_2_A-G5
- J4 pad 34: unconnected-(J4-Pad34) -> Cube_2_A-F5
- J4 pad 47: unconnected-(J4-Pad47) -> Cube_2_A-G4
- J4 pad 48: unconnected-(J4-Pad48) -> Cube_2_A-F4
- J4 pad 49: unconnected-(J4-Pad49) -> Cube_2_A-H4
- J4 pad 50: unconnected-(J4-Pad50) -> Cube_2_A-E4
- J4 pad 51: unconnected-(J4-Pad51) -> Cube_2_A-H3
- J4 pad 52: unconnected-(J4-Pad52) -> Cube_2_A-E3
- J4 pad 53: unconnected-(J4-Pad53) -> Cube_2_A-G3
- J4 pad 54: unconnected-(J4-Pad54) -> Cube_2_A-F3
- J4 pad 67: unconnected-(J4-Pad67) -> Cube_2_A-G2
- J4 pad 68: unconnected-(J4-Pad68) -> Cube_2_A-F2
- J4 pad 69: unconnected-(J4-Pad69) -> Cube_2_A-H2
- J4 pad 70: unconnected-(J4-Pad70) -> Cube_2_A-E2
- J4 pad 71: unconnected-(J4-Pad71) -> Cube_2_A-H1
- J4 pad 72: unconnected-(J4-Pad72) -> Cube_2_A-E1
- J4 pad 73: unconnected-(J4-Pad73) -> Cube_2_A-G1
- J4 pad 74: unconnected-(J4-Pad74) -> Cube_2_A-F1
- MPPC1 pad 1: unconnected-(MPPC1-SignalOut-Pad1) -> Cube_1_A-F1
- MPPC1 pad 10: unconnected-(MPPC1-SignalOut-Pad10) -> Cube_1_A-E2
- MPPC1 pad 100: unconnected-(MPPC1-SignalOut-Pad100) -> Cube_2_A-G4
- MPPC1 pad 101: unconnected-(MPPC1-SignalOut-Pad101) -> Cube_1_A-H5
- MPPC1 pad 102: unconnected-(MPPC1-SignalOut-Pad102) -> Cube_1_A-H5
- MPPC1 pad 103: unconnected-(MPPC1-SignalOut-Pad103) -> Cube_2_A-H4
- MPPC1 pad 104: unconnected-(MPPC1-SignalOut-Pad104) -> Cube_2_A-H4
- MPPC1 pad 105: unconnected-(MPPC1-SignalOut-Pad105) -> Cube_1_A-H6
- MPPC1 pad 106: unconnected-(MPPC1-SignalOut-Pad106) -> Cube_1_A-H6
- MPPC1 pad 107: unconnected-(MPPC1-SignalOut-Pad107) -> Cube_2_A-H3
- MPPC1 pad 108: unconnected-(MPPC1-SignalOut-Pad108) -> Cube_2_A-H3
- MPPC1 pad 109: unconnected-(MPPC1-SignalOut-Pad109) -> Cube_1_A-G6
- MPPC1 pad 11: unconnected-(MPPC1-SignalOut-Pad11) -> Cube_2_A-E7
- MPPC1 pad 110: unconnected-(MPPC1-SignalOut-Pad110) -> Cube_1_A-G6
- MPPC1 pad 111: unconnected-(MPPC1-SignalOut-Pad111) -> Cube_2_A-G3
- MPPC1 pad 112: unconnected-(MPPC1-SignalOut-Pad112) -> Cube_2_A-G3
- MPPC1 pad 113: unconnected-(MPPC1-SignalOut-Pad113) -> Cube_1_A-G7
- MPPC1 pad 114: unconnected-(MPPC1-SignalOut-Pad114) -> Cube_1_A-G7
- MPPC1 pad 115: unconnected-(MPPC1-SignalOut-Pad115) -> Cube_2_A-G2
- MPPC1 pad 116: unconnected-(MPPC1-SignalOut-Pad116) -> Cube_2_A-G2
- MPPC1 pad 117: unconnected-(MPPC1-SignalOut-Pad117) -> Cube_1_A-H7
- MPPC1 pad 118: unconnected-(MPPC1-SignalOut-Pad118) -> Cube_1_A-H7
- MPPC1 pad 119: unconnected-(MPPC1-SignalOut-Pad119) -> Cube_2_A-H2
- MPPC1 pad 12: unconnected-(MPPC1-SignalOut-Pad12) -> Cube_2_A-E7
- MPPC1 pad 120: unconnected-(MPPC1-SignalOut-Pad120) -> Cube_2_A-H2
- MPPC1 pad 121: unconnected-(MPPC1-SignalOut-Pad121) -> Cube_1_A-H8
- MPPC1 pad 122: unconnected-(MPPC1-SignalOut-Pad122) -> Cube_1_A-H8
- MPPC1 pad 123: unconnected-(MPPC1-SignalOut-Pad123) -> Cube_2_A-H1
- MPPC1 pad 124: unconnected-(MPPC1-SignalOut-Pad124) -> Cube_2_A-H1
- MPPC1 pad 125: unconnected-(MPPC1-SignalOut-Pad125) -> Cube_1_A-G8
- MPPC1 pad 126: unconnected-(MPPC1-SignalOut-Pad126) -> Cube_1_A-G8
- MPPC1 pad 127: unconnected-(MPPC1-SignalOut-Pad127) -> Cube_2_A-G1
- MPPC1 pad 128: unconnected-(MPPC1-SignalOut-Pad128) -> Cube_2_A-G1
- MPPC1 pad 129: unconnected-(MPPC1-+HV-Pad129) -> +HV
- MPPC1 pad 13: unconnected-(MPPC1-SignalOut-Pad13) -> Cube_1_A-F2
- MPPC1 pad 130: unconnected-(MPPC1-+HV-Pad130) -> +HV
- MPPC1 pad 131: unconnected-(MPPC1-+HV-Pad131) -> +HV
- MPPC1 pad 132: unconnected-(MPPC1-+HV-Pad132) -> +HV
- MPPC1 pad 133: unconnected-(MPPC1-+HV-Pad133) -> +HV
- MPPC1 pad 134: unconnected-(MPPC1-+HV-Pad134) -> +HV
- MPPC1 pad 135: unconnected-(MPPC1-+HV-Pad135) -> +HV
- MPPC1 pad 136: unconnected-(MPPC1-+HV-Pad136) -> +HV
- MPPC1 pad 137: unconnected-(MPPC1-+HV-Pad137) -> +HV
- MPPC1 pad 138: unconnected-(MPPC1-+HV-Pad138) -> +HV
- MPPC1 pad 139: unconnected-(MPPC1-+HV-Pad139) -> +HV
- MPPC1 pad 14: unconnected-(MPPC1-SignalOut-Pad14) -> Cube_1_A-F2
- MPPC1 pad 140: unconnected-(MPPC1-+HV-Pad140) -> +HV
- MPPC1 pad 141: unconnected-(MPPC1-+HV-Pad141) -> +HV
- MPPC1 pad 142: unconnected-(MPPC1-+HV-Pad142) -> +HV
- MPPC1 pad 143: unconnected-(MPPC1-+HV-Pad143) -> +HV
- MPPC1 pad 144: unconnected-(MPPC1-+HV-Pad144) -> +HV
- MPPC1 pad 145: unconnected-(MPPC1-+HV-Pad145) -> +HV
- MPPC1 pad 146: unconnected-(MPPC1-+HV-Pad146) -> +HV
- MPPC1 pad 147: unconnected-(MPPC1-+HV-Pad147) -> +HV
- MPPC1 pad 148: unconnected-(MPPC1-+HV-Pad148) -> +HV
- MPPC1 pad 149: unconnected-(MPPC1-+HV-Pad149) -> +HV
- MPPC1 pad 15: unconnected-(MPPC1-SignalOut-Pad15) -> Cube_2_A-F7
- MPPC1 pad 150: unconnected-(MPPC1-+HV-Pad150) -> +HV
- MPPC1 pad 151: unconnected-(MPPC1-+HV-Pad151) -> +HV
- MPPC1 pad 152: unconnected-(MPPC1-+HV-Pad152) -> +HV
- MPPC1 pad 153: unconnected-(MPPC1-+HV-Pad153) -> +HV
- MPPC1 pad 154: unconnected-(MPPC1-+HV-Pad154) -> +HV
- MPPC1 pad 155: unconnected-(MPPC1-+HV-Pad155) -> +HV
- MPPC1 pad 156: unconnected-(MPPC1-+HV-Pad156) -> +HV
- MPPC1 pad 157: unconnected-(MPPC1-+HV-Pad157) -> +HV
- MPPC1 pad 158: unconnected-(MPPC1-+HV-Pad158) -> +HV
- MPPC1 pad 159: unconnected-(MPPC1-+HV-Pad159) -> +HV
- MPPC1 pad 16: unconnected-(MPPC1-SignalOut-Pad16) -> Cube_2_A-F7
- MPPC1 pad 160: unconnected-(MPPC1-+HV-Pad160) -> +HV
- MPPC1 pad 161: unconnected-(MPPC1-+HV-Pad161) -> +HV
- MPPC1 pad 162: unconnected-(MPPC1-+HV-Pad162) -> +HV
- MPPC1 pad 17: unconnected-(MPPC1-SignalOut-Pad17) -> Cube_1_A-F3
- MPPC1 pad 18: unconnected-(MPPC1-SignalOut-Pad18) -> Cube_1_A-F3
- MPPC1 pad 19: unconnected-(MPPC1-SignalOut-Pad19) -> Cube_2_A-F6
- MPPC1 pad 2: unconnected-(MPPC1-SignalOut-Pad2) -> Cube_1_A-F1
- MPPC1 pad 20: unconnected-(MPPC1-SignalOut-Pad20) -> Cube_2_A-F6
- MPPC1 pad 21: unconnected-(MPPC1-SignalOut-Pad21) -> Cube_1_A-E3
- MPPC1 pad 22: unconnected-(MPPC1-SignalOut-Pad22) -> Cube_1_A-E3
- MPPC1 pad 23: unconnected-(MPPC1-SignalOut-Pad23) -> Cube_2_A-E6
- MPPC1 pad 24: unconnected-(MPPC1-SignalOut-Pad24) -> Cube_2_A-E6
- MPPC1 pad 25: unconnected-(MPPC1-SignalOut-Pad25) -> Cube_1_A-E4
- MPPC1 pad 26: unconnected-(MPPC1-SignalOut-Pad26) -> Cube_1_A-E4
- MPPC1 pad 27: unconnected-(MPPC1-SignalOut-Pad27) -> Cube_2_A-E5
- MPPC1 pad 28: unconnected-(MPPC1-SignalOut-Pad28) -> Cube_2_A-E5
- MPPC1 pad 29: unconnected-(MPPC1-SignalOut-Pad29) -> Cube_1_A-F4
- MPPC1 pad 3: unconnected-(MPPC1-SignalOut-Pad3) -> Cube_2_A-F8
- MPPC1 pad 30: unconnected-(MPPC1-SignalOut-Pad30) -> Cube_1_A-F4
- MPPC1 pad 31: unconnected-(MPPC1-SignalOut-Pad31) -> Cube_2_A-F5
- MPPC1 pad 32: unconnected-(MPPC1-SignalOut-Pad32) -> Cube_2_A-F5
- MPPC1 pad 33: unconnected-(MPPC1-SignalOut-Pad33) -> Cube_1_A-F5
- MPPC1 pad 34: unconnected-(MPPC1-SignalOut-Pad34) -> Cube_1_A-F5
- MPPC1 pad 35: unconnected-(MPPC1-SignalOut-Pad35) -> Cube_2_A-F4
- MPPC1 pad 36: unconnected-(MPPC1-SignalOut-Pad36) -> Cube_2_A-F4
- MPPC1 pad 37: unconnected-(MPPC1-SignalOut-Pad37) -> Cube_1_A-E5
- MPPC1 pad 38: unconnected-(MPPC1-SignalOut-Pad38) -> Cube_1_A-E5
- MPPC1 pad 39: unconnected-(MPPC1-SignalOut-Pad39) -> Cube_2_A-E4
- MPPC1 pad 4: unconnected-(MPPC1-SignalOut-Pad4) -> Cube_2_A-F8
- MPPC1 pad 40: unconnected-(MPPC1-SignalOut-Pad40) -> Cube_2_A-E4
- MPPC1 pad 41: unconnected-(MPPC1-SignalOut-Pad41) -> Cube_1_A-E6
- MPPC1 pad 42: unconnected-(MPPC1-SignalOut-Pad42) -> Cube_1_A-E6
- MPPC1 pad 43: unconnected-(MPPC1-SignalOut-Pad43) -> Cube_2_A-E3
- MPPC1 pad 44: unconnected-(MPPC1-SignalOut-Pad44) -> Cube_2_A-E3
- MPPC1 pad 45: unconnected-(MPPC1-SignalOut-Pad45) -> Cube_1_A-F6
- MPPC1 pad 46: unconnected-(MPPC1-SignalOut-Pad46) -> Cube_1_A-F6
- MPPC1 pad 47: unconnected-(MPPC1-SignalOut-Pad47) -> Cube_2_A-F3
- MPPC1 pad 48: unconnected-(MPPC1-SignalOut-Pad48) -> Cube_2_A-F3
- MPPC1 pad 49: unconnected-(MPPC1-SignalOut-Pad49) -> Cube_1_A-F7
- MPPC1 pad 5: unconnected-(MPPC1-SignalOut-Pad5) -> Cube_1_A-E1
- MPPC1 pad 50: unconnected-(MPPC1-SignalOut-Pad50) -> Cube_1_A-F7
- MPPC1 pad 51: unconnected-(MPPC1-SignalOut-Pad51) -> Cube_2_A-F2
- MPPC1 pad 52: unconnected-(MPPC1-SignalOut-Pad52) -> Cube_2_A-F2
- MPPC1 pad 53: unconnected-(MPPC1-SignalOut-Pad53) -> Cube_1_A-E7
- MPPC1 pad 54: unconnected-(MPPC1-SignalOut-Pad54) -> Cube_1_A-E7
- MPPC1 pad 55: unconnected-(MPPC1-SignalOut-Pad55) -> Cube_2_A-E2
- MPPC1 pad 56: unconnected-(MPPC1-SignalOut-Pad56) -> Cube_2_A-E2
- MPPC1 pad 57: unconnected-(MPPC1-SignalOut-Pad57) -> Cube_1_A-E8
- MPPC1 pad 58: unconnected-(MPPC1-SignalOut-Pad58) -> Cube_1_A-E8
- MPPC1 pad 59: unconnected-(MPPC1-SignalOut-Pad59) -> Cube_2_A-E1
- MPPC1 pad 6: unconnected-(MPPC1-SignalOut-Pad6) -> Cube_1_A-E1
- MPPC1 pad 60: unconnected-(MPPC1-SignalOut-Pad60) -> Cube_2_A-E1
- MPPC1 pad 61: unconnected-(MPPC1-SignalOut-Pad61) -> Cube_1_A-F8
- MPPC1 pad 62: unconnected-(MPPC1-SignalOut-Pad62) -> Cube_1_A-F8
- MPPC1 pad 63: unconnected-(MPPC1-SignalOut-Pad63) -> Cube_2_A-F1
- MPPC1 pad 64: unconnected-(MPPC1-SignalOut-Pad64) -> Cube_2_A-F1
- MPPC1 pad 65: unconnected-(MPPC1-SignalOut-Pad65) -> Cube_1_A-G1
- MPPC1 pad 66: unconnected-(MPPC1-SignalOut-Pad66) -> Cube_1_A-G1
- MPPC1 pad 67: unconnected-(MPPC1-SignalOut-Pad67) -> Cube_2_A-G8
- MPPC1 pad 68: unconnected-(MPPC1-SignalOut-Pad68) -> Cube_2_A-G8
- MPPC1 pad 69: unconnected-(MPPC1-SignalOut-Pad69) -> Cube_1_A-H1
- MPPC1 pad 7: unconnected-(MPPC1-SignalOut-Pad7) -> Cube_2_A-E8
- MPPC1 pad 70: unconnected-(MPPC1-SignalOut-Pad70) -> Cube_1_A-H1
- MPPC1 pad 71: unconnected-(MPPC1-SignalOut-Pad71) -> Cube_2_A-H8
- MPPC1 pad 72: unconnected-(MPPC1-SignalOut-Pad72) -> Cube_2_A-H8
- MPPC1 pad 73: unconnected-(MPPC1-SignalOut-Pad73) -> Cube_1_A-H2
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Routing:
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
Commit message: .
Parts:
- removed J10, J11, J12, J13: ST4-40-1.00-L-D-P-TR, FARICH:SAMTEC_ST4-40-1.00-L-D-P-TR
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- renumbered J8 to J7, J7 to J8
Connections:
- J3 pad 07: Cube_1_A-B1 -> Cube_1_A-C8
- J3 pad 08: Cube_1_A-C1 -> Cube_1_A-B8
- J3 pad 09: Cube_1_A-A1 -> Cube_1_A-D8
- J3 pad 10: Cube_1_A-D1 -> Cube_1_A-A8
- J3 pad 11: Cube_1_A-A2 -> Cube_1_A-D7
- J3 pad 12: Cube_1_A-D2 -> Cube_1_A-A7
- J3 pad 13: Cube_1_A-B2 -> Cube_1_A-C7
- J3 pad 14: Cube_1_A-C2 -> Cube_1_A-B7
- J3 pad 27: Cube_1_A-B3 -> Cube_1_A-C6
- J3 pad 28: Cube_1_A-C3 -> Cube_1_A-B6
- J3 pad 29: Cube_1_A-A3 -> Cube_1_A-D6
- J3 pad 30: Cube_1_A-D3 -> Cube_1_A-A6
- J3 pad 31: Cube_1_A-A4 -> Cube_1_A-D5
- J3 pad 32: Cube_1_A-D4 -> Cube_1_A-A5
- J3 pad 33: Cube_1_A-B4 -> Cube_1_A-C5
- J3 pad 34: Cube_1_A-C4 -> Cube_1_A-B5
- J3 pad 47: Cube_1_A-B5 -> Cube_1_A-C4
- J3 pad 48: Cube_1_A-C5 -> Cube_1_A-B4
- J3 pad 49: Cube_1_A-A5 -> Cube_1_A-D4
- J3 pad 50: Cube_1_A-D5 -> Cube_1_A-A4
- J3 pad 51: Cube_1_A-A6 -> Cube_1_A-D3
- J3 pad 52: Cube_1_A-D6 -> Cube_1_A-A3
- J3 pad 53: Cube_1_A-B6 -> Cube_1_A-C3
- J3 pad 54: Cube_1_A-C6 -> Cube_1_A-B3
- J3 pad 67: Cube_1_A-B7 -> Cube_1_A-C2
- J3 pad 68: Cube_1_A-C7 -> Cube_1_A-B2
- J3 pad 69: Cube_1_A-A7 -> Cube_1_A-D2
- J3 pad 70: Cube_1_A-D7 -> Cube_1_A-A2
- J3 pad 71: Cube_1_A-A8 -> Cube_1_A-D1
- J3 pad 72: Cube_1_A-D8 -> Cube_1_A-A1
- J3 pad 73: Cube_1_A-B8 -> Cube_1_A-C1
- J3 pad 74: Cube_1_A-C8 -> Cube_1_A-B1
- J5 pad 07: unconnected-(J5-Pad07) -> Cube_2_A-C8
- J5 pad 08: unconnected-(J5-Pad08) -> Cube_2_A-B8
- J5 pad 09: unconnected-(J5-Pad09) -> Cube_2_A-D8
- J5 pad 10: unconnected-(J5-Pad10) -> Cube_2_A-A8
- J5 pad 11: unconnected-(J5-Pad11) -> Cube_2_A-D7
- J5 pad 12: unconnected-(J5-Pad12) -> Cube_2_A-A7
- J5 pad 13: unconnected-(J5-Pad13) -> Cube_2_A-C7
- J5 pad 14: unconnected-(J5-Pad14) -> Cube_2_A-B7
- J5 pad 27: unconnected-(J5-Pad27) -> Cube_2_A-C6
- J5 pad 28: unconnected-(J5-Pad28) -> Cube_2_A-B6
- J5 pad 29: unconnected-(J5-Pad29) -> Cube_2_A-D6
- J5 pad 30: unconnected-(J5-Pad30) -> Cube_2_A-A6
- J5 pad 31: unconnected-(J5-Pad31) -> Cube_2_A-D5
- J5 pad 32: unconnected-(J5-Pad32) -> Cube_2_A-A5
- J5 pad 33: unconnected-(J5-Pad33) -> Cube_2_A-C5
- J5 pad 34: unconnected-(J5-Pad34) -> Cube_2_A-B5
- J5 pad 47: unconnected-(J5-Pad47) -> Cube_2_A-C4
- J5 pad 48: unconnected-(J5-Pad48) -> Cube_2_A-B4
- J5 pad 49: unconnected-(J5-Pad49) -> Cube_2_A-D4
- J5 pad 50: unconnected-(J5-Pad50) -> Cube_2_A-A4
- J5 pad 51: unconnected-(J5-Pad51) -> Cube_2_A-D3
- J5 pad 52: unconnected-(J5-Pad52) -> Cube_2_A-A3
- J5 pad 53: unconnected-(J5-Pad53) -> Cube_2_A-C3
- J5 pad 54: unconnected-(J5-Pad54) -> Cube_2_A-B3
- J5 pad 67: unconnected-(J5-Pad67) -> Cube_2_A-C2
- J5 pad 68: unconnected-(J5-Pad68) -> Cube_2_A-B2
- J5 pad 69: unconnected-(J5-Pad69) -> Cube_2_A-D2
- J5 pad 70: unconnected-(J5-Pad70) -> Cube_2_A-A2
- J5 pad 71: unconnected-(J5-Pad71) -> Cube_2_A-D1
- J5 pad 72: unconnected-(J5-Pad72) -> Cube_2_A-A1
- J5 pad 73: unconnected-(J5-Pad73) -> Cube_2_A-C1
- J5 pad 74: unconnected-(J5-Pad74) -> Cube_2_A-B1
- J6 pad 07: unconnected-(J6-Pad07) -> Cube_3_A-G8
- J6 pad 08: unconnected-(J6-Pad08) -> Cube_3_A-F8
- J6 pad 09: unconnected-(J6-Pad09) -> Cube_3_A-H8
- J6 pad 10: unconnected-(J6-Pad10) -> Cube_3_A-E8
- J6 pad 11: unconnected-(J6-Pad11) -> Cube_3_A-H7
- J6 pad 12: unconnected-(J6-Pad12) -> Cube_3_A-E7
- J6 pad 13: unconnected-(J6-Pad13) -> Cube_3_A-G7
- J6 pad 14: unconnected-(J6-Pad14) -> Cube_3_A-F7
- J6 pad 27: unconnected-(J6-Pad27) -> Cube_3_A-G6
- J6 pad 28: unconnected-(J6-Pad28) -> Cube_3_A-F6
- J6 pad 29: unconnected-(J6-Pad29) -> Cube_3_A-H6
- J6 pad 30: unconnected-(J6-Pad30) -> Cube_3_A-E6
- J6 pad 31: unconnected-(J6-Pad31) -> Cube_3_A-H5
- J6 pad 32: unconnected-(J6-Pad32) -> Cube_3_A-E5
- J6 pad 33: unconnected-(J6-Pad33) -> Cube_3_A-G5
- J6 pad 34: unconnected-(J6-Pad34) -> Cube_3_A-F5
- J6 pad 47: unconnected-(J6-Pad47) -> Cube_3_A-G4
- J6 pad 48: unconnected-(J6-Pad48) -> Cube_3_A-F4
- J6 pad 49: unconnected-(J6-Pad49) -> Cube_3_A-H4
- J6 pad 50: unconnected-(J6-Pad50) -> Cube_3_A-E4
- J6 pad 51: unconnected-(J6-Pad51) -> Cube_3_A-H3
- J6 pad 52: unconnected-(J6-Pad52) -> Cube_3_A-E3
- J6 pad 53: unconnected-(J6-Pad53) -> Cube_3_A-G3
- J6 pad 54: unconnected-(J6-Pad54) -> Cube_3_A-F3
- J6 pad 67: unconnected-(J6-Pad67) -> Cube_3_A-G2
- J6 pad 68: unconnected-(J6-Pad68) -> Cube_3_A-F2
- J6 pad 69: unconnected-(J6-Pad69) -> Cube_3_A-H2
- J6 pad 70: unconnected-(J6-Pad70) -> Cube_3_A-E2
- J6 pad 71: unconnected-(J6-Pad71) -> Cube_3_A-H1
- J6 pad 72: unconnected-(J6-Pad72) -> Cube_3_A-E1
- J6 pad 73: unconnected-(J6-Pad73) -> Cube_3_A-G1
- J6 pad 74: unconnected-(J6-Pad74) -> Cube_3_A-F1
- J7 pad 07: unconnected-(J8-Pad07) -> Cube_4_A-G8
- J7 pad 08: unconnected-(J8-Pad08) -> Cube_4_A-F8
- J7 pad 09: unconnected-(J8-Pad09) -> Cube_4_A-H8
- J7 pad 10: unconnected-(J8-Pad10) -> Cube_4_A-E8
- J7 pad 11: unconnected-(J8-Pad11) -> Cube_4_A-H7
- J7 pad 12: unconnected-(J8-Pad12) -> Cube_4_A-E7
- J7 pad 13: unconnected-(J8-Pad13) -> Cube_4_A-G7
- J7 pad 14: unconnected-(J8-Pad14) -> Cube_4_A-F7
- J7 pad 27: unconnected-(J8-Pad27) -> Cube_4_A-G6
- J7 pad 28: unconnected-(J8-Pad28) -> Cube_4_A-F6
- J7 pad 29: unconnected-(J8-Pad29) -> Cube_4_A-H6
- J7 pad 30: unconnected-(J8-Pad30) -> Cube_4_A-E6
- J7 pad 31: unconnected-(J8-Pad31) -> Cube_4_A-H5
- J7 pad 32: unconnected-(J8-Pad32) -> Cube_4_A-E5
- J7 pad 33: unconnected-(J8-Pad33) -> Cube_4_A-G5
- J7 pad 34: unconnected-(J8-Pad34) -> Cube_4_A-F5
- J7 pad 47: unconnected-(J8-Pad47) -> Cube_4_A-G4
- J7 pad 48: unconnected-(J8-Pad48) -> Cube_4_A-F4
- J7 pad 49: unconnected-(J8-Pad49) -> Cube_4_A-H4
- J7 pad 50: unconnected-(J8-Pad50) -> Cube_4_A-E4
- J7 pad 51: unconnected-(J8-Pad51) -> Cube_4_A-H3
- J7 pad 52: unconnected-(J8-Pad52) -> Cube_4_A-E3
- J7 pad 53: unconnected-(J8-Pad53) -> Cube_4_A-G3
- J7 pad 54: unconnected-(J8-Pad54) -> Cube_4_A-F3
- J7 pad 67: unconnected-(J8-Pad67) -> Cube_4_A-G2
- J7 pad 68: unconnected-(J8-Pad68) -> Cube_4_A-F2
- J7 pad 69: unconnected-(J8-Pad69) -> Cube_4_A-H2
- J7 pad 70: unconnected-(J8-Pad70) -> Cube_4_A-E2
- J7 pad 71: unconnected-(J8-Pad71) -> Cube_4_A-H1
- J7 pad 72: unconnected-(J8-Pad72) -> Cube_4_A-E1
- J7 pad 73: unconnected-(J8-Pad73) -> Cube_4_A-G1
- J7 pad 74: unconnected-(J8-Pad74) -> Cube_4_A-F1
- J8 pad 07: unconnected-(J7-Pad07) -> Cube_3_A-C8
- J8 pad 08: unconnected-(J7-Pad08) -> Cube_3_A-B8
- J8 pad 09: unconnected-(J7-Pad09) -> Cube_3_A-D8
- J8 pad 10: unconnected-(J7-Pad10) -> Cube_3_A-A8
- J8 pad 11: unconnected-(J7-Pad11) -> Cube_3_A-D7
- J8 pad 12: unconnected-(J7-Pad12) -> Cube_3_A-A7
- J8 pad 13: unconnected-(J7-Pad13) -> Cube_3_A-C7
- J8 pad 14: unconnected-(J7-Pad14) -> Cube_3_A-B7
- J8 pad 27: unconnected-(J7-Pad27) -> Cube_3_A-C6
- J8 pad 28: unconnected-(J7-Pad28) -> Cube_3_A-B6
- J8 pad 29: unconnected-(J7-Pad29) -> Cube_3_A-D6
- J8 pad 30: unconnected-(J7-Pad30) -> Cube_3_A-A6
- J8 pad 31: unconnected-(J7-Pad31) -> Cube_3_A-D5
- J8 pad 32: unconnected-(J7-Pad32) -> Cube_3_A-A5
- J8 pad 33: unconnected-(J7-Pad33) -> Cube_3_A-C5
- J8 pad 34: unconnected-(J7-Pad34) -> Cube_3_A-B5
- J8 pad 47: unconnected-(J7-Pad47) -> Cube_3_A-C4
- J8 pad 48: unconnected-(J7-Pad48) -> Cube_3_A-B4
- J8 pad 49: unconnected-(J7-Pad49) -> Cube_3_A-D4
- J8 pad 50: unconnected-(J7-Pad50) -> Cube_3_A-A4
- J8 pad 51: unconnected-(J7-Pad51) -> Cube_3_A-D3
- J8 pad 52: unconnected-(J7-Pad52) -> Cube_3_A-A3
- J8 pad 53: unconnected-(J7-Pad53) -> Cube_3_A-C3
- J8 pad 54: unconnected-(J7-Pad54) -> Cube_3_A-B3
- J8 pad 67: unconnected-(J7-Pad67) -> Cube_3_A-C2
- J8 pad 68: unconnected-(J7-Pad68) -> Cube_3_A-B2
- J8 pad 69: unconnected-(J7-Pad69) -> Cube_3_A-D2
- J8 pad 70: unconnected-(J7-Pad70) -> Cube_3_A-A2
- J8 pad 71: unconnected-(J7-Pad71) -> Cube_3_A-D1
- J8 pad 72: unconnected-(J7-Pad72) -> Cube_3_A-A1
- J8 pad 73: unconnected-(J7-Pad73) -> Cube_3_A-C1
- J8 pad 74: unconnected-(J7-Pad74) -> Cube_3_A-B1
- J9 pad 07: unconnected-(J9-Pad07) -> Cube_4_A-C8
- J9 pad 08: unconnected-(J9-Pad08) -> Cube_4_A-B8
- J9 pad 09: unconnected-(J9-Pad09) -> Cube_4_A-D8
- J9 pad 10: unconnected-(J9-Pad10) -> Cube_4_A-A8
- J9 pad 11: unconnected-(J9-Pad11) -> Cube_4_A-D7
- J9 pad 12: unconnected-(J9-Pad12) -> Cube_4_A-A7
- J9 pad 13: unconnected-(J9-Pad13) -> Cube_4_A-C7
- J9 pad 14: unconnected-(J9-Pad14) -> Cube_4_A-B7
- J9 pad 27: unconnected-(J9-Pad27) -> Cube_4_A-C6
- J9 pad 28: unconnected-(J9-Pad28) -> Cube_4_A-B6
- J9 pad 29: unconnected-(J9-Pad29) -> Cube_4_A-D6
- J9 pad 30: unconnected-(J9-Pad30) -> Cube_4_A-A6
- J9 pad 31: unconnected-(J9-Pad31) -> Cube_4_A-D5
- J9 pad 32: unconnected-(J9-Pad32) -> Cube_4_A-A5
- J9 pad 33: unconnected-(J9-Pad33) -> Cube_4_A-C5
- J9 pad 34: unconnected-(J9-Pad34) -> Cube_4_A-B5
- J9 pad 47: unconnected-(J9-Pad47) -> Cube_4_A-C4
- J9 pad 48: unconnected-(J9-Pad48) -> Cube_4_A-B4
- J9 pad 49: unconnected-(J9-Pad49) -> Cube_4_A-D4
- J9 pad 50: unconnected-(J9-Pad50) -> Cube_4_A-A4
- J9 pad 51: unconnected-(J9-Pad51) -> Cube_4_A-D3
- J9 pad 52: unconnected-(J9-Pad52) -> Cube_4_A-A3
- J9 pad 53: unconnected-(J9-Pad53) -> Cube_4_A-C3
- J9 pad 54: unconnected-(J9-Pad54) -> Cube_4_A-B3
- J9 pad 67: unconnected-(J9-Pad67) -> Cube_4_A-C2
- J9 pad 68: unconnected-(J9-Pad68) -> Cube_4_A-B2
- J9 pad 69: unconnected-(J9-Pad69) -> Cube_4_A-D2
- J9 pad 70: unconnected-(J9-Pad70) -> Cube_4_A-A2
- J9 pad 71: unconnected-(J9-Pad71) -> Cube_4_A-D1
- J9 pad 72: unconnected-(J9-Pad72) -> Cube_4_A-A1
- J9 pad 73: unconnected-(J9-Pad73) -> Cube_4_A-C1
- J9 pad 74: unconnected-(J9-Pad74) -> Cube_4_A-B1
- MPPC2 pad 1: unconnected-(MPPC2-SignalOut-Pad1) -> Cube_1_A-B1
- MPPC2 pad 10: unconnected-(MPPC2-SignalOut-Pad10) -> Cube_1_A-A2
- MPPC2 pad 100: unconnected-(MPPC2-SignalOut-Pad100) -> Cube_2_A-C4
- MPPC2 pad 101: unconnected-(MPPC2-SignalOut-Pad101) -> Cube_1_A-D5
- MPPC2 pad 102: unconnected-(MPPC2-SignalOut-Pad102) -> Cube_1_A-D5
- MPPC2 pad 103: unconnected-(MPPC2-SignalOut-Pad103) -> Cube_2_A-D4
- MPPC2 pad 104: unconnected-(MPPC2-SignalOut-Pad104) -> Cube_2_A-D4
- MPPC2 pad 105: unconnected-(MPPC2-SignalOut-Pad105) -> Cube_1_A-D6
- MPPC2 pad 106: unconnected-(MPPC2-SignalOut-Pad106) -> Cube_1_A-D6
- MPPC2 pad 107: unconnected-(MPPC2-SignalOut-Pad107) -> Cube_2_A-D3
- MPPC2 pad 108: unconnected-(MPPC2-SignalOut-Pad108) -> Cube_2_A-D3
- MPPC2 pad 109: unconnected-(MPPC2-SignalOut-Pad109) -> Cube_1_A-C6
- MPPC2 pad 11: unconnected-(MPPC2-SignalOut-Pad11) -> Cube_2_A-A7
- MPPC2 pad 110: unconnected-(MPPC2-SignalOut-Pad110) -> Cube_1_A-C6
- MPPC2 pad 111: unconnected-(MPPC2-SignalOut-Pad111) -> Cube_2_A-C3
- MPPC2 pad 112: unconnected-(MPPC2-SignalOut-Pad112) -> Cube_2_A-C3
- MPPC2 pad 113: unconnected-(MPPC2-SignalOut-Pad113) -> Cube_1_A-C7
- MPPC2 pad 114: unconnected-(MPPC2-SignalOut-Pad114) -> Cube_1_A-C7
- MPPC2 pad 115: unconnected-(MPPC2-SignalOut-Pad115) -> Cube_2_A-C2
- MPPC2 pad 116: unconnected-(MPPC2-SignalOut-Pad116) -> Cube_2_A-C2
- MPPC2 pad 117: unconnected-(MPPC2-SignalOut-Pad117) -> Cube_1_A-D7
- MPPC2 pad 118: unconnected-(MPPC2-SignalOut-Pad118) -> Cube_1_A-D7
- MPPC2 pad 119: unconnected-(MPPC2-SignalOut-Pad119) -> Cube_2_A-D2
- MPPC2 pad 12: unconnected-(MPPC2-SignalOut-Pad12) -> Cube_2_A-A7
- MPPC2 pad 120: unconnected-(MPPC2-SignalOut-Pad120) -> Cube_2_A-D2
- MPPC2 pad 121: unconnected-(MPPC2-SignalOut-Pad121) -> Cube_1_A-D8
- MPPC2 pad 122: unconnected-(MPPC2-SignalOut-Pad122) -> Cube_1_A-D8
- MPPC2 pad 123: unconnected-(MPPC2-SignalOut-Pad123) -> Cube_2_A-D1
- MPPC2 pad 124: unconnected-(MPPC2-SignalOut-Pad124) -> Cube_2_A-D1
- MPPC2 pad 125: unconnected-(MPPC2-SignalOut-Pad125) -> Cube_1_A-C8
- MPPC2 pad 126: unconnected-(MPPC2-SignalOut-Pad126) -> Cube_1_A-C8
- MPPC2 pad 127: unconnected-(MPPC2-SignalOut-Pad127) -> Cube_2_A-C1
- MPPC2 pad 128: unconnected-(MPPC2-SignalOut-Pad128) -> Cube_2_A-C1
- MPPC2 pad 13: unconnected-(MPPC2-SignalOut-Pad13) -> Cube_1_A-B2
- MPPC2 pad 14: unconnected-(MPPC2-SignalOut-Pad14) -> Cube_1_A-B2
- MPPC2 pad 15: unconnected-(MPPC2-SignalOut-Pad15) -> Cube_2_A-B7
- MPPC2 pad 16: unconnected-(MPPC2-SignalOut-Pad16) -> Cube_2_A-B7
- MPPC2 pad 17: unconnected-(MPPC2-SignalOut-Pad17) -> Cube_1_A-B3
- MPPC2 pad 18: unconnected-(MPPC2-SignalOut-Pad18) -> Cube_1_A-B3
- MPPC2 pad 19: unconnected-(MPPC2-SignalOut-Pad19) -> Cube_2_A-B6
- MPPC2 pad 2: unconnected-(MPPC2-SignalOut-Pad2) -> Cube_1_A-B1
- MPPC2 pad 20: unconnected-(MPPC2-SignalOut-Pad20) -> Cube_2_A-B6
- MPPC2 pad 21: unconnected-(MPPC2-SignalOut-Pad21) -> Cube_1_A-A3
- MPPC2 pad 22: unconnected-(MPPC2-SignalOut-Pad22) -> Cube_1_A-A3
- MPPC2 pad 23: unconnected-(MPPC2-SignalOut-Pad23) -> Cube_2_A-A6
- MPPC2 pad 24: unconnected-(MPPC2-SignalOut-Pad24) -> Cube_2_A-A6
- MPPC2 pad 25: unconnected-(MPPC2-SignalOut-Pad25) -> Cube_1_A-A4
- MPPC2 pad 26: unconnected-(MPPC2-SignalOut-Pad26) -> Cube_1_A-A4
- MPPC2 pad 27: unconnected-(MPPC2-SignalOut-Pad27) -> Cube_2_A-A5
- MPPC2 pad 28: unconnected-(MPPC2-SignalOut-Pad28) -> Cube_2_A-A5
- MPPC2 pad 29: unconnected-(MPPC2-SignalOut-Pad29) -> Cube_1_A-B4
- MPPC2 pad 3: unconnected-(MPPC2-SignalOut-Pad3) -> Cube_2_A-B8
- MPPC2 pad 30: unconnected-(MPPC2-SignalOut-Pad30) -> Cube_1_A-B4
- MPPC2 pad 31: unconnected-(MPPC2-SignalOut-Pad31) -> Cube_2_A-B5
- MPPC2 pad 32: unconnected-(MPPC2-SignalOut-Pad32) -> Cube_2_A-B5
- MPPC2 pad 33: unconnected-(MPPC2-SignalOut-Pad33) -> Cube_1_A-B5
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Routing:
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- removed copper zone on In5.Cu, net GND
- removed copper zone on In6.Cu, net GND
Other:
- copper layers 8 -> 6
