File: 4-MPPC_FARICH_Prototype/4-MPPC_FARICH_Prototype.kicad_pcb (KiCad board)
At the start: 6 copper layers, 164.1 x 52.9 mm, 43 parts, among them J1 1778764, J2 ST4-40-1.00-L-D-P-TR, J3 ST4-40-1.00-L-D-P-TR, J4 ST4-40-1.00-L-D-P-TR, J5 ST4-40-1.00-L-D-P-TR, J6 ST4-40-1.00-L-D-P-TR, J7 ST4-40-1.00-L-D-P-TR, J8 ST4-40-1.00-L-D-P-TR, J9 ST4-40-1.00-L-D-P-TR

Commit message: .
Connections:
- J1 pad SH1: (no net) -> GND
- J1 pad SH2: (no net) -> GND
Routing:
- net +HV: track 6.36 -> 0.00 mm, vias 20 -> 21
- net Cube_1_A-F3: track 2.68 -> 0.00 mm
- net Cube_3_A-F3: track 2.68 -> 0.00 mm
- net Cube_3_A-C3: track 2.68 -> 0.00 mm
- net Cube_1_A-B3: track 2.68 -> 0.00 mm
- net Cube_1_A-A8: track 2.68 -> 0.00 mm
- net Cube_4_A-C7: track 2.68 -> 0.00 mm
- net Cube_4_A-C3: track 2.68 -> 0.00 mm
- net Cube_4_A-G6: track 2.68 -> 0.00 mm
- net Cube_4_A-B7: track 2.68 -> 0.00 mm
- net Cube_4_A-B5: track 2.68 -> 0.00 mm
- net Cube_4_A-B1: track 2.68 -> 0.00 mm
- net Cube_2_A-F5: track 2.68 -> 0.00 mm
- net Cube_3_A-F1: track 2.68 -> 0.00 mm
- net Cube_2_A-B7: track 2.68 -> 0.00 mm
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- removed copper zone on B.Cu, net +HV
