File: 4-MPPC_FARICH_Prototype/4-MPPC_FARICH_Prototype.kicad_sch (KiCad schematic)
At the start: 4 parts

Commit message: .
Parts:
- added J1: 1778764, HV_Connector:PHOENIX_1778764, symbol HV_Connector:1778764
- added J10, J11, J12, J13, J2, J3, J4, J5, J6, J7, J8, J9: ST4-40-1.00-L-D-P-TR, FARICH:SAMTEC_ST4-40-1.00-L-D-P-TR, symbol FARICH:ST4-40-1.00-L-D-P-TR
Connections:
- new net +HV: J1.1
- new net GND: J1.2
Other:
- note added: "Cube_1"
- note added: "Cube_2"
- note added: "Cube_3"
- note added: "Cube_4"
- note added: "Cube_5"
- note added: "Cube_6"
- moved on the sheet: MPPC1, MPPC2, MPPC3, MPPC4

Commit message: .
Parts:
- added H1, H2, H3, H4: MountingHole, MountingHole:MountingHole_3.2mm_M3_DIN965_Pad, symbol Mechanical:MountingHole

Commit message: .
Connections:
- net GND: now also J10.05, J10.06, J10.15, J10.16, J10.25, J10.26, J10.35, J10.36, J10.45, J10.46, J10.55, J10.56, J10.65, J10.66, J10.75, J10.76, J11.05, J11.06, J11.15, J11.16, J11.25, J11.26, J11.35, J11.36, J11.45, J11.46, J11.55, J11.56, J11.65, J11.66, J11.75, J11.76, J12.05, J12.06, J12.15, J12.16, J12.25, J12.26, J12.35, J12.36, J12.45, J12.46, J12.55, J12.56, J12.65, J12.66, J12.75, J12.76, J13.05, J13.06, J13.15, J13.16, J13.25, J13.26, J13.35, J13.36, J13.45, J13.46, J13.55, J13.56, J13.65, J13.66, J13.75, J13.76, J2.05, J2.06, J2.15, J2.16, J2.25, J2.26, J2.35, J2.36, J2.45, J2.46, J2.55, J2.56, J2.65, J2.66, J2.75, J2.76, J3.05, J3.06, J3.15, J3.16, J3.25, J3.26, J3.35, J3.36, J3.45, J3.46, J3.55, J3.56, J3.65, J3.66, J3.75, J3.76, J4.05, J4.06, J4.15, J4.16, J4.25, J4.26, J4.35, J4.36, J4.45, J4.46, J4.55, J4.56, J4.65, J4.66, J4.75, J4.76, J5.05, J5.06, J5.15, J5.16, J5.25, J5.26, J5.35, J5.36, J5.45, J5.46, J5.55, J5.56, J5.65, J5.66, J5.75, J5.76, J6.05, J6.06, J6.15, J6.16, J6.25, J6.26, J6.35, J6.36, J6.45, J6.46, J6.55, J6.56, J6.65, J6.66, J6.75, J6.76, J7.05, J7.06, J7.15, J7.16, J7.25, J7.26, J7.35, J7.36, J7.45, J7.46, J7.55, J7.56, J7.65, J7.66, J7.75, J7.76, J8.05, J8.06, J8.15, J8.16, J8.25, J8.26, J8.35, J8.36, J8.45, J8.46, J8.55, J8.56, J8.65, J8.66, J8.75, J8.76, J9.05, J9.06, J9.15, J9.16, J9.25, J9.26, J9.35, J9.36, J9.45, J9.46, J9.55, J9.56, J9.65, J9.66, J9.75, J9.76
- net Onboard_HV: now reaches J9.01
- net Onboard_HV: now also J10.01, J10.02, J10.03, J10.04, J10.17, J10.18, J10.19, J10.20, J10.21, J10.22, J10.23, J10.24, J10.37, J10.38, J10.39, J10.40, J10.41, J10.42, J10.43, J10.44, J10.57, J10.58, J10.59, J10.60, J10.61, J10.62, J10.63, J10.64, J10.77, J10.78, J10.79, J10.80, J11.01, J11.02, J11.03, J11.04, J11.17, J11.18, J11.19, J11.20, J11.21, J11.22, J11.23, J11.24, J11.37, J11.38, J11.39, J11.40, J11.41, J11.42, J11.43, J11.44, J11.57, J11.58, J11.59, J11.60, J11.61, J11.62, J11.63, J11.64, J11.77, J11.78, J11.79, J11.80, J12.01, J12.02, J12.03, J12.04, J12.17, J12.18, J12.19, J12.20, J12.21, J12.22, J12.23, J12.24, J12.37, J12.38, J12.39, J12.40, J12.41, J12.42, J12.43, J12.44, J12.57, J12.58, J12.59, J12.60, J12.61, J12.62, J12.63, J12.64, J12.77, J12.78, J12.79, J12.80, J13.01, J13.02, J13.03, J13.04, J13.17, J13.18, J13.19, J13.20, J13.21, J13.22, J13.23, J13.24, J13.37, J13.38, J13.39, J13.40, J13.41, J13.42, J13.43, J13.44, J13.57, J13.58, J13.59, J13.60, J13.61, J13.62, J13.63, J13.64, J13.77, J13.78, J13.79, J13.80, J2.01, J2.02, J2.03, J2.04, J2.17, J2.18, J2.19, J2.20, J2.21, J2.22, J2.23, J2.24, J2.37, J2.38, J2.39, J2.40, J2.41, J2.42, J2.43, J2.44, J2.57, J2.58, J2.59, J2.60, J2.61, J2.62, J2.63, J2.64, J2.77, J2.78, J2.79, J2.80, J3.01, J3.02, J3.03, J3.04, J3.17, J3.18, J3.19, J3.20, J3.21, J3.22, J3.23, J3.24, J3.37, J3.38, J3.39, J3.40, J3.41, J3.42, J3.43, J3.44, J3.57, J3.58, J3.59, J3.60, J3.61, J3.62, J3.63, J3.64, J3.77, J3.78, J3.79, J3.80, J4.01, J4.02, J4.03, J4.04, J4.17, J4.18, J4.19, J4.20, J4.21, J4.22, J4.23, J4.24, J4.37, J4.38, J4.39, J4.40, J4.41, J4.42, J4.43, J4.44, J4.57, J4.58, J4.59, J4.60, J4.61, J4.62, J4.63, J4.64, J4.77, J4.78, J4.79, J4.80, J5.01, J5.02, J5.03, J5.04, J5.17, J5.18, J5.19, J5.20, J5.21, J5.22, J5.23, J5.24, J5.37, J5.38, J5.39, J5.40, J5.41, J5.42, J5.43, J5.44, J5.57, J5.58, J5.59, J5.60, J5.61, J5.62, J5.63, J5.64, J5.77, J5.78, J5.79, J5.80, J6.01, J6.02, J6.03, J6.04, J6.17, J6.18, J6.19, J6.20, J6.21, J6.22, J6.23, J6.24, J6.37, J6.38, J6.39, J6.40, J6.41, J6.42, J6.43, J6.44, J6.57, J6.58, J6.59, J6.60, J6.61, J6.62, J6.63, J6.64, J6.77, J6.78, J6.79, J6.80, J7.01, J7.02, J7.03, J7.04, J7.17, J7.18, J7.19, J7.20, J7.21, J7.22, J7.23, J7.24, J7.37, J7.38, J7.39, J7.40, J7.41, J7.42, J7.43, J7.44, J7.57, J7.58, J7.59, J7.60, J7.61, J7.62, J7.63, J7.64, J7.77, J7.78, J7.79, J7.80, J8.01, J8.02, J8.03, J8.04, J8.17, J8.18, J8.19, J8.20, J8.21, J8.22, J8.23, J8.24, J8.37, J8.38, J8.39, J8.40, J8.41, J8.42, J8.43, J8.44, J8.57, J8.58, J8.59, J8.60, J8.61, J8.62, J8.63, J8.64, J8.77, J8.78, J8.79, J8.80, J9.02, J9.03, J9.04, J9.17, J9.18, J9.19, J9.20, J9.21, J9.22, J9.23, J9.24, J9.37, J9.38, J9.39, J9.40, J9.41, J9.42, J9.43, J9.44, J9.57, J9.58, J9.59, J9.60, J9.61, J9.62, J9.63, J9.64, J9.77, J9.78, J9.79, J9.80
Other:
- moved on the sheet: H1, H2, H3, H4, J1
