File: 4-MPPC_FARICH_Prototype/4-MPPC_FARICH_Prototype.kicad_sch (KiCad schematic)
At the start: 21 parts, among them J1 1778764, J10 ST4-40-1.00-L-D-P-TR, J11 ST4-40-1.00-L-D-P-TR, J12 ST4-40-1.00-L-D-P-TR, J13 ST4-40-1.00-L-D-P-TR, J2 ST4-40-1.00-L-D-P-TR, J3 ST4-40-1.00-L-D-P-TR, J4 ST4-40-1.00-L-D-P-TR, J5 ST4-40-1.00-L-D-P-TR, J6 ST4-40-1.00-L-D-P-TR, J7 ST4-40-1.00-L-D-P-TR, J8 ST4-40-1.00-L-D-P-TR, J9 ST4-40-1.00-L-D-P-TR

Commit message: .
Connections:
- net +HV: now also MPPC1.129 (+HV), MPPC1.130 (+HV), MPPC1.131 (+HV), MPPC1.132 (+HV), MPPC1.133 (+HV), MPPC1.134 (+HV), MPPC1.135 (+HV), MPPC1.136 (+HV), MPPC1.137 (+HV), MPPC1.138 (+HV), MPPC1.139 (+HV), MPPC1.140 (+HV), MPPC1.141 (+HV), MPPC1.142 (+HV), MPPC1.143 (+HV), MPPC1.144 (+HV), MPPC1.145 (+HV), MPPC1.146 (+HV), MPPC1.147 (+HV), MPPC1.148 (+HV), MPPC1.149 (+HV), MPPC1.150 (+HV), MPPC1.151 (+HV), MPPC1.152 (+HV), MPPC1.153 (+HV), MPPC1.154 (+HV), MPPC1.155 (+HV), MPPC1.156 (+HV), MPPC1.157 (+HV), MPPC1.158 (+HV), MPPC1.159 (+HV), MPPC1.160 (+HV), MPPC1.161 (+HV), MPPC1.162 (+HV), MPPC2.129 (+HV), MPPC2.130 (+HV), MPPC2.131 (+HV), MPPC2.132 (+HV), MPPC2.133 (+HV), MPPC2.134 (+HV), MPPC2.135 (+HV), MPPC2.136 (+HV), MPPC2.137 (+HV), MPPC2.138 (+HV), MPPC2.139 (+HV), MPPC2.140 (+HV), MPPC2.141 (+HV), MPPC2.142 (+HV), MPPC2.143 (+HV), MPPC2.144 (+HV), MPPC2.145 (+HV), MPPC2.146 (+HV), MPPC2.147 (+HV), MPPC2.148 (+HV), MPPC2.149 (+HV), MPPC2.150 (+HV), MPPC2.151 (+HV), MPPC2.152 (+HV), MPPC2.153 (+HV), MPPC2.154 (+HV), MPPC2.155 (+HV), MPPC2.156 (+HV), MPPC2.157 (+HV), MPPC2.158 (+HV), MPPC2.159 (+HV), MPPC2.160 (+HV), MPPC2.161 (+HV), MPPC2.162 (+HV), MPPC3.129 (+HV), MPPC3.130 (+HV), MPPC3.131 (+HV), MPPC3.132 (+HV), MPPC3.133 (+HV), MPPC3.134 (+HV), MPPC3.135 (+HV), MPPC3.136 (+HV), MPPC3.137 (+HV), MPPC3.138 (+HV), MPPC3.139 (+HV), MPPC3.140 (+HV), MPPC3.141 (+HV), MPPC3.142 (+HV), MPPC3.143 (+HV), MPPC3.144 (+HV), MPPC3.145 (+HV), MPPC3.146 (+HV), MPPC3.147 (+HV), MPPC3.148 (+HV), MPPC3.149 (+HV), MPPC3.150 (+HV), MPPC3.151 (+HV), MPPC3.152 (+HV), MPPC3.153 (+HV), MPPC3.154 (+HV), MPPC3.155 (+HV), MPPC3.156 (+HV), MPPC3.157 (+HV), MPPC3.158 (+HV), MPPC3.159 (+HV), MPPC3.160 (+HV), MPPC3.161 (+HV), MPPC3.162 (+HV), MPPC4.129 (+HV), MPPC4.130 (+HV), MPPC4.131 (+HV), MPPC4.132 (+HV), MPPC4.133 (+HV), MPPC4.134 (+HV), MPPC4.135 (+HV), MPPC4.136 (+HV), MPPC4.137 (+HV), MPPC4.138 (+HV), MPPC4.139 (+HV), MPPC4.140 (+HV), MPPC4.141 (+HV), MPPC4.142 (+HV), MPPC4.143 (+HV), MPPC4.144 (+HV), MPPC4.145 (+HV), MPPC4.146 (+HV), MPPC4.147 (+HV), MPPC4.148 (+HV), MPPC4.149 (+HV), MPPC4.150 (+HV), MPPC4.151 (+HV), MPPC4.152 (+HV), MPPC4.153 (+HV), MPPC4.154 (+HV), MPPC4.155 (+HV), MPPC4.156 (+HV), MPPC4.157 (+HV), MPPC4.158 (+HV), MPPC4.159 (+HV), MPPC4.160 (+HV), MPPC4.161 (+HV), MPPC4.162 (+HV)
- net Cube_1_A-E1: now also MPPC1.5 (SignalOut), MPPC1.6 (SignalOut)
- net Cube_1_A-E2: now also MPPC1.10 (SignalOut), MPPC1.9 (SignalOut)
- net Cube_1_A-E3: now also MPPC1.21 (SignalOut), MPPC1.22 (SignalOut)
- net Cube_1_A-E4: now also MPPC1.25 (SignalOut), MPPC1.26 (SignalOut)
- net Cube_1_A-E5: now also MPPC1.37 (SignalOut), MPPC1.38 (SignalOut)
- net Cube_1_A-E6: now also MPPC1.41 (SignalOut), MPPC1.42 (SignalOut)
- net Cube_1_A-E7: now also MPPC1.53 (SignalOut), MPPC1.54 (SignalOut)
- net Cube_1_A-E8: now also MPPC1.57 (SignalOut), MPPC1.58 (SignalOut)
- net Cube_1_A-F1: now also MPPC1.1 (SignalOut), MPPC1.2 (SignalOut)
- net Cube_1_A-F2: now also MPPC1.13 (SignalOut), MPPC1.14 (SignalOut)
- net Cube_1_A-F3: now also MPPC1.17 (SignalOut), MPPC1.18 (SignalOut)
- net Cube_1_A-F4: now also MPPC1.29 (SignalOut), MPPC1.30 (SignalOut)
- net Cube_1_A-F5: now also MPPC1.33 (SignalOut), MPPC1.34 (SignalOut)
- net Cube_1_A-F6: now also MPPC1.45 (SignalOut), MPPC1.46 (SignalOut)
- net Cube_1_A-F7: now also MPPC1.49 (SignalOut), MPPC1.50 (SignalOut)
- net Cube_1_A-F8: now also MPPC1.61 (SignalOut), MPPC1.62 (SignalOut)
- net Cube_1_A-G1: now also MPPC1.65 (SignalOut), MPPC1.66 (SignalOut)
- net Cube_1_A-G2: now also MPPC1.77 (SignalOut), MPPC1.78 (SignalOut)
- net Cube_1_A-G3: now also MPPC1.81 (SignalOut), MPPC1.82 (SignalOut)
- net Cube_1_A-G4: now also MPPC1.93 (SignalOut), MPPC1.94 (SignalOut)
- net Cube_1_A-G5: now also MPPC1.97 (SignalOut), MPPC1.98 (SignalOut)
- net Cube_1_A-G6: now also MPPC1.109 (SignalOut), MPPC1.110 (SignalOut)
- net Cube_1_A-G7: now also MPPC1.113 (SignalOut), MPPC1.114 (SignalOut)
- net Cube_1_A-G8: now also MPPC1.125 (SignalOut), MPPC1.126 (SignalOut)
- net Cube_1_A-H1: now also MPPC1.69 (SignalOut), MPPC1.70 (SignalOut)
- net Cube_1_A-H2: now also MPPC1.73 (SignalOut), MPPC1.74 (SignalOut)
- net Cube_1_A-H3: now also MPPC1.85 (SignalOut), MPPC1.86 (SignalOut)
- net Cube_1_A-H4: now also MPPC1.89 (SignalOut), MPPC1.90 (SignalOut)
- net Cube_1_A-H5: now also MPPC1.101 (SignalOut), MPPC1.102 (SignalOut)
- net Cube_1_A-H6: now also MPPC1.105 (SignalOut), MPPC1.106 (SignalOut)
- net Cube_1_A-H7: now also MPPC1.117 (SignalOut), MPPC1.118 (SignalOut)
- net Cube_1_A-H8: now also MPPC1.121 (SignalOut), MPPC1.122 (SignalOut)
- net Cube_2_A-G8: now reaches J4.07
- net Cube_2_A-G8: now also MPPC1.67 (SignalOut), MPPC1.68 (SignalOut)
- net Cube_2_A-F8: now reaches J4.08
- net Cube_2_A-F8: now also MPPC1.3 (SignalOut), MPPC1.4 (SignalOut)
- net Cube_2_A-H8: now reaches J4.09
- net Cube_2_A-H8: now also MPPC1.71 (SignalOut), MPPC1.72 (SignalOut)
- net Cube_2_A-E8: now reaches J4.10
- net Cube_2_A-E8: now also MPPC1.7 (SignalOut), MPPC1.8 (SignalOut)
- net Cube_2_A-H7: now reaches J4.11
- net Cube_2_A-H7: now also MPPC1.75 (SignalOut), MPPC1.76 (SignalOut)
- net Cube_2_A-E7: now reaches J4.12
- net Cube_2_A-E7: now also MPPC1.11 (SignalOut), MPPC1.12 (SignalOut)
- net Cube_2_A-G7: now reaches J4.13
- net Cube_2_A-G7: now also MPPC1.79 (SignalOut), MPPC1.80 (SignalOut)
- net Cube_2_A-F7: now reaches J4.14
- net Cube_2_A-F7: now also MPPC1.15 (SignalOut), MPPC1.16 (SignalOut)
- net Cube_2_A-G6: now reaches J4.27
- net Cube_2_A-G6: now also MPPC1.83 (SignalOut), MPPC1.84 (SignalOut)
- net Cube_2_A-F6: now reaches J4.28
- net Cube_2_A-F6: now also MPPC1.19 (SignalOut), MPPC1.20 (SignalOut)
- net Cube_2_A-H6: now reaches J4.29
- net Cube_2_A-H6: now also MPPC1.87 (SignalOut), MPPC1.88 (SignalOut)
- net Cube_2_A-E6: now reaches J4.30
- net Cube_2_A-E6: now also MPPC1.23 (SignalOut), MPPC1.24 (SignalOut)
- net Cube_2_A-H5: now reaches J4.31
- net Cube_2_A-H5: now also MPPC1.91 (SignalOut), MPPC1.92 (SignalOut)
- net Cube_2_A-E5: now reaches J4.32
- net Cube_2_A-E5: now also MPPC1.27 (SignalOut), MPPC1.28 (SignalOut)
- net Cube_2_A-G5: now reaches J4.33
- net Cube_2_A-G5: now also MPPC1.95 (SignalOut), MPPC1.96 (SignalOut)
- net Cube_2_A-F5: now reaches J4.34
- net Cube_2_A-F5: now also MPPC1.31 (SignalOut), MPPC1.32 (SignalOut)
- net Cube_2_A-G4: now reaches J4.47
- net Cube_2_A-G4: now also MPPC1.100 (SignalOut), MPPC1.99 (SignalOut)
- net Cube_2_A-F4: now reaches J4.48
- net Cube_2_A-F4: now also MPPC1.35 (SignalOut), MPPC1.36 (SignalOut)
- net Cube_2_A-H4: now reaches J4.49
- net Cube_2_A-H4: now also MPPC1.103 (SignalOut), MPPC1.104 (SignalOut)
- net Cube_2_A-E4: now reaches J4.50
- net Cube_2_A-E4: now also MPPC1.39 (SignalOut), MPPC1.40 (SignalOut)
- net Cube_2_A-H3: now reaches J4.51
- net Cube_2_A-H3: now also MPPC1.107 (SignalOut), MPPC1.108 (SignalOut)
- net Cube_2_A-E3: now reaches J4.52
- net Cube_2_A-E3: now also MPPC1.43 (SignalOut), MPPC1.44 (SignalOut)
- net Cube_2_A-G3: now reaches J4.53
- net Cube_2_A-G3: now also MPPC1.111 (SignalOut), MPPC1.112 (SignalOut)
- net Cube_2_A-F3: now reaches J4.54
- net Cube_2_A-F3: now also MPPC1.47 (SignalOut), MPPC1.48 (SignalOut)
- net Cube_2_A-G2: now reaches J4.67
- net Cube_2_A-G2: now also MPPC1.115 (SignalOut), MPPC1.116 (SignalOut)
- net Cube_2_A-F2: now reaches J4.68
- net Cube_2_A-F2: now also MPPC1.51 (SignalOut), MPPC1.52 (SignalOut)
- net Cube_2_A-H2: now reaches J4.69
- net Cube_2_A-H2: now also MPPC1.119 (SignalOut), MPPC1.120 (SignalOut)
- net Cube_2_A-E2: now reaches J4.70
- net Cube_2_A-E2: now also MPPC1.55 (SignalOut), MPPC1.56 (SignalOut)
- net Cube_2_A-H1: now reaches J4.71
- net Cube_2_A-H1: now also MPPC1.123 (SignalOut), MPPC1.124 (SignalOut)
- net Cube_2_A-E1: now reaches J4.72
- net Cube_2_A-E1: now also MPPC1.59 (SignalOut), MPPC1.60 (SignalOut)
- net Cube_2_A-G1: now reaches J4.73
- net Cube_2_A-G1: now also MPPC1.127 (SignalOut), MPPC1.128 (SignalOut)
- net Cube_2_A-F1: now reaches J4.74
- net Cube_2_A-F1: now also MPPC1.63 (SignalOut), MPPC1.64 (SignalOut)

Commit message: .
Parts:
- removed J10, J11, J12, J13: ST4-40-1.00-L-D-P-TR, FARICH:SAMTEC_ST4-40-1.00-L-D-P-TR, symbol FARICH:ST4-40-1.00-L-D-P-TR
- renumbered J8 to J7, J7 to J8
Connections:
- net Cube_1_A-A1: now also J3.72, MPPC2.5 (SignalOut), MPPC2.6 (SignalOut); no longer J3.09
- net Cube_1_A-A2: now also J3.70, MPPC2.10 (SignalOut), MPPC2.9 (SignalOut); no longer J3.11
- net Cube_1_A-A3: now also J3.52, MPPC2.21 (SignalOut), MPPC2.22 (SignalOut); no longer J3.29
- net Cube_1_A-A4: now also J3.50, MPPC2.25 (SignalOut), MPPC2.26 (SignalOut); no longer J3.31
- net Cube_1_A-A5: now also J3.32, MPPC2.37 (SignalOut), MPPC2.38 (SignalOut); no longer J3.49
- net Cube_1_A-A6: now also J3.30, MPPC2.41 (SignalOut), MPPC2.42 (SignalOut); no longer J3.51
- net Cube_1_A-A7: now also J3.12, MPPC2.53 (SignalOut), MPPC2.54 (SignalOut); no longer J3.69
- net Cube_1_A-A8: now also J3.10, MPPC2.57 (SignalOut), MPPC2.58 (SignalOut); no longer J3.71
- net Cube_1_A-B1: now also J3.74, MPPC2.1 (SignalOut), MPPC2.2 (SignalOut); no longer J3.07
- net Cube_1_A-B2: now also J3.68, MPPC2.13 (SignalOut), MPPC2.14 (SignalOut); no longer J3.13
- net Cube_1_A-B3: now also J3.54, MPPC2.17 (SignalOut), MPPC2.18 (SignalOut); no longer J3.27
- net Cube_1_A-B4: now also J3.48, MPPC2.29 (SignalOut), MPPC2.30 (SignalOut); no longer J3.33
- net Cube_1_A-B5: now also J3.34, MPPC2.33 (SignalOut), MPPC2.34 (SignalOut); no longer J3.47
- net Cube_1_A-B6: now also J3.28, MPPC2.45 (SignalOut), MPPC2.46 (SignalOut); no longer J3.53
- net Cube_1_A-B7: now also J3.14, MPPC2.49 (SignalOut), MPPC2.50 (SignalOut); no longer J3.67
- net Cube_1_A-B8: now also J3.08, MPPC2.61 (SignalOut), MPPC2.62 (SignalOut); no longer J3.73
- net Cube_1_A-C1: now also J3.73, MPPC2.65 (SignalOut), MPPC2.66 (SignalOut); no longer J3.08
- net Cube_1_A-C2: now also J3.67, MPPC2.77 (SignalOut), MPPC2.78 (SignalOut); no longer J3.14
- net Cube_1_A-C3: now also J3.53, MPPC2.81 (SignalOut), MPPC2.82 (SignalOut); no longer J3.28
- net Cube_1_A-C4: now also J3.47, MPPC2.93 (SignalOut), MPPC2.94 (SignalOut); no longer J3.34
- net Cube_1_A-C5: now also J3.33, MPPC2.97 (SignalOut), MPPC2.98 (SignalOut); no longer J3.48
- net Cube_1_A-C6: now also J3.27, MPPC2.109 (SignalOut), MPPC2.110 (SignalOut); no longer J3.54
- net Cube_1_A-C7: now also J3.13, MPPC2.113 (SignalOut), MPPC2.114 (SignalOut); no longer J3.68
- net Cube_1_A-C8: now also J3.07, MPPC2.125 (SignalOut), MPPC2.126 (SignalOut); no longer J3.74
- net Cube_1_A-D1: now also J3.71, MPPC2.69 (SignalOut), MPPC2.70 (SignalOut); no longer J3.10
- net Cube_1_A-D2: now also J3.69, MPPC2.73 (SignalOut), MPPC2.74 (SignalOut); no longer J3.12
- net Cube_1_A-D3: now also J3.51, MPPC2.85 (SignalOut), MPPC2.86 (SignalOut); no longer J3.30
- net Cube_1_A-D4: now also J3.49, MPPC2.89 (SignalOut), MPPC2.90 (SignalOut); no longer J3.32
- net Cube_1_A-D5: now also J3.31, MPPC2.101 (SignalOut), MPPC2.102 (SignalOut); no longer J3.50
- net Cube_1_A-D6: now also J3.29, MPPC2.105 (SignalOut), MPPC2.106 (SignalOut); no longer J3.52
- net Cube_1_A-D7: now also J3.11, MPPC2.117 (SignalOut), MPPC2.118 (SignalOut); no longer J3.70
- net Cube_1_A-D8: now also J3.09, MPPC2.121 (SignalOut), MPPC2.122 (SignalOut); no longer J3.72
- net Cube_4_A-C8: now reaches J9.07
- net Cube_4_A-C8: now also MPPC4.127 (SignalOut), MPPC4.128 (SignalOut)
- net Cube_4_A-B8: now reaches J9.08
- net Cube_4_A-B8: now also MPPC4.63 (SignalOut), MPPC4.64 (SignalOut)
- net Cube_4_A-D8: now reaches J9.09
- net Cube_4_A-D8: now also MPPC4.123 (SignalOut), MPPC4.124 (SignalOut)
- net Cube_4_A-A8: now reaches J9.10
- net Cube_4_A-A8: now also MPPC4.59 (SignalOut), MPPC4.60 (SignalOut)
- net Cube_4_A-D7: now reaches J9.11
- net Cube_4_A-D7: now also MPPC4.119 (SignalOut), MPPC4.120 (SignalOut)
- net Cube_4_A-A7: now reaches J9.12
- net Cube_4_A-A7: now also MPPC4.55 (SignalOut), MPPC4.56 (SignalOut)
- net Cube_4_A-C7: now reaches J9.13
- net Cube_4_A-C7: now also MPPC4.115 (SignalOut), MPPC4.116 (SignalOut)
- net Cube_4_A-B7: now reaches J9.14
- net Cube_4_A-B7: now also MPPC4.51 (SignalOut), MPPC4.52 (SignalOut)
- net Cube_4_A-C6: now reaches J9.27
- net Cube_4_A-C6: now also MPPC4.111 (SignalOut), MPPC4.112 (SignalOut)
- net Cube_4_A-B6: now reaches J9.28
- net Cube_4_A-B6: now also MPPC4.47 (SignalOut), MPPC4.48 (SignalOut)
- net Cube_4_A-D6: now reaches J9.29
- net Cube_4_A-D6: now also MPPC4.107 (SignalOut), MPPC4.108 (SignalOut)
- net Cube_4_A-A6: now reaches J9.30
- net Cube_4_A-A6: now also MPPC4.43 (SignalOut), MPPC4.44 (SignalOut)
- net Cube_4_A-D5: now reaches J9.31
- net Cube_4_A-D5: now also MPPC4.103 (SignalOut), MPPC4.104 (SignalOut)
- net Cube_4_A-A5: now reaches J9.32
- net Cube_4_A-A5: now also MPPC4.39 (SignalOut), MPPC4.40 (SignalOut)
- net Cube_4_A-C5: now reaches J9.33
- net Cube_4_A-C5: now also MPPC4.100 (SignalOut), MPPC4.99 (SignalOut)
- net Cube_4_A-B5: now reaches J9.34
- net Cube_4_A-B5: now also MPPC4.35 (SignalOut), MPPC4.36 (SignalOut)
- net Cube_4_A-C4: now reaches J9.47
- net Cube_4_A-C4: now also MPPC4.95 (SignalOut), MPPC4.96 (SignalOut)
- net Cube_4_A-B4: now reaches J9.48
- net Cube_4_A-B4: now also MPPC4.31 (SignalOut), MPPC4.32 (SignalOut)
- net Cube_4_A-D4: now reaches J9.49
- net Cube_4_A-D4: now also MPPC4.91 (SignalOut), MPPC4.92 (SignalOut)
- net Cube_4_A-A4: now reaches J9.50
- net Cube_4_A-A4: now also MPPC4.27 (SignalOut), MPPC4.28 (SignalOut)
- net Cube_4_A-D3: now reaches J9.51
- net Cube_4_A-D3: now also MPPC4.87 (SignalOut), MPPC4.88 (SignalOut)
- net Cube_4_A-A3: now reaches J9.52
- net Cube_4_A-A3: now also MPPC4.23 (SignalOut), MPPC4.24 (SignalOut)
- net Cube_4_A-C3: now reaches J9.53
- net Cube_4_A-C3: now also MPPC4.83 (SignalOut), MPPC4.84 (SignalOut)
- net Cube_4_A-B3: now reaches J9.54
- net Cube_4_A-B3: now also MPPC4.19 (SignalOut), MPPC4.20 (SignalOut)
- net Cube_4_A-C2: now reaches J9.67
- net Cube_4_A-C2: now also MPPC4.79 (SignalOut), MPPC4.80 (SignalOut)
- net Cube_4_A-B2: now reaches J9.68
- net Cube_4_A-B2: now also MPPC4.15 (SignalOut), MPPC4.16 (SignalOut)
- net Cube_4_A-D2: now reaches J9.69
- net Cube_4_A-D2: now also MPPC4.75 (SignalOut), MPPC4.76 (SignalOut)
- net Cube_4_A-A2: now reaches J9.70
- net Cube_4_A-A2: now also MPPC4.11 (SignalOut), MPPC4.12 (SignalOut)
- net Cube_4_A-D1: now reaches J9.71
- net Cube_4_A-D1: now also MPPC4.71 (SignalOut), MPPC4.72 (SignalOut)
- net Cube_4_A-A1: now reaches J9.72
- net Cube_4_A-A1: now also MPPC4.7 (SignalOut), MPPC4.8 (SignalOut)
- net Cube_4_A-C1: now reaches J9.73
- net Cube_4_A-C1: now also MPPC4.67 (SignalOut), MPPC4.68 (SignalOut)
- net Cube_4_A-B1: now reaches J9.74
- net Cube_4_A-B1: now also MPPC4.3 (SignalOut), MPPC4.4 (SignalOut)
- net Cube_3_A-F8: now reaches MPPC3.1 (SignalOut)
- net Cube_3_A-F8: now also J6.08, MPPC3.2 (SignalOut)
- net Cube_3_A-E7: now reaches MPPC3.10 (SignalOut)
- net Cube_3_A-E7: now also J6.12, MPPC3.9 (SignalOut)
- net Cube_4_A-G4: now reaches MPPC3.100 (SignalOut)
- net Cube_4_A-G4: now also J7.47, MPPC3.99 (SignalOut)
- net Cube_3_A-H5: now reaches MPPC3.101 (SignalOut)
- net Cube_3_A-H5: now also J6.31, MPPC3.102 (SignalOut)
- net Cube_4_A-H4: now reaches MPPC3.103 (SignalOut)
- net Cube_4_A-H4: now also J7.49, MPPC3.104 (SignalOut)
- net Cube_3_A-H6: now reaches MPPC3.105 (SignalOut)
- net Cube_3_A-H6: now also J6.29, MPPC3.106 (SignalOut)
- net Cube_4_A-H3: now reaches MPPC3.107 (SignalOut)
- net Cube_4_A-H3: now also J7.51, MPPC3.108 (SignalOut)
- net Cube_3_A-G6: now reaches MPPC3.109 (SignalOut)
- net Cube_3_A-G6: now also J6.27, MPPC3.110 (SignalOut)
- net Cube_4_A-E2: now reaches MPPC3.11 (SignalOut)
- net Cube_4_A-E2: now also J7.70, MPPC3.12 (SignalOut)
- net Cube_4_A-G3: now reaches MPPC3.111 (SignalOut)
- net Cube_4_A-G3: now also J7.53, MPPC3.112 (SignalOut)
- net Cube_3_A-G7: now reaches MPPC3.113 (SignalOut)
- net Cube_3_A-G7: now also J6.13, MPPC3.114 (SignalOut)
- net Cube_4_A-G2: now reaches MPPC3.115 (SignalOut)
- net Cube_4_A-G2: now also J7.67, MPPC3.116 (SignalOut)
- net Cube_3_A-H7: now reaches MPPC3.117 (SignalOut)
- net Cube_3_A-H7: now also J6.11, MPPC3.118 (SignalOut)
- net Cube_4_A-H2: now reaches MPPC3.119 (SignalOut)
- net Cube_4_A-H2: now also J7.69, MPPC3.120 (SignalOut)
- net Cube_3_A-H8: now reaches MPPC3.121 (SignalOut)
- net Cube_3_A-H8: now also J6.09, MPPC3.122 (SignalOut)
- net Cube_4_A-H1: now reaches MPPC3.123 (SignalOut)
- net Cube_4_A-H1: now also J7.71, MPPC3.124 (SignalOut)
- net Cube_3_A-G8: now reaches MPPC3.125 (SignalOut)
- net Cube_3_A-G8: now also J6.07, MPPC3.126 (SignalOut)
- net Cube_4_A-G1: now reaches MPPC3.127 (SignalOut)
- net Cube_4_A-G1: now also J7.73, MPPC3.128 (SignalOut)
- net Cube_3_A-F7: now reaches MPPC3.13 (SignalOut)
- net Cube_3_A-F7: now also J6.14, MPPC3.14 (SignalOut)
- net Cube_4_A-F2: now reaches MPPC3.15 (SignalOut)
- net Cube_4_A-F2: now also J7.68, MPPC3.16 (SignalOut)
- net Cube_3_A-F6: now reaches MPPC3.17 (SignalOut)
- net Cube_3_A-F6: now also J6.28, MPPC3.18 (SignalOut)
- net Cube_4_A-F3: now reaches MPPC3.19 (SignalOut)
- net Cube_4_A-F3: now also J7.54, MPPC3.20 (SignalOut)
- net Cube_3_A-E6: now reaches MPPC3.21 (SignalOut)
- net Cube_3_A-E6: now also J6.30, MPPC3.22 (SignalOut)
- net Cube_4_A-E3: now reaches MPPC3.23 (SignalOut)
- net Cube_4_A-E3: now also J7.52, MPPC3.24 (SignalOut)
- net Cube_3_A-E5: now reaches MPPC3.25 (SignalOut)
- net Cube_3_A-E5: now also J6.32, MPPC3.26 (SignalOut)
- net Cube_4_A-E4: now reaches MPPC3.27 (SignalOut)
- net Cube_4_A-E4: now also J7.50, MPPC3.28 (SignalOut)
- net Cube_3_A-F5: now reaches MPPC3.29 (SignalOut)
- net Cube_3_A-F5: now also J6.34, MPPC3.30 (SignalOut)
- net Cube_4_A-F1: now reaches MPPC3.3 (SignalOut)
- net Cube_4_A-F1: now also J7.74, MPPC3.4 (SignalOut)
- net Cube_4_A-F4: now reaches MPPC3.31 (SignalOut)
- net Cube_4_A-F4: now also J7.48, MPPC3.32 (SignalOut)
- net Cube_3_A-F4: now reaches MPPC3.33 (SignalOut)
- net Cube_3_A-F4: now also J6.48, MPPC3.34 (SignalOut)
- net Cube_4_A-F5: now reaches MPPC3.35 (SignalOut)
- net Cube_4_A-F5: now also J7.34, MPPC3.36 (SignalOut)
- net Cube_3_A-E4: now reaches MPPC3.37 (SignalOut)
- net Cube_3_A-E4: now also J6.50, MPPC3.38 (SignalOut)
- net Cube_4_A-E5: now reaches MPPC3.39 (SignalOut)
- net Cube_4_A-E5: now also J7.32, MPPC3.40 (SignalOut)
- net Cube_3_A-E3: now reaches MPPC3.41 (SignalOut)
- net Cube_3_A-E3: now also J6.52, MPPC3.42 (SignalOut)
- net Cube_4_A-E6: now reaches MPPC3.43 (SignalOut)
- net Cube_4_A-E6: now also J7.30, MPPC3.44 (SignalOut)
- net Cube_3_A-F3: now reaches MPPC3.45 (SignalOut)
- net Cube_3_A-F3: now also J6.54, MPPC3.46 (SignalOut)
- net Cube_4_A-F6: now reaches MPPC3.47 (SignalOut)
- net Cube_4_A-F6: now also J7.28, MPPC3.48 (SignalOut)
- net Cube_3_A-F2: now reaches MPPC3.49 (SignalOut)
- net Cube_3_A-F2: now also J6.68, MPPC3.50 (SignalOut)
- net Cube_3_A-E8: now reaches MPPC3.5 (SignalOut)
- net Cube_3_A-E8: now also J6.10, MPPC3.6 (SignalOut)
- net Cube_4_A-F7: now reaches MPPC3.51 (SignalOut)
- net Cube_4_A-F7: now also J7.14, MPPC3.52 (SignalOut)
- net Cube_3_A-E2: now reaches MPPC3.53 (SignalOut)
- net Cube_3_A-E2: now also J6.70, MPPC3.54 (SignalOut)
- net Cube_4_A-E7: now reaches MPPC3.55 (SignalOut)
- net Cube_4_A-E7: now also J7.12, MPPC3.56 (SignalOut)
- net Cube_3_A-E1: now reaches MPPC3.57 (SignalOut)
- net Cube_3_A-E1: now also J6.72, MPPC3.58 (SignalOut)
- net Cube_4_A-E8: now reaches MPPC3.59 (SignalOut)
- net Cube_4_A-E8: now also J7.10, MPPC3.60 (SignalOut)
- net Cube_3_A-F1: now reaches MPPC3.61 (SignalOut)
- net Cube_3_A-F1: now also J6.74, MPPC3.62 (SignalOut)
- net Cube_4_A-F8: now reaches MPPC3.63 (SignalOut)
- net Cube_4_A-F8: now also J7.08, MPPC3.64 (SignalOut)
- net Cube_3_A-G1: now reaches MPPC3.65 (SignalOut)
- net Cube_3_A-G1: now also J6.73, MPPC3.66 (SignalOut)
- net Cube_4_A-G8: now reaches MPPC3.67 (SignalOut)
- net Cube_4_A-G8: now also J7.07, MPPC3.68 (SignalOut)
- net Cube_3_A-H1: now reaches MPPC3.69 (SignalOut)
- net Cube_3_A-H1: now also J6.71, MPPC3.70 (SignalOut)
- net Cube_4_A-E1: now reaches MPPC3.7 (SignalOut)
- net Cube_4_A-E1: now also J7.72, MPPC3.8 (SignalOut)
- net Cube_4_A-H8: now reaches MPPC3.71 (SignalOut)
- net Cube_4_A-H8: now also J7.09, MPPC3.72 (SignalOut)
- net Cube_3_A-H2: now reaches MPPC3.73 (SignalOut)
- net Cube_3_A-H2: now also J6.69, MPPC3.74 (SignalOut)
- net Cube_4_A-H7: now reaches MPPC3.75 (SignalOut)
- net Cube_4_A-H7: now also J7.11, MPPC3.76 (SignalOut)
- net Cube_3_A-G2: now reaches MPPC3.77 (SignalOut)
- net Cube_3_A-G2: now also J6.67, MPPC3.78 (SignalOut)
- net Cube_4_A-G7: now reaches MPPC3.79 (SignalOut)
- net Cube_4_A-G7: now also J7.13, MPPC3.80 (SignalOut)
- net Cube_3_A-G3: now reaches MPPC3.81 (SignalOut)
- net Cube_3_A-G3: now also J6.53, MPPC3.82 (SignalOut)
- net Cube_4_A-G6: now reaches MPPC3.83 (SignalOut)
- net Cube_4_A-G6: now also J7.27, MPPC3.84 (SignalOut)
- net Cube_3_A-H3: now reaches MPPC3.85 (SignalOut)
- net Cube_3_A-H3: now also J6.51, MPPC3.86 (SignalOut)
- net Cube_4_A-H6: now reaches MPPC3.87 (SignalOut)
- net Cube_4_A-H6: now also J7.29, MPPC3.88 (SignalOut)
- net Cube_3_A-H4: now reaches MPPC3.89 (SignalOut)
- net Cube_3_A-H4: now also J6.49, MPPC3.90 (SignalOut)
- net Cube_4_A-H5: now reaches MPPC3.91 (SignalOut)
- net Cube_4_A-H5: now also J7.31, MPPC3.92 (SignalOut)
- net Cube_3_A-G4: now reaches MPPC3.93 (SignalOut)
- net Cube_3_A-G4: now also J6.47, MPPC3.94 (SignalOut)
- net Cube_4_A-G5: now reaches MPPC3.95 (SignalOut)
- net Cube_4_A-G5: now also J7.33, MPPC3.96 (SignalOut)
- net Cube_3_A-G5: now reaches MPPC3.97 (SignalOut)
- net Cube_3_A-G5: now also J6.33, MPPC3.98 (SignalOut)
- net Cube_2_A-C8: now reaches J5.07
- net Cube_2_A-C8: now also MPPC2.67 (SignalOut), MPPC2.68 (SignalOut)
- net Cube_2_A-B8: now reaches J5.08
- net Cube_2_A-B8: now also MPPC2.3 (SignalOut), MPPC2.4 (SignalOut)
- net Cube_2_A-D8: now reaches J5.09
- net Cube_2_A-D8: now also MPPC2.71 (SignalOut), MPPC2.72 (SignalOut)
- net Cube_2_A-A8: now reaches J5.10
- net Cube_2_A-A8: now also MPPC2.7 (SignalOut), MPPC2.8 (SignalOut)
- net Cube_2_A-D7: now reaches J5.11
- net Cube_2_A-D7: now also MPPC2.75 (SignalOut), MPPC2.76 (SignalOut)
- net Cube_2_A-A7: now reaches J5.12
- net Cube_2_A-A7: now also MPPC2.11 (SignalOut), MPPC2.12 (SignalOut)
- net Cube_2_A-C7: now reaches J5.13
- net Cube_2_A-C7: now also MPPC2.79 (SignalOut), MPPC2.80 (SignalOut)
- net Cube_2_A-B7: now reaches J5.14
- net Cube_2_A-B7: now also MPPC2.15 (SignalOut), MPPC2.16 (SignalOut)
- net Cube_2_A-C6: now reaches J5.27
- net Cube_2_A-C6: now also MPPC2.83 (SignalOut), MPPC2.84 (SignalOut)
- net Cube_2_A-B6: now reaches J5.28
- net Cube_2_A-B6: now also MPPC2.19 (SignalOut), MPPC2.20 (SignalOut)
- net Cube_2_A-D6: now reaches J5.29
- net Cube_2_A-D6: now also MPPC2.87 (SignalOut), MPPC2.88 (SignalOut)
- net Cube_2_A-A6: now reaches J5.30
- net Cube_2_A-A6: now also MPPC2.23 (SignalOut), MPPC2.24 (SignalOut)
- net Cube_2_A-D5: now reaches J5.31
- net Cube_2_A-D5: now also MPPC2.91 (SignalOut), MPPC2.92 (SignalOut)
- net Cube_2_A-A5: now reaches J5.32
- net Cube_2_A-A5: now also MPPC2.27 (SignalOut), MPPC2.28 (SignalOut)
- net Cube_2_A-C5: now reaches J5.33
- net Cube_2_A-C5: now also MPPC2.95 (SignalOut), MPPC2.96 (SignalOut)
- net Cube_2_A-B5: now reaches J5.34
- net Cube_2_A-B5: now also MPPC2.31 (SignalOut), MPPC2.32 (SignalOut)
- net Cube_2_A-C4: now reaches J5.47
- net Cube_2_A-C4: now also MPPC2.100 (SignalOut), MPPC2.99 (SignalOut)
- net Cube_2_A-B4: now reaches J5.48
- net Cube_2_A-B4: now also MPPC2.35 (SignalOut), MPPC2.36 (SignalOut)
- net Cube_2_A-D4: now reaches J5.49
- net Cube_2_A-D4: now also MPPC2.103 (SignalOut), MPPC2.104 (SignalOut)
- net Cube_2_A-A4: now reaches J5.50
- net Cube_2_A-A4: now also MPPC2.39 (SignalOut), MPPC2.40 (SignalOut)
- net Cube_2_A-D3: now reaches J5.51
- net Cube_2_A-D3: now also MPPC2.107 (SignalOut), MPPC2.108 (SignalOut)
- net Cube_2_A-A3: now reaches J5.52
- net Cube_2_A-A3: now also MPPC2.43 (SignalOut), MPPC2.44 (SignalOut)
- net Cube_2_A-C3: now reaches J5.53
- net Cube_2_A-C3: now also MPPC2.111 (SignalOut), MPPC2.112 (SignalOut)
- net Cube_2_A-B3: now reaches J5.54
- net Cube_2_A-B3: now also MPPC2.47 (SignalOut), MPPC2.48 (SignalOut)
- net Cube_2_A-C2: now reaches J5.67
- net Cube_2_A-C2: now also MPPC2.115 (SignalOut), MPPC2.116 (SignalOut)
- net Cube_2_A-B2: now reaches J5.68
- net Cube_2_A-B2: now also MPPC2.51 (SignalOut), MPPC2.52 (SignalOut)
- net Cube_2_A-D2: now reaches J5.69
- net Cube_2_A-D2: now also MPPC2.119 (SignalOut), MPPC2.120 (SignalOut)
- net Cube_2_A-A2: now reaches J5.70
- net Cube_2_A-A2: now also MPPC2.55 (SignalOut), MPPC2.56 (SignalOut)
- net Cube_2_A-D1: now reaches J5.71
- net Cube_2_A-D1: now also MPPC2.123 (SignalOut), MPPC2.124 (SignalOut)
- net Cube_2_A-A1: now reaches J5.72
- net Cube_2_A-A1: now also MPPC2.59 (SignalOut), MPPC2.60 (SignalOut)
- net Cube_2_A-C1: now reaches J5.73
- net Cube_2_A-C1: now also MPPC2.127 (SignalOut), MPPC2.128 (SignalOut)
- net Cube_2_A-B1: now reaches J5.74
- net Cube_2_A-B1: now also MPPC2.63 (SignalOut), MPPC2.64 (SignalOut)
- net Cube_3_A-B8: now reaches MPPC4.1 (SignalOut)
- net Cube_3_A-B8: now also J8.08, MPPC4.2 (SignalOut)
- net Cube_3_A-A7: now reaches MPPC4.10 (SignalOut)
- net Cube_3_A-A7: now also J8.12, MPPC4.9 (SignalOut)
- net Cube_3_A-D4: now reaches MPPC4.101 (SignalOut)
- net Cube_3_A-D4: now also J8.49, MPPC4.102 (SignalOut)
- net Cube_3_A-D3: now reaches MPPC4.105 (SignalOut)
- net Cube_3_A-D3: now also J8.51, MPPC4.106 (SignalOut)
- net Cube_3_A-C3: now reaches MPPC4.109 (SignalOut)
- net Cube_3_A-C3: now also J8.53, MPPC4.110 (SignalOut)
- net Cube_3_A-C2: now reaches MPPC4.113 (SignalOut)
- net Cube_3_A-C2: now also J8.67, MPPC4.114 (SignalOut)
- net Cube_3_A-D2: now reaches MPPC4.117 (SignalOut)
- net Cube_3_A-D2: now also J8.69, MPPC4.118 (SignalOut)
- net Cube_3_A-D1: now reaches MPPC4.121 (SignalOut)
- net Cube_3_A-D1: now also J8.71, MPPC4.122 (SignalOut)
- net Cube_3_A-C1: now reaches MPPC4.125 (SignalOut)
- net Cube_3_A-C1: now also J8.73, MPPC4.126 (SignalOut)
- net Cube_3_A-B7: now reaches MPPC4.13 (SignalOut)
- net Cube_3_A-B7: now also J8.14, MPPC4.14 (SignalOut)
- net Cube_3_A-B6: now reaches MPPC4.17 (SignalOut)
- net Cube_3_A-B6: now also J8.28, MPPC4.18 (SignalOut)
- net Cube_3_A-A6: now reaches MPPC4.21 (SignalOut)
- net Cube_3_A-A6: now also J8.30, MPPC4.22 (SignalOut)
- net Cube_3_A-A5: now reaches MPPC4.25 (SignalOut)
- net Cube_3_A-A5: now also J8.32, MPPC4.26 (SignalOut)
- net Cube_3_A-B5: now reaches MPPC4.29 (SignalOut)
- net Cube_3_A-B5: now also J8.34, MPPC4.30 (SignalOut)
- net Cube_3_A-B4: now reaches MPPC4.33 (SignalOut)
- net Cube_3_A-B4: now also J8.48, MPPC4.34 (SignalOut)
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Other:
- note removed: "Cube_5"
- note removed: "Cube_6"
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
Commit message: .
Parts:
- added C1, C2, C3, C4, C5, C6, C7, C8: 0.1uF, Capacitor_SMD:C_0603_1608Metric_Pad1.08x0.95mm_HandSolder, symbol Device:C
- added R1, R2, R3, R4, R5, R6, R7, R8: 1k, Resistor_SMD:R_0603_1608Metric_Pad0.98x0.95mm_HandSolder, symbol Device:R
Connections:
- net +HV: now also R1.2, R2.2, R3.2, R4.2, R5.2, R6.2, R7.2, R8.2; no longer MPPC1.129 (+HV), MPPC1.130 (+HV), MPPC1.131 (+HV), MPPC1.132 (+HV), MPPC1.133 (+HV), MPPC1.134 (+HV), MPPC1.135 (+HV), MPPC1.136 (+HV), MPPC1.137 (+HV), MPPC1.138 (+HV), MPPC1.139 (+HV), MPPC1.140 (+HV), MPPC1.141 (+HV), MPPC1.142 (+HV), MPPC1.143 (+HV), MPPC1.144 (+HV), MPPC1.145 (+HV), MPPC1.146 (+HV), MPPC1.147 (+HV), MPPC1.148 (+HV), MPPC1.149 (+HV), MPPC1.150 (+HV), MPPC1.151 (+HV), MPPC1.152 (+HV), MPPC1.153 (+HV), MPPC1.154 (+HV), MPPC1.155 (+HV), MPPC1.156 (+HV), MPPC1.157 (+HV), MPPC1.158 (+HV), MPPC1.159 (+HV), MPPC1.160 (+HV), MPPC1.161 (+HV), MPPC1.162 (+HV), MPPC2.129 (+HV), MPPC2.130 (+HV), MPPC2.131 (+HV), MPPC2.132 (+HV), MPPC2.133 (+HV), MPPC2.134 (+HV), MPPC2.135 (+HV), MPPC2.136 (+HV), MPPC2.137 (+HV), MPPC2.138 (+HV), MPPC2.139 (+HV), MPPC2.140 (+HV), MPPC2.141 (+HV), MPPC2.142 (+HV), MPPC2.143 (+HV), MPPC2.144 (+HV), MPPC2.145 (+HV), MPPC2.146 (+HV), MPPC2.147 (+HV), MPPC2.148 (+HV), MPPC2.149 (+HV), MPPC2.150 (+HV), MPPC2.151 (+HV), MPPC2.152 (+HV), MPPC2.153 (+HV), MPPC2.154 (+HV), MPPC2.155 (+HV), MPPC2.156 (+HV), MPPC2.157 (+HV), MPPC2.158 (+HV), MPPC2.159 (+HV), MPPC2.160 (+HV), MPPC2.161 (+HV), MPPC2.162 (+HV), MPPC3.129 (+HV), MPPC3.130 (+HV), MPPC3.131 (+HV), MPPC3.132 (+HV), MPPC3.133 (+HV), MPPC3.134 (+HV), MPPC3.135 (+HV), MPPC3.136 (+HV), MPPC3.137 (+HV), MPPC3.138 (+HV), MPPC3.139 (+HV), MPPC3.140 (+HV), MPPC3.141 (+HV), MPPC3.142 (+HV), MPPC3.143 (+HV), MPPC3.144 (+HV), MPPC3.145 (+HV), MPPC3.146 (+HV), MPPC3.147 (+HV), MPPC3.148 (+HV), MPPC3.149 (+HV), MPPC3.150 (+HV), MPPC3.151 (+HV), MPPC3.152 (+HV), MPPC3.153 (+HV), MPPC3.154 (+HV), MPPC3.155 (+HV), MPPC3.156 (+HV), MPPC3.157 (+HV), MPPC3.158 (+HV), MPPC3.159 (+HV), MPPC3.160 (+HV), MPPC3.161 (+HV), MPPC3.162 (+HV), MPPC4.129 (+HV), MPPC4.130 (+HV), MPPC4.131 (+HV), MPPC4.132 (+HV), MPPC4.133 (+HV), MPPC4.134 (+HV), MPPC4.135 (+HV), MPPC4.136 (+HV), MPPC4.137 (+HV), MPPC4.138 (+HV), MPPC4.139 (+HV), MPPC4.140 (+HV), MPPC4.141 (+HV), MPPC4.142 (+HV), MPPC4.143 (+HV), MPPC4.144 (+HV), MPPC4.145 (+HV), MPPC4.146 (+HV), MPPC4.147 (+HV), MPPC4.148 (+HV), MPPC4.149 (+HV), MPPC4.150 (+HV), MPPC4.151 (+HV), MPPC4.152 (+HV), MPPC4.153 (+HV), MPPC4.154 (+HV), MPPC4.155 (+HV), MPPC4.156 (+HV), MPPC4.157 (+HV), MPPC4.158 (+HV), MPPC4.159 (+HV), MPPC4.160 (+HV), MPPC4.161 (+HV), MPPC4.162 (+HV)
- net Cube_3_A-G1: no longer J6.73
- net Cube_3_A-G2: no longer J6.67
- net Cube_3_A-G3: no longer J6.53
- net Cube_3_A-G4: no longer J6.47
- net Cube_3_A-G5: no longer J6.33
- net Cube_3_A-G6: no longer J6.27
- net Cube_3_A-G7: no longer J6.13
- net Cube_3_A-G8: no longer J6.07
- net Cube_3_A-H1: no longer J6.71
- net Cube_3_A-H2: no longer J6.69
- net Cube_3_A-H3: no longer J6.51
- net Cube_3_A-H4: no longer J6.49
- net Cube_3_A-H5: no longer J6.31
- net Cube_3_A-H6: no longer J6.29
- net Cube_3_A-H7: no longer J6.11
- net Cube_3_A-H8: no longer J6.09
- net Cube_4_A-G1: now also J7.07; no longer J7.73
- net Cube_4_A-G2: now also J7.13; no longer J7.67
- net Cube_4_A-G3: now also J7.27; no longer J7.53
- net Cube_4_A-G4: now also J7.33; no longer J7.47
- net Cube_4_A-G5: now also J7.47; no longer J7.33
- net Cube_4_A-G6: now also J7.53; no longer J7.27
- net Cube_4_A-G7: now also J7.67; no longer J7.13
- net Cube_4_A-G8: now also J7.73; no longer J7.07
- net Cube_4_A-H1: now also J7.09; no longer J7.71
- net Cube_4_A-H2: now also J7.11; no longer J7.69
- net Cube_4_A-H3: now also J7.29; no longer J7.51
- net Cube_4_A-H4: now also J7.31; no longer J7.49
- net Cube_4_A-H5: now also J7.49; no longer J7.31
- net Cube_4_A-H6: now also J7.51; no longer J7.29
- net Cube_4_A-H7: now also J7.69; no longer J7.11
- net Cube_4_A-H8: now also J7.71; no longer J7.09
- net GND: now also C1.2, C2.2, C3.2, C4.2, C5.2, C6.2, C7.2, C8.2
- new net: C4.1, C8.1, MPPC4.129 (+HV), MPPC4.130 (+HV), MPPC4.131 (+HV), MPPC4.132 (+HV), MPPC4.133 (+HV), MPPC4.134 (+HV), MPPC4.135 (+HV), MPPC4.136 (+HV), MPPC4.137 (+HV), MPPC4.138 (+HV), MPPC4.139 (+HV), MPPC4.140 (+HV), MPPC4.141 (+HV), MPPC4.142 (+HV), MPPC4.143 (+HV), MPPC4.144 (+HV), MPPC4.145 (+HV), MPPC4.146 (+HV), MPPC4.147 (+HV), MPPC4.148 (+HV), MPPC4.149 (+HV), MPPC4.150 (+HV), MPPC4.151 (+HV), MPPC4.152 (+HV), MPPC4.153 (+HV), MPPC4.154 (+HV), MPPC4.155 (+HV), MPPC4.156 (+HV), MPPC4.157 (+HV), MPPC4.158 (+HV), MPPC4.159 (+HV), MPPC4.160 (+HV), MPPC4.161 (+HV), MPPC4.162 (+HV), R4.1, R8.1
- new net: C2.1, C6.1, MPPC2.129 (+HV), MPPC2.130 (+HV), MPPC2.131 (+HV), MPPC2.132 (+HV), MPPC2.133 (+HV), MPPC2.134 (+HV), MPPC2.135 (+HV), MPPC2.136 (+HV), MPPC2.137 (+HV), MPPC2.138 (+HV), MPPC2.139 (+HV), MPPC2.140 (+HV), MPPC2.141 (+HV), MPPC2.142 (+HV), MPPC2.143 (+HV), MPPC2.144 (+HV), MPPC2.145 (+HV), MPPC2.146 (+HV), MPPC2.147 (+HV), MPPC2.148 (+HV), MPPC2.149 (+HV), MPPC2.150 (+HV), MPPC2.151 (+HV), MPPC2.152 (+HV), MPPC2.153 (+HV), MPPC2.154 (+HV), MPPC2.155 (+HV), MPPC2.156 (+HV), MPPC2.157 (+HV), MPPC2.158 (+HV), MPPC2.159 (+HV), MPPC2.160 (+HV), MPPC2.161 (+HV), MPPC2.162 (+HV), R2.1, R6.1
- new net: C1.1, C5.1, MPPC1.129 (+HV), MPPC1.130 (+HV), MPPC1.131 (+HV), MPPC1.132 (+HV), MPPC1.133 (+HV), MPPC1.134 (+HV), MPPC1.135 (+HV), MPPC1.136 (+HV), MPPC1.137 (+HV), MPPC1.138 (+HV), MPPC1.139 (+HV), MPPC1.140 (+HV), MPPC1.141 (+HV), MPPC1.142 (+HV), MPPC1.143 (+HV), MPPC1.144 (+HV), MPPC1.145 (+HV), MPPC1.146 (+HV), MPPC1.147 (+HV), MPPC1.148 (+HV), MPPC1.149 (+HV), MPPC1.150 (+HV), MPPC1.151 (+HV), MPPC1.152 (+HV), MPPC1.153 (+HV), MPPC1.154 (+HV), MPPC1.155 (+HV), MPPC1.156 (+HV), MPPC1.157 (+HV), MPPC1.158 (+HV), MPPC1.159 (+HV), MPPC1.160 (+HV), MPPC1.161 (+HV), MPPC1.162 (+HV), R1.1, R5.1
- new net: C3.1, C7.1, MPPC3.129 (+HV), MPPC3.130 (+HV), MPPC3.131 (+HV), MPPC3.132 (+HV), MPPC3.133 (+HV), MPPC3.134 (+HV), MPPC3.135 (+HV), MPPC3.136 (+HV), MPPC3.137 (+HV), MPPC3.138 (+HV), MPPC3.139 (+HV), MPPC3.140 (+HV), MPPC3.141 (+HV), MPPC3.142 (+HV), MPPC3.143 (+HV), MPPC3.144 (+HV), MPPC3.145 (+HV), MPPC3.146 (+HV), MPPC3.147 (+HV), MPPC3.148 (+HV), MPPC3.149 (+HV), MPPC3.150 (+HV), MPPC3.151 (+HV), MPPC3.152 (+HV), MPPC3.153 (+HV), MPPC3.154 (+HV), MPPC3.155 (+HV), MPPC3.156 (+HV), MPPC3.157 (+HV), MPPC3.158 (+HV), MPPC3.159 (+HV), MPPC3.160 (+HV), MPPC3.161 (+HV), MPPC3.162 (+HV), R3.1, R7.1
Other:
- moved on the sheet: H1

Commit message: .
Connections:
- net Cube_3_A-G1: now also J6.07
- net Cube_3_A-G2: now also J6.13
- net Cube_3_A-G3: now also J6.27
- net Cube_3_A-G4: now also J6.33
- net Cube_3_A-G5: now also J6.47
- net Cube_3_A-G6: now also J6.53
- net Cube_3_A-G7: now also J6.67
- net Cube_3_A-G8: now also J6.73
- net Cube_3_A-H1: now also J6.09
- net Cube_3_A-H2: now also J6.11
- net Cube_3_A-H3: now also J6.29
- net Cube_3_A-H4: now also J6.31
- net Cube_3_A-H5: now also J6.49
- net Cube_3_A-H6: now also J6.51
- net Cube_3_A-H7: now also J6.69
- net Cube_3_A-H8: now also J6.71
Changed lines of the file:
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@@
 	(global_label "Cube_3_A-H4"
 		(shape input)
-		(at 232.41 320.04 180)
+		(at 237.49 320.04 180)
 		(fields_autoplaced yes)
 		(effects
@@
 		)
 		(property "Intersheetrefs" "${INTERSHEET_REFS}"
-			(at 216.4225 320.04 0)
+			(at 221.5025 320.04 0)
 			(effects
 				(font
@@
 	(global_label "Cube_3_A-H7"
 		(shape input)
-		(at 232.41 368.3 180)
+		(at 237.49 368.3 180)
 		(fields_autoplaced yes)
 		(effects
@@
 		)
 		(property "Intersheetrefs" "${INTERSHEET_REFS}"
-			(at 216.4225 368.3 0)
+			(at 221.5025 368.3 0)
 			(effects
 				(font
@@
 	(global_label "Cube_3_A-H8"
 		(shape input)
-		(at 232.41 370.84 180)
+		(at 237.49 370.84 180)
 		(fields_autoplaced yes)
 		(effects
@@
 		)
 		(property "Intersheetrefs" "${INTERSHEET_REFS}"
-			(at 216.4225 370.84 0)
+			(at 221.5025 370.84 0)
 			(effects
 				(font
@@
 	(global_label "Cube_3_A-H2"
 		(shape input)
-		(at 232.41 294.64 180)
+		(at 237.49 294.64 180)
 		(fields_autoplaced yes)
 		(effects
@@
 		)
 		(property "Intersheetrefs" "${INTERSHEET_REFS}"
-			(at 216.4225 294.64 0)
+			(at 221.5025 294.64 0)
 			(effects
 				(font
@@
 	(global_label "Cube_3_A-G7"
 		(shape input)
-		(at 232.41 365.76 180)
+		(at 237.49 365.76 180)
 		(fields_autoplaced yes)
 		(effects
@@
 		)
 		(property "Intersheetrefs" "${INTERSHEET_REFS}"
-			(at 216.483 365.76 0)
+			(at 221.563 365.76 0)
 			(effects
 				(font
@@
 	(global_label "Cube_3_A-H3"
 		(shape input)
-		(at 232.41 317.5 180)
+		(at 237.49 317.5 180)
 		(fields_autoplaced yes)
 		(effects
@@
 		)
 		(property "Intersheetrefs" "${INTERSHEET_REFS}"
-			(at 216.4225 317.5 0)
+			(at 221.5025 317.5 0)
 			(effects
 				(font
@@
 	(global_label "Cube_3_A-H5"
 		(shape input)
-		(at 232.41 342.9 180)
+		(at 237.49 342.9 180)
 		(fields_autoplaced yes)
 		(effects
@@
 		)
 		(property "Intersheetrefs" "${INTERSHEET_REFS}"
-			(at 216.4225 342.9 0)
+			(at 221.5025 342.9 0)
 			(effects
 				(font
@@
 	(global_label "Cube_3_A-G2"
 		(shape input)
-		(at 232.41 297.18 180)
+		(at 237.49 297.18 180)
 		(fields_autoplaced yes)
 		(effects
@@
 		)
 		(property "Intersheetrefs" "${INTERSHEET_REFS}"
-			(at 216.483 297.18 0)
+			(at 221.563 297.18 0)
 			(effects
 				(font
@@
 	(global_label "Cube_3_A-G6"
 		(shape input)
-		(at 232.41 347.98 180)
+		(at 237.49 347.98 180)
 		(fields_autoplaced yes)
 		(effects
@@
 		)
 		(property "Intersheetrefs" "${INTERSHEET_REFS}"
-			(at 216.483 347.98 0)
+			(at 221.563 347.98 0)
 			(effects
 				(font
@@
 	(global_label "Cube_3_A-G4"
 		(shape input)
-		(at 232.41 322.58 180)
+		(at 237.49 322.58 180)
 		(fields_autoplaced yes)
 		(effects
@@
 		)
 		(property "Intersheetrefs" "${INTERSHEET_REFS}"
-			(at 216.483 322.58 0)
+			(at 221.563 322.58 0)
 			(effects
 				(font
@@
 	(global_label "Cube_3_A-H6"
 		(shape input)
-		(at 232.41 345.44 180)
+		(at 237.49 345.44 180)
 		(fields_autoplaced yes)
 		(effects
@@
 		)
 		(property "Intersheetrefs" "${INTERSHEET_REFS}"
-			(at 216.4225 345.44 0)
+			(at 221.5025 345.44 0)
 			(effects
 				(font
@@
 	(global_label "Cube_3_A-H1"
 		(shape input)
-		(at 232.41 292.1 180)
+		(at 237.49 292.1 180)
 		(fields_autoplaced yes)
 		(effects
@@
 		)
 		(property "Intersheetrefs" "${INTERSHEET_REFS}"
-			(at 216.4225 292.1 0)
+			(at 221.5025 292.1 0)
 			(effects
 				(font
@@
 	(global_label "Cube_3_A-G3"
 		(shape input)
-		(at 232.41 314.96 180)
+		(at 237.49 314.96 180)
 		(fields_autoplaced yes)
 		(effects
@@
 		)
 		(property "Intersheetrefs" "${INTERSHEET_REFS}"
-			(at 216.483 314.96 0)
+			(at 221.563 314.96 0)
 			(effects
 				(font
@@
 	(global_label "Cube_3_A-G5"
 		(shape input)
-		(at 232.41 340.36 180)
+		(at 237.49 340.36 180)
 		(fields_autoplaced yes)
 		(effects
@@
 		)
 		(property "Intersheetrefs" "${INTERSHEET_REFS}"
-			(at 216.483 340.36 0)
+			(at 221.563 340.36 0)
 			(effects
 				(font
@@
 	(global_label "Cube_3_A-G1"
 		(shape input)
-		(at 232.41 289.56 180)
+		(at 237.49 289.56 180)
 		(fields_autoplaced yes)
 		(effects
@@
 		)
 		(property "Intersheetrefs" "${INTERSHEET_REFS}"
-			(at 216.483 289.56 0)
+			(at 221.563 289.56 0)
 			(effects
 				(font
@@
 	(global_label "Cube_3_A-G8"
 		(shape input)
-		(at 232.41 373.38 180)
+		(at 237.49 373.38 180)
 		(fields_autoplaced yes)
 		(effects
@@
 		)
 		(property "Intersheetrefs" "${INTERSHEET_REFS}"
-			(at 216.483 373.38 0)
+			(at 221.563 373.38 0)
 			(effects
 				(font

Commit message: .
Connections:
- net GND: now also J1.SH1, J1.SH2
Changed lines of the file:
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@@
 	)
 	(junction
+		(at 674.37 434.34)
+		(diameter 0)
+		(color 0 0 0 0)
+	)
+	(junction
 		(at 326.39 356.87)
 		(diameter 0)
@@
 	(wire
 		(pts
+			(xy 673.1 434.34) (xy 674.37 434.34)
+		)
+		(stroke
+			(width 0)
+			(type default)
+		)
+	)
+	(wire
+		(pts
 			(xy 149.86 228.6) (xy 149.86 231.14)
 		)
@@
 	(wire
 		(pts
+			(xy 675.64 434.34) (xy 674.37 434.34)
+		)
+		(stroke
+			(width 0)
+			(type default)
+		)
+	)
+	(wire
+		(pts
 			(xy 262.89 373.38) (xy 265.43 373.38)
 		)
@@
 	(wire
 		(pts
+			(xy 673.1 433.07) (xy 673.1 434.34)
+		)
+		(stroke
+			(width 0)
+			(type default)
+		)
+	)
+	(wire
+		(pts
 			(xy 328.93 363.22) (xy 326.39 363.22)
 		)
@@
 	(wire
 		(pts
+			(xy 675.64 433.07) (xy 675.64 434.34)
+		)
+		(stroke
+			(width 0)
+			(type default)
+		)
+	)
+	(wire
+		(pts
 			(xy 295.91 439.42) (xy 295.91 438.15)
 		)
@@
 		(pin "1"
 		)
+		(pin "SH2"
+		)
+		(pin "SH1"
+		)
 		(instances
 			(project "4-MPPC_FARICH_Prototype"
@@
 					(unit 1)
 				)
+			)
+		)
+	)
+	(symbol
+		(lib_id "power:GND")
+		(at 674.37 434.34 0)
+		(unit 1)
+		(exclude_from_sim no)
+		(in_bom yes)
+		(on_board yes)
+		(dnp no)
+		(fields_autoplaced yes)
+		(property "Reference" "#PWR074"
+			(at 674.37 440.69 0)
+			(effects
+				(font
+					(size 1.27 1.27)
+				)
+				(hide yes)
+			)
+		)
+		(property "Value" "GND"
+			(at 674.37 439.42 0)
+			(effects
+				(font
+					(size 1.27 1.27)
+				)
+			)
+		)
+		(property "Footprint" ""
+			(at 674.37 434.34 0)
+			(effects
+				(font
+					(size 1.27 1.27)
+				)
+				(hide yes)
+			)
+		)
+		(property "Datasheet" ""
+			(at 674.37 434.34 0)
+			(effects
+				(font
+					(size 1.27 1.27)
+				)
+				(hide yes)
+			)
+		)
+		(property "Description" "Power symbol creates a global label with name \"GND\" , ground"
+			(at 674.37 434.34 0)
+			(effects
+				(font
+					(size 1.27 1.27)
+				)
+				(hide yes)
+			)
+		)
+		(pin "1"
+		)
+		(instances
+			(project "4-MPPC_FARICH_Prototype"
+				(path "/87fe9a77-45d2-4007-8a54-2fe097a18bc5"
+					(reference "#PWR074")
+					(unit 1)
+				)
