File: FARICH_injection_board/FARICH Injection Board/FARICH Injection Board.kicad_pcb (KiCad board)
At the start: 4 copper layers, 32 x 32 mm, 33 parts, among them J1 ST4-40-1.00-L-D-P-TR

Commit message: .
Routing:
- net Cube_1_A-F8: track 8.62 -> 9.13 mm
