File: FARICH_injection_board/FARICH Injection Board/FARICH Injection Board.kicad_sch (KiCad schematic)
At the start: 33 parts, among them J1 ST4-40-1.00-L-D-P-TR

Commit message: .
Connections:
- removed net Onboard_HV: J1.01, J1.02, J1.03, J1.04, J1.17, J1.18, J1.19, J1.20, J1.21, J1.22, J1.23, J1.24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
