File: UV_LED_Driver/UV_LED_Pulse/UV_LED_Pulse.kicad_pcb (KiCad board)
At the start: 2 copper layers, 37.5 x 18.1 mm, 25 parts, among them J1 PWR/Signal, Q1 BC817, Q2 2N7002

Commit message: .
Other:
- board text added: "Title: Pulsated UV LED REV: 0/January 2025 Author: Dr. Alexandru Enciu Institution: TU Darmstadt"
- board text removed: "Title: Pulsated UV LED REV: 0/January 2025 Author: Dr. Alexandru Enciu Institution: Technische Universität Darmstadt"
Changed lines of the file:
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@@
 		(tags "capacitor")
 		(property "Reference" "C3"
-			(at 0 -1.43 360)
+			(at 0 -1.43 0)
 			(layer "F.SilkS")
 			(effects
@@
 		)
 		(property "Value" "1uF"
-			(at 0 1.43 360)
+			(at 0 1.43 0)
 			(layer "F.Fab")
 			(effects
@@
 		)
 		(fp_text user "${REFERENCE}"
-			(at 0 0 360)
+			(at 0 0 0)
 			(layer "F.Fab")
 			(effects
@@
 			(net 4 "Net-(U1-INTV_cc)")
 			(pintype "passive")
+			(teardrops
+				(best_length_ratio 0.5)
+				(max_length 1)
+				(best_width_ratio 1)
+				(max_width 2)
+				(curve_points 0)
+				(filter_ratio 0.9)
+				(enabled yes)
+				(allow_two_segments yes)
+				(prefer_zone_connections yes)
+			)
 		)
 		(pad "2" smd roundrect
@@
 		)
 		(property "Value" "D_Schottky"
-			(at 7.875 1.365 360)
+			(at 7.875 1.365 0)
 			(layer "F.Fab")
 			(effects
@@
 		)
 		(property "Footprint" "UV_Leds:SOT323_INFINEON"
-			(at 0 0 360)
+			(at 0 0 0)
 			(layer "F.Fab")
 			(hide yes)
@@
 		)
 		(property "Datasheet" ""
-			(at 0 0 360)
+			(at 0 0 0)
 			(layer "F.Fab")
 			(hide yes)
@@
 		)
 		(property "Description" "Schottky diode"
-			(at 0 0 360)
+			(at 0 0 0)
 			(layer "F.Fab")
 			(hide yes)
@@
 		)
 		(property "Value" "4.7u"
-			(at 0 2.3 360)
+			(at 0 2.3 0)
 			(layer "F.Fab")
 			(effects
@@
 		)
 		(fp_text user "${REFERENCE}"
-			(at 0 0 360)
+			(at 0 0 0)
 			(layer "F.Fab")
 			(effects
@@
 		(tags "resistor")
 		(property "Reference" "R4"
-			(at 0 1.32 360)
+			(at 0 1.32 0)
 			(layer "F.SilkS")
 			(effects
@@
 		)
 		(property "Value" "150"
-			(at 0 1.43 360)
+			(at 0 1.43 0)
 			(layer "F.Fab")
 			(effects
@@
 		)
 		(fp_text user "${REFERENCE}"
-			(at 0 0 360)
+			(at 0 0 0)
 			(layer "F.Fab")
 			(effects
@@
 		)
 		(property "Value" "4.7u"
-			(at 0 2.3 360)
+			(at 0 2.3 0)
 			(layer "F.Fab")
 			(effects
@@
 		)
 		(fp_text user "${REFERENCE}"
-			(at 0 0 360)
+			(at 0 0 0)
 			(layer "F.Fab")
 			(effects
@@
 		(layer "Edge.Cuts")
 	)
-	(gr_text "Title: Pulsated UV LED\nREV: 0/January 2025\nAuthor: Dr. Alexandru Enciu\nInstitution: Technische Universität Darmstadt\n"
-		(at 98.125 79.91 0)
+	(gr_text "Title: Pulsated UV LED\nREV: 0/January 2025\nAuthor: Dr. Alexandru Enciu\nInstitution: TU Darmstadt\n"
+		(at 100.095 64.54 90)
 		(layer "B.SilkS")
 		(effects
@@
 	)
 	(zone
-		(net 2)
-		(net_name "GND")
-		(layer "F.Cu")
-		(hatch edge 0.5)
-		(priority 1)
-		(connect_pads yes
-			(clearance 0.15)
-		)
-		(min_thickness 0.15)
-		(filled_areas_thickness no)
-		(fill yes
-			(thermal_gap 0.5)
-			(thermal_bridge_width 0.5)
-		)
-		(polygon
-			(pts
-				(xy 74 75.9) (xy 74 80.44) (xy 85.54 80.43) (xy 85.54 73.99) (xy 79.4 74) (xy 79.4 77.7) (xy 77 77.7)
-				(xy 77 75.9)
-			)
-		)
-	)
-	(zone
 		(net 10)
 		(net_name "GPIO_PWM")
@@
 	)
 	(zone
+		(net 2)
+		(net_name "GND")
+		(layer "F.Cu")
+		(hatch edge 0.5)
+		(priority 1)
+		(connect_pads yes
+			(clearance 0.15)
+		)
+		(min_thickness 0.15)
+		(filled_areas_thickness no)
+		(fill yes
+			(thermal_gap 0.5)
+			(thermal_bridge_width 0.5)
+		)
+		(polygon
+			(pts
+				(xy 74 75.9) (xy 74 80.44) (xy 85.54 80.43) (xy 85.54 73.99) (xy 79.4 74) (xy 79.4 77.7) (xy 77 77.7)
+				(xy 77 75.9)
+			)
+		)
+	)
+	(zone
 		(net 3)
 		(net_name "+3V3")
@@
 			)
 		)
+	)
+	(zone
+		(net 4)
+		(net_name "Net-(U1-INTV_cc)")
+		(layer "F.Cu")
+		(name "$teardrop_padvia$")
+		(hatch full 0.1)
+		(priority 30000)
+		(attr
+			(teardrop
+				(type padvia)
+			)
+		)
+		(connect_pads yes
+			(clearance 0)
+		)
+		(min_thickness 0.0254)
+		(filled_areas_thickness no)
+		(fill yes
+			(thermal_gap 0.5)
+			(thermal_bridge_width 0.5)
+			(island_removal_mode 1)
+			(island_area_min 10)
+		)
+		(polygon
+			(pts
+				(xy 99.102318 68.83) (xy 99.102318 69.13) (xy 100.000162 69.13) (xy 99.9884 68.655) (xy 99.551109 68.336076)
+			)
+		)

Commit message: .
Parts:
- added REF**: OSHW-Logo2_7.3x6mm_SilkScreen, Symbol:OSHW-Logo2_7.3x6mm_SilkScreen, F.Cu at (97.4, 77.6)
- added REF**: WEEE-Logo_4.2x6mm_SilkScreen, Symbol:WEEE-Logo_4.2x6mm_SilkScreen, B.Cu at (69.6, 71.8)

Commit message: .
Parts:
- removed the REF** at (69.6, 71.8)
- added D3: LED, LED_SMD:LED_0603_1608Metric, F.Cu at (84.9, 66.4)
- added D4: LED, LED_SMD:LED_0603_1608Metric, F.Cu at (88.5, 66.4)
- added R8: 600, Resistor_SMD:R_0603_1608Metric, F.Cu at (86.5, 66.4)
- added R9: 1k, Resistor_SMD:R_0603_1608Metric, F.Cu at (90.2, 66.4)
- moved REF** 2.00 mm to (70.6, 78.9)
- moved REF** 2.00 mm to (70.6, 64.9)
- moved REF** 0.53 mm to (102.6, 78.9)
- moved REF** 0.52 mm to (102.6, 64.9)
Routing:
- net GND: track 4.12 -> 6.13 mm, vias 54 -> 56
- net Net-(D4-A): track 0.00 -> 1.62 mm
- net Net-(D3-A): track 0.00 -> 1.62 mm
Other:
- board size 37.5 x 18.1 mm -> 36 x 18 mm
