File: UV_LED_Driver/UV_LED_Pulse/UV_LED_Pulse.kicad_sch (KiCad schematic)
At the start: 25 parts, among them J1 PWR/Signal, Q1 BC817, Q2 2N7002

Commit message: .
Other:
- added sheet UV LED datasheet (Wavelength_Intensity.kicad_sch)
- moved on the sheet: C1, C2, C3, C4, C5, C6, C7, D1, D2, D3, D4, J1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

Commit message: .
Parts:
- R1: value 4k7 -> 249
- R5: value 9k09 -> 90.9k
- R6: value 24k9 -> 35.7k
- R7: value 392 -> 0
Changed lines of the file:
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@@
 (kicad_sch
-	(version 20231120)
+	(version 20250114)
 	(generator "eeschema")
-	(generator_version "8.0")
+	(generator_version "9.0")
 	(paper "A5")
 	(title_block
@@
 		(rev "0")
 	)
+	(rectangle
+		(start 129.54 58.42)
+		(end 172.72 101.6)
+		(stroke
+			(width 0)
+			(type dash)
+		)
+		(fill
+			(type color)
+			(color 255 213 184 0.56)
+		)
+	)
+	(rectangle
+		(start 13.97 13.97)
+		(end 82.55 60.96)
+		(stroke
+			(width 0)
+			(type dash)
+		)
+		(fill
+			(type color)
+			(color 255 255 168 1)
+		)
+	)
+	(rectangle
+		(start 80.01 77.47)
+		(end 128.27 95.25)
+		(stroke
+			(width 0)
+			(type dash)
+		)
+		(fill
+			(type color)
+			(color 251 204 255 1)
+		)
+	)
+	(rectangle
+		(start 83.82 24.13)
+		(end 156.21 48.26)
+		(stroke
+			(width 0)
+			(type dash)
+		)
+		(fill
+			(type color)
+			(color 255 187 185 1)
+		)
+	)
+	(text "Populate only if a \nPULL-UP/DOWN is needed"
+		(exclude_from_sim no)
+		(at 157.734 81.534 0)
+		(effects
+			(font
+				(size 1.27 1.27)
+			)
+		)
+	)
+	(text "3.3V to 5.8V Step-UP converter"
+		(exclude_from_sim no)
+		(at 46.736 16.51 0)
+		(effects
+			(font
+				(size 1.27 1.27)
+				(thickness 0.254)
+				(bold yes)
+			)
+		)
+	)
+	(text "Pulse Trigger"
+		(exclude_from_sim no)
+		(at 142.748 93.726 0)
+		(effects
+			(font
+				(size 1.27 1.27)
+			)
+		)
+	)
+	(text "LED curent control via PWM"
+		(exclude_from_sim no)
+		(at 94.488 94.488 0)
+		(effects
+			(font
+				(size 1.27 1.27)
+			)
+		)
+	)
 	(junction
 		(at 49.53 26.67)
@@
 		)
 	)
-	(rectangle
-		(start 129.54 58.42)
-		(end 172.72 101.6)
-		(stroke
-			(width 0)
-			(type dash)
-		)
-		(fill
-			(type color)
-			(color 255 213 184 0.56)
-		)
-	)
-	(rectangle
-		(start 13.97 13.97)
-		(end 82.55 60.96)
-		(stroke
-			(width 0)
-			(type dash)
-		)
-		(fill
-			(type color)
-			(color 255 255 168 1)
-		)
-	)
-	(rectangle
-		(start 80.01 77.47)
-		(end 128.27 95.25)
-		(stroke
-			(width 0)
-			(type dash)
-		)
-		(fill
-			(type color)
-			(color 251 204 255 1)
-		)
-	)
-	(rectangle
-		(start 83.82 24.13)
-		(end 156.21 48.26)
-		(stroke
-			(width 0)
-			(type dash)
-		)
-		(fill
-			(type color)
-			(color 255 187 185 1)
-		)
-	)
-	(text "Populate only if a \nPULL-UP/DOWN is needed"
-		(exclude_from_sim no)
-		(at 157.734 81.534 0)
-		(effects
-			(font
-				(size 1.27 1.27)
-			)
-		)
-	)
-	(text "3.3V to 5.8V Step-UP converter"
-		(exclude_from_sim no)
-		(at 46.736 16.51 0)
-		(effects
-			(font
-				(size 1.27 1.27)
-				(thickness 0.254)
-				(bold yes)
-			)
-		)
-	)
-	(text "Pulse Trigger"
-		(exclude_from_sim no)
-		(at 142.748 93.726 0)
-		(effects
-			(font
-				(size 1.27 1.27)
-			)
-		)
-	)
-	(text "LED curent control via PWM"
-		(exclude_from_sim no)
-		(at 94.488 94.488 0)
-		(effects
-			(font
-				(size 1.27 1.27)
-			)
-		)
-	)
 	(label "LED_Power"
 		(at 67.31 26.67 0)
-		(fields_autoplaced yes)
 		(effects
 			(font
@@
 			)
 		)
-		(property "Value" "4k7"
+		(property "Value" "249"
 			(at 97.79 82.55 90)
 			(effects
@@
 			)
 		)
-		(property "Value" "392"
+		(property "Value" "0"
 			(at 60.96 30.48 90)
 			(effects
@@
 			)
 		)
-		(property "Value" "24k9"
+		(property "Value" "35.7k"
 			(at 60.96 46.99 90)
 			(effects
@@
 			)
 		)
-		(property "Value" "9k09"
+		(property "Value" "90.9k"
 			(at 60.96 38.1 90)
 			(effects
@@
 		(at 93.98 68.58)
 		(size 17.78 5.08)
+		(exclude_from_sim no)
+		(in_bom yes)
+		(on_board yes)
+		(dnp no)
 		(stroke
 			(width 0.1524)
@@
 		)
 	)
+	(embedded_fonts no)
 )

Commit message: .
Parts:
- L1: value 0.68uH -> 4.7 uH; Component WURTH WE-MAPI 3012 744383340068 -> WE 744029004
Changed lines of the file:
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@@
 			)
 		)
-		(property "Value" "0.68uH"
+		(property "Value" "4.7 uH"
 			(at 44.45 24.13 90)
 			(effects
@@
 			)
 		)
-		(property "Component" "WURTH WE-MAPI 3012 744383340068"
+		(property "Component" "WE 744029004"
 			(at 44.45 26.67 90)
 			(effects

Commit message: .
Parts:
- R2, R3: now not fitted
- R5: value 90.9k -> 90k9
- R6: value 35.7k -> 35k7
Changed lines of the file:
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@@
 		(in_bom yes)
 		(on_board yes)
-		(dnp no)
+		(dnp yes)
 		(property "Reference" "R2"
-			(at 137.16 77.216 90)
+			(at 137.16 78.74 90)
 			(effects
 				(font
@@
 		)
 		(property "Value" "10k"
-			(at 137.16 74.93 90)
+			(at 137.16 76.962 90)
 			(effects
 				(font
@@
 			)
 		)
-		(property "Value" "35.7k"
+		(property "Value" "35k7"
 			(at 60.96 46.99 90)
 			(effects
@@
 			)
 		)
-		(property "Value" "90.9k"
+		(property "Value" "90k9"
 			(at 60.96 38.1 90)
 			(effects
@@
 		(in_bom yes)
 		(on_board yes)
-		(dnp no)
+		(dnp yes)
 		(property "Reference" "R3"
+			(at 147.32 78.994 90)
+			(effects
+				(font
+					(size 1.27 1.27)
+				)
+			)
+		)
+		(property "Value" "10k"
 			(at 147.32 77.216 90)
 			(effects
 				(font
-					(size 1.27 1.27)
-				)
-			)
-		)
-		(property "Value" "10k"
-			(at 147.32 74.93 90)
-			(effects
-				(font
