File: HV_PSU/HV_PSU_C11204-01_V2/HV_PSU_C11204-01_V2/HV_PSU_C11204-01_V2.kicad_sch (KiCad schematic)
At the start: 53 parts, among them J1 TMP1, J2 HV, Q1 2N7002, Q2 2N7002, Q3 S9014, U3 DM-OLED096-636

Commit message: .
Connections:
- net +3V3: now also U4.1 (+); no longer U4.10 (-)
- net at D1.2 (A), Q3.3 (C): now also U4.10 (-); no longer U4.1 (+)
Other:
- moved on the sheet: D1
Changed lines of the file:
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@@
 	(paper "A4")
 	(junction
-		(at 232.41 93.98)
-		(diameter 0)
-		(color 0 0 0 0)
-	)
-	(junction
 		(at 223.52 104.14)
 		(diameter 0)
@@
 	)
 	(junction
-		(at 76.2 52.07)
+		(at 229.87 82.55)
 		(diameter 0)
 		(color 0 0 0 0)
 	)
 	(junction
-		(at 186.69 36.83)
+		(at 76.2 52.07)
 		(diameter 0)
 		(color 0 0 0 0)
 	)
 	(junction
-		(at 257.81 86.36)
+		(at 186.69 36.83)
 		(diameter 0)
 		(color 0 0 0 0)
@@
 	)
 	(junction
+		(at 229.87 90.17)
+		(diameter 0)
+		(color 0 0 0 0)
+	)
+	(junction
 		(at 111.76 39.37)
 		(diameter 0)
@@
 	(wire
 		(pts
-			(xy 232.41 86.36) (xy 232.41 93.98)
-		)
-		(stroke
-			(width 0)
-			(type default)
-		)
-	)
-	(wire
-		(pts
 			(xy 115.57 139.7) (xy 116.84 139.7)
 		)
@@
 	(wire
 		(pts
-			(xy 180.34 50.8) (xy 173.99 50.8)
+			(xy 233.68 82.55) (xy 233.68 93.98)
 		)
 		(stroke
@@
 	(wire
 		(pts
-			(xy 63.5 165.1) (xy 63.5 163.83)
+			(xy 180.34 50.8) (xy 173.99 50.8)
 		)
 		(stroke
@@
 	(wire
 		(pts
-			(xy 190.5 36.83) (xy 189.23 36.83)
+			(xy 63.5 165.1) (xy 63.5 163.83)
 		)
 		(stroke
@@
 	(wire
 		(pts
-			(xy 232.41 93.98) (xy 233.68 93.98)
+			(xy 190.5 36.83) (xy 189.23 36.83)
 		)
 		(stroke
@@
 	(wire
 		(pts
-			(xy 228.6 93.98) (xy 232.41 93.98)
+			(xy 228.6 93.98) (xy 229.87 93.98)
 		)
 		(stroke
@@
 	(wire
 		(pts
+			(xy 229.87 81.28) (xy 229.87 82.55)
+		)
+		(stroke
+			(width 0)
+			(type default)
+		)
+	)
+	(wire
+		(pts
 			(xy 175.26 36.83) (xy 173.99 36.83)
 		)
@@
 	(wire
 		(pts
+			(xy 229.87 90.17) (xy 229.87 93.98)
+		)
+		(stroke
+			(width 0)
+			(type default)
+		)
+	)
+	(wire
+		(pts
 			(xy 168.91 82.55) (xy 175.26 82.55)
 		)
@@
 	(wire
 		(pts
-			(xy 257.81 86.36) (xy 257.81 93.98)
-		)
-		(stroke
-			(width 0)
-			(type default)
-		)
-	)
-	(wire
-		(pts
 			(xy 180.34 29.21) (xy 173.99 29.21)
 		)
@@
 	(wire
 		(pts
-			(xy 214.63 104.14) (xy 214.63 93.98)
-		)
-		(stroke
-			(width 0)
-			(type default)
-		)
-	)
-	(wire
-		(pts
-			(xy 102.87 39.37) (xy 101.6 39.37)
+			(xy 256.54 90.17) (xy 229.87 90.17)
 		)
 		(stroke
@@
 	(wire
 		(pts
-			(xy 223.52 114.3) (xy 223.52 113.03)
+			(xy 214.63 104.14) (xy 214.63 93.98)
 		)
 		(stroke
@@
 	(wire
 		(pts
-			(xy 248.92 86.36) (xy 257.81 86.36)
+			(xy 102.87 39.37) (xy 101.6 39.37)
 		)
 		(stroke
@@
 	(wire
 		(pts
-			(xy 257.81 93.98) (xy 256.54 93.98)
+			(xy 223.52 114.3) (xy 223.52 113.03)
 		)
 		(stroke
@@
 	(wire
 		(pts
+			(xy 256.54 93.98) (xy 256.54 90.17)
+		)
+		(stroke
+			(width 0)
+			(type default)
+		)
+	)
+	(wire
+		(pts
 			(xy 172.72 140.97) (xy 173.99 140.97)
 		)
@@
 	(wire
 		(pts
-			(xy 241.3 86.36) (xy 232.41 86.36)
+			(xy 233.68 82.55) (xy 229.87 82.55)
 		)
 		(stroke
@@
 	(symbol
 		(lib_id "power:+3V3")
-		(at 257.81 86.36 0)
+		(at 229.87 81.28 0)
 		(unit 1)
 		(exclude_from_sim no)
@@
 		(fields_autoplaced yes)
 		(property "Reference" "#PWR040"
-			(at 257.81 90.17 0)
+			(at 229.87 85.09 0)
 			(effects
 				(font
@@
 		)
 		(property "Value" "+3V3"
-			(at 257.81 81.28 0)
+			(at 229.87 76.2 0)
 			(effects
 				(font
@@
 		)
 		(property "Footprint" ""
-			(at 257.81 86.36 0)
+			(at 229.87 81.28 0)
 			(effects
 				(font
@@
 		)
 		(property "Datasheet" ""
-			(at 257.81 86.36 0)
+			(at 229.87 81.28 0)
 			(effects
 				(font
@@
 		)
 		(property "Description" "Power symbol creates a global label with name \"+3V3\""
-			(at 257.81 86.36 0)
+			(at 229.87 81.28 0)
 			(effects
 				(font
@@
 	(symbol
 		(lib_id "Device:D")
-		(at 245.11 86.36 0)
-		(mirror y)
+		(at 229.87 86.36 90)
+		(mirror x)
 		(unit 1)
 		(exclude_from_sim no)
@@
 		(dnp no)
 		(property "Reference" "D1"
-			(at 245.11 80.01 0)
+			(at 223.52 86.36 0)
 			(effects
 				(font
@@
 		)
 		(property "Value" "TS4148rcg"
-			(at 245.11 82.55 0)
+			(at 226.06 86.36 0)
 			(effects
 				(font
@@
 		)
 		(property "Footprint" "Diode_SMD:D_0603_1608Metric"
-			(at 245.11 86.36 0)
+			(at 229.87 86.36 0)
 			(effects
 				(font
@@
 		)
 		(property "Datasheet" "~"
-			(at 245.11 86.36 0)
+			(at 229.87 86.36 0)
 			(effects
 				(font
@@
 		)
 		(property "Description" "Diode"
-			(at 245.11 86.36 0)
+			(at 229.87 86.36 0)
 			(effects
 				(font
@@
 		)
 		(property "Sim.Device" "D"
-			(at 245.11 86.36 0)
+			(at 229.87 86.36 0)
 			(effects
 				(font
@@
 		)
 		(property "Sim.Pins" "1=K 2=A"
-			(at 245.11 86.36 0)
+			(at 229.87 86.36 0)
 			(effects
 				(font

Commit message: .
Other:
- moved on the sheet: D1, HV_On1, Q3
