File: HV_PSU/HV_PSU_C11204-01_V2/HV_PSU_C11204-01_V2/HV_PSU_C11204-01_V2.kicad_pcb (KiCad board)
At the start: 4 copper layers, 62.7 x 26 mm, 53 parts, among them J1 TMP1, J2 HV, Q1 2N7002, Q2 2N7002, Q3 S9014, U3 DM-OLED096-636

Commit message: .
Parts:
- moved D1 10.4 mm to (112.6, 80.9)
Connections:
- U4 pad 1: Net-(D1-A) -> +3V3
- U4 pad 10: +3V3 -> Net-(D1-A)
Routing:
- net Net-(D1-A): track 15.6 -> 9.97 mm
- net +3V3: track 12.4 -> 15.4 mm

Commit message: .
Routing:
- net GND: track 41.9 -> 40.3 mm
- net SW1: track 23.9 -> 23.0 mm
