File: SmallFiber/SiPM_Array_for_VMM3a_Rev-0/SiPM_Array_for_VMM3a_Rev-0.kicad_pcb (KiCad board)
At the start: 4 copper layers, 60 x 25 mm, 2 parts

Commit message: .
Parts:
- removed U101: ~, 0_lib:Hirose-FX10
- added C1: 100nF/100V, Capacitor_SMD:C_0201_0603Metric, B.Cu at (112.8, 85.2)
- added C10: 100nF/100V, Capacitor_SMD:C_0201_0603Metric, F.Cu at (86.0, 67.5)
- added C11: 100nF/100V, Capacitor_SMD:C_0201_0603Metric, F.Cu at (86.0, 69.5)
- added C12: 100nF/100V, Capacitor_SMD:C_0201_0603Metric, F.Cu at (86.0, 71.4)
- added C2: 100nF/100V, Capacitor_SMD:C_0201_0603Metric, B.Cu at (113.3, 85.7)
- added C3: 100nF/100V, Capacitor_SMD:C_0201_0603Metric, B.Cu at (110.8, 85.2)
- added C4: 100nF/100V, Capacitor_SMD:C_0201_0603Metric, B.Cu at (112.3, 86.7)
- added C5: 100nF/100V, Capacitor_SMD:C_0201_0603Metric, B.Cu at (111.3, 85.7)
- added C6: 100nF/100V, Capacitor_SMD:C_0201_0603Metric, B.Cu at (111.8, 86.2)
- added C7: 100nF/100V, Capacitor_SMD:C_0201_0603Metric, F.Cu at (83.1, 69.5)
- added C8: 100nF/100V, Capacitor_SMD:C_0201_0603Metric, F.Cu at (83.1, 71.4)
- added C9: 100nF/100V, Capacitor_SMD:C_0201_0603Metric, F.Cu at (86.0, 65.5)
- added J1: ERM6-30-01.5-L-DV-A-K-TR, 0_lib:SAMTEC_ERM6-30-01.5-L-DV-A-K-TR, B.Cu at (126.3, 81.9)
- added J2: ERM6-30-01.5-L-DV-A-K-TR, 0_lib:SAMTEC_ERM6-30-01.5-L-DV-A-K-TR, B.Cu at (126.3, 97.9)
- added R1: R, Resistor_SMD:R_0201_0603Metric, B.Cu at (115.8, 84.2)
- added R2: R, Resistor_SMD:R_0201_0603Metric, B.Cu at (112.3, 84.7)
- added R3: R, Resistor_SMD:R_0201_0603Metric, B.Cu at (111.8, 84.2)
- added R4: R, Resistor_SMD:R_0201_0603Metric, F.Cu at (77.7, 69.9)
- added R5: R, Resistor_SMD:R_0201_0603Metric, F.Cu at (77.3, 73.5)
- added R6: R, Resistor_SMD:R_0201_0603Metric, F.Cu at (77.3, 75.5)
- moved MPPC1 0.98 mm to (126.3, 89.9)
Connections:
- MPPC1 pad 1: unconnected-(MPPC1-SignalOut-Pad1) -> Ch_1
- MPPC1 pad 10: unconnected-(MPPC1-SignalOut-Pad10) -> Ch_5
- MPPC1 pad 100: unconnected-(MPPC1-SignalOut-Pad100) -> Ch_50
- MPPC1 pad 101: unconnected-(MPPC1-SignalOut-Pad101) -> Ch_51
- MPPC1 pad 102: unconnected-(MPPC1-SignalOut-Pad102) -> Ch_51
- MPPC1 pad 103: unconnected-(MPPC1-SignalOut-Pad103) -> Ch_52
- MPPC1 pad 104: unconnected-(MPPC1-SignalOut-Pad104) -> Ch_52
- MPPC1 pad 105: unconnected-(MPPC1-SignalOut-Pad105) -> Ch_53
- MPPC1 pad 106: unconnected-(MPPC1-SignalOut-Pad106) -> Ch_53
- MPPC1 pad 107: unconnected-(MPPC1-SignalOut-Pad107) -> Ch_54
- MPPC1 pad 108: unconnected-(MPPC1-SignalOut-Pad108) -> Ch_54
- MPPC1 pad 109: unconnected-(MPPC1-SignalOut-Pad109) -> Ch_55
- MPPC1 pad 11: unconnected-(MPPC1-SignalOut-Pad11) -> Ch_6
- MPPC1 pad 110: unconnected-(MPPC1-SignalOut-Pad110) -> Ch_55
- MPPC1 pad 111: unconnected-(MPPC1-SignalOut-Pad111) -> Ch_56
- MPPC1 pad 112: unconnected-(MPPC1-SignalOut-Pad112) -> Ch_56
- MPPC1 pad 113: unconnected-(MPPC1-SignalOut-Pad113) -> Ch_57
- MPPC1 pad 114: unconnected-(MPPC1-SignalOut-Pad114) -> Ch_57
- MPPC1 pad 115: unconnected-(MPPC1-SignalOut-Pad115) -> Ch_58
- MPPC1 pad 116: unconnected-(MPPC1-SignalOut-Pad116) -> Ch_58
- MPPC1 pad 117: unconnected-(MPPC1-SignalOut-Pad117) -> Ch_59
- MPPC1 pad 118: unconnected-(MPPC1-SignalOut-Pad118) -> Ch_59
- MPPC1 pad 119: unconnected-(MPPC1-SignalOut-Pad119) -> Ch_60
- MPPC1 pad 12: unconnected-(MPPC1-SignalOut-Pad12) -> Ch_6
- MPPC1 pad 120: unconnected-(MPPC1-SignalOut-Pad120) -> Ch_60
- MPPC1 pad 121: unconnected-(MPPC1-SignalOut-Pad121) -> Ch_61
- MPPC1 pad 122: unconnected-(MPPC1-SignalOut-Pad122) -> Ch_61
- MPPC1 pad 123: unconnected-(MPPC1-SignalOut-Pad123) -> Ch_62
- MPPC1 pad 124: unconnected-(MPPC1-SignalOut-Pad124) -> Ch_62
- MPPC1 pad 125: unconnected-(MPPC1-SignalOut-Pad125) -> Ch_63
- MPPC1 pad 126: unconnected-(MPPC1-SignalOut-Pad126) -> Ch_63
- MPPC1 pad 127: unconnected-(MPPC1-SignalOut-Pad127) -> Ch_64
- MPPC1 pad 128: unconnected-(MPPC1-SignalOut-Pad128) -> Ch_64
- MPPC1 pad 13: unconnected-(MPPC1-SignalOut-Pad13) -> Ch_7
- MPPC1 pad 14: unconnected-(MPPC1-SignalOut-Pad14) -> Ch_7
- MPPC1 pad 15: unconnected-(MPPC1-SignalOut-Pad15) -> Ch_8
- MPPC1 pad 16: unconnected-(MPPC1-SignalOut-Pad16) -> Ch_8
- MPPC1 pad 17: unconnected-(MPPC1-SignalOut-Pad17) -> Ch_9
- MPPC1 pad 18: unconnected-(MPPC1-SignalOut-Pad18) -> Ch_9
- MPPC1 pad 19: unconnected-(MPPC1-SignalOut-Pad19) -> Ch_10
- MPPC1 pad 2: unconnected-(MPPC1-SignalOut-Pad2) -> Ch_1
- MPPC1 pad 20: unconnected-(MPPC1-SignalOut-Pad20) -> Ch_10
- MPPC1 pad 21: unconnected-(MPPC1-SignalOut-Pad21) -> Ch_11
- MPPC1 pad 22: unconnected-(MPPC1-SignalOut-Pad22) -> Ch_11
- MPPC1 pad 23: unconnected-(MPPC1-SignalOut-Pad23) -> Ch_12
- MPPC1 pad 24: unconnected-(MPPC1-SignalOut-Pad24) -> Ch_12
- MPPC1 pad 25: unconnected-(MPPC1-SignalOut-Pad25) -> Ch_13
- MPPC1 pad 26: unconnected-(MPPC1-SignalOut-Pad26) -> Ch_13
- MPPC1 pad 27: unconnected-(MPPC1-SignalOut-Pad27) -> Ch_14
- MPPC1 pad 28: unconnected-(MPPC1-SignalOut-Pad28) -> Ch_14
- MPPC1 pad 29: unconnected-(MPPC1-SignalOut-Pad29) -> Ch_15
- MPPC1 pad 3: unconnected-(MPPC1-SignalOut-Pad3) -> Ch_2
- MPPC1 pad 30: unconnected-(MPPC1-SignalOut-Pad30) -> Ch_15
- MPPC1 pad 31: unconnected-(MPPC1-SignalOut-Pad31) -> Ch_16
- MPPC1 pad 32: unconnected-(MPPC1-SignalOut-Pad32) -> Ch_16
- MPPC1 pad 33: unconnected-(MPPC1-SignalOut-Pad33) -> Ch_17
- MPPC1 pad 34: unconnected-(MPPC1-SignalOut-Pad34) -> Ch_17
- MPPC1 pad 35: unconnected-(MPPC1-SignalOut-Pad35) -> Ch_18
- MPPC1 pad 36: unconnected-(MPPC1-SignalOut-Pad36) -> Ch_18
- MPPC1 pad 37: unconnected-(MPPC1-SignalOut-Pad37) -> Ch_19
- MPPC1 pad 38: unconnected-(MPPC1-SignalOut-Pad38) -> Ch_19
- MPPC1 pad 39: unconnected-(MPPC1-SignalOut-Pad39) -> Ch_20
- MPPC1 pad 4: unconnected-(MPPC1-SignalOut-Pad4) -> Ch_2
- MPPC1 pad 40: unconnected-(MPPC1-SignalOut-Pad40) -> Ch_20
- MPPC1 pad 41: unconnected-(MPPC1-SignalOut-Pad41) -> Ch_21
- MPPC1 pad 42: unconnected-(MPPC1-SignalOut-Pad42) -> Ch_21
- MPPC1 pad 43: unconnected-(MPPC1-SignalOut-Pad43) -> Ch_22
- MPPC1 pad 44: unconnected-(MPPC1-SignalOut-Pad44) -> Ch_22
- MPPC1 pad 45: unconnected-(MPPC1-SignalOut-Pad45) -> Ch_23
- MPPC1 pad 46: unconnected-(MPPC1-SignalOut-Pad46) -> Ch_23
- MPPC1 pad 47: unconnected-(MPPC1-SignalOut-Pad47) -> Ch_24
- MPPC1 pad 48: unconnected-(MPPC1-SignalOut-Pad48) -> Ch_24
- MPPC1 pad 49: unconnected-(MPPC1-SignalOut-Pad49) -> Ch_25
- MPPC1 pad 5: unconnected-(MPPC1-SignalOut-Pad5) -> Ch_3
- MPPC1 pad 50: unconnected-(MPPC1-SignalOut-Pad50) -> Ch_25
- MPPC1 pad 51: unconnected-(MPPC1-SignalOut-Pad51) -> Ch_26
- MPPC1 pad 52: unconnected-(MPPC1-SignalOut-Pad52) -> Ch_26
- MPPC1 pad 53: unconnected-(MPPC1-SignalOut-Pad53) -> Ch_27
- MPPC1 pad 54: unconnected-(MPPC1-SignalOut-Pad54) -> Ch_27
- MPPC1 pad 55: unconnected-(MPPC1-SignalOut-Pad55) -> Ch_28
- MPPC1 pad 56: unconnected-(MPPC1-SignalOut-Pad56) -> Ch_28
- MPPC1 pad 57: unconnected-(MPPC1-SignalOut-Pad57) -> Ch_29
- MPPC1 pad 58: unconnected-(MPPC1-SignalOut-Pad58) -> Ch_29
- MPPC1 pad 59: unconnected-(MPPC1-SignalOut-Pad59) -> Ch_30
- MPPC1 pad 6: unconnected-(MPPC1-SignalOut-Pad6) -> Ch_3
- MPPC1 pad 60: unconnected-(MPPC1-SignalOut-Pad60) -> Ch_30
- MPPC1 pad 61: unconnected-(MPPC1-SignalOut-Pad61) -> Ch_31
- MPPC1 pad 62: unconnected-(MPPC1-SignalOut-Pad62) -> Ch_31
- MPPC1 pad 63: unconnected-(MPPC1-SignalOut-Pad63) -> Ch_32
- MPPC1 pad 64: unconnected-(MPPC1-SignalOut-Pad64) -> Ch_32
- MPPC1 pad 65: unconnected-(MPPC1-SignalOut-Pad65) -> Ch_33
- MPPC1 pad 66: unconnected-(MPPC1-SignalOut-Pad66) -> Ch_33
- MPPC1 pad 67: unconnected-(MPPC1-SignalOut-Pad67) -> Ch_34
- MPPC1 pad 68: unconnected-(MPPC1-SignalOut-Pad68) -> Ch_34
- MPPC1 pad 69: unconnected-(MPPC1-SignalOut-Pad69) -> Ch_35
- MPPC1 pad 7: unconnected-(MPPC1-SignalOut-Pad7) -> Ch_4
- MPPC1 pad 70: unconnected-(MPPC1-SignalOut-Pad70) -> Ch_35
- MPPC1 pad 71: unconnected-(MPPC1-SignalOut-Pad71) -> Ch_36
- MPPC1 pad 72: unconnected-(MPPC1-SignalOut-Pad72) -> Ch_36
- MPPC1 pad 73: unconnected-(MPPC1-SignalOut-Pad73) -> Ch_37
- MPPC1 pad 74: unconnected-(MPPC1-SignalOut-Pad74) -> Ch_37
- MPPC1 pad 75: unconnected-(MPPC1-SignalOut-Pad75) -> Ch_38
- MPPC1 pad 76: unconnected-(MPPC1-SignalOut-Pad76) -> Ch_38
- MPPC1 pad 77: unconnected-(MPPC1-SignalOut-Pad77) -> Ch_39
- MPPC1 pad 78: unconnected-(MPPC1-SignalOut-Pad78) -> Ch_39
- MPPC1 pad 79: unconnected-(MPPC1-SignalOut-Pad79) -> Ch_40
- MPPC1 pad 8: unconnected-(MPPC1-SignalOut-Pad8) -> Ch_4
- MPPC1 pad 80: unconnected-(MPPC1-SignalOut-Pad80) -> Ch_40
- MPPC1 pad 81: unconnected-(MPPC1-SignalOut-Pad81) -> Ch_41
- MPPC1 pad 82: unconnected-(MPPC1-SignalOut-Pad82) -> Ch_41
- MPPC1 pad 83: unconnected-(MPPC1-SignalOut-Pad83) -> Ch_42
- MPPC1 pad 84: unconnected-(MPPC1-SignalOut-Pad84) -> Ch_42
- MPPC1 pad 85: unconnected-(MPPC1-SignalOut-Pad85) -> Ch_43
- MPPC1 pad 86: unconnected-(MPPC1-SignalOut-Pad86) -> Ch_43
- MPPC1 pad 87: unconnected-(MPPC1-SignalOut-Pad87) -> Ch_44
- MPPC1 pad 88: unconnected-(MPPC1-SignalOut-Pad88) -> Ch_44
- MPPC1 pad 89: unconnected-(MPPC1-SignalOut-Pad89) -> Ch_45
- MPPC1 pad 9: unconnected-(MPPC1-SignalOut-Pad9) -> Ch_5
- MPPC1 pad 90: unconnected-(MPPC1-SignalOut-Pad90) -> Ch_45
- MPPC1 pad 91: unconnected-(MPPC1-SignalOut-Pad91) -> Ch_46
- MPPC1 pad 92: unconnected-(MPPC1-SignalOut-Pad92) -> Ch_46
- MPPC1 pad 93: unconnected-(MPPC1-SignalOut-Pad93) -> Ch_47
- MPPC1 pad 94: unconnected-(MPPC1-SignalOut-Pad94) -> Ch_47
- MPPC1 pad 95: unconnected-(MPPC1-SignalOut-Pad95) -> Ch_48
- MPPC1 pad 96: unconnected-(MPPC1-SignalOut-Pad96) -> Ch_48
- MPPC1 pad 97: unconnected-(MPPC1-SignalOut-Pad97) -> Ch_49
- MPPC1 pad 98: unconnected-(MPPC1-SignalOut-Pad98) -> Ch_49
- MPPC1 pad 99: unconnected-(MPPC1-SignalOut-Pad99) -> Ch_50
Routing:
- net Ch_2: track 0.00 -> 17.1 mm, vias 0 -> 3
- net Ch_63: track 0.00 -> 17.1 mm, vias 0 -> 3
- net Ch_1: track 0.00 -> 16.9 mm, vias 0 -> 2
- net Ch_3: track 0.00 -> 16.1 mm, vias 0 -> 3
- net Ch_62: track 0.00 -> 16.1 mm, vias 0 -> 3
- net Ch_61: track 0.00 -> 15.9 mm, vias 0 -> 2
- net Ch_5: track 0.00 -> 15.9 mm, vias 0 -> 2
- net Ch_4: track 0.00 -> 15.8 mm, vias 0 -> 2
- net Ch_59: track 0.00 -> 15.8 mm, vias 0 -> 3
- net Ch_6: track 0.00 -> 15.8 mm, vias 0 -> 3
- net Ch_60: track 0.00 -> 15.6 mm, vias 0 -> 2
- net Ch_7: track 0.00 -> 15.2 mm, vias 0 -> 3
- net Ch_58: track 0.00 -> 14.8 mm, vias 0 -> 3
- net Ch_9: track 0.00 -> 14.6 mm, vias 0 -> 2
- net Ch_57: track 0.00 -> 14.6 mm, vias 0 -> 2
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- added copper zone on In1.Cu, net GND
- added copper zone on In2.Cu, net GND
Other:
- board size 60 x 25 mm -> 32.5 x 20 mm

Commit message: .
Parts:
- removed C1, C10, C11, C2, C3, C4, C5, C7, C8, C9: 100nF/100V, Capacitor_SMD:C_0201_0603Metric
- C12: footprint Capacitor_SMD:C_0201_0603Metric -> Capacitor_SMD:C_0603_1608Metric
- C6: footprint Capacitor_SMD:C_0201_0603Metric -> Capacitor_SMD:C_0603_1608Metric; moved to F.Cu
- R1, R2, R3: moved to F.Cu
- moved R4 22.6 mm to (95.1, 84.3)
- moved R5 21.8 mm to (95.1, 86.0)
- moved R6 21.7 mm to (95.1, 87.8)
- moved R1 21.3 mm to (95.1, 79.0), turned to 0 degrees
- moved R2 17.6 mm to (95.1, 80.8), turned to 0 degrees
- moved R3 16.8 mm to (95.1, 82.5), turned to 0 degrees
- moved C12 16.3 mm to (98.4, 81.9)
- moved C6 15.1 mm to (98.4, 79.4), turned to 0 degrees
Routing:
- net HV_1-64: track 0.00 -> 16.5 mm
- net HV_65-128: track 0.00 -> 16.5 mm
- net GND: vias 3 -> 0

Commit message: .
Parts:
- added C13: 100nF/100V, Capacitor_SMD:C_0603_1608Metric, F.Cu at (141.4, 94.6)
- added C7: 100nF/100V, Capacitor_SMD:C_0603_1608Metric, F.Cu at (112.2, 84.1)
- R1, R2, R3, R4, R5, R6: moved to B.Cu
- moved R6 45.7 mm to (140.5, 94.0), turned to 45 degrees
- moved R5 45.7 mm to (139.9, 95.1), turned to -45 degrees
- moved R4 45.2 mm to (138.9, 95.6), turned to 45 degrees
- moved C12 43.9 mm to (140.4, 94.6), turned to -90 degrees
- moved R1 19.6 mm to (114.1, 84.3), turned to -135 degrees
- moved R2 18.4 mm to (113.0, 84.8), turned to 135 degrees
- moved R3 17.7 mm to (112.5, 85.8), turned to -135 degrees
- moved C6 13.6 mm to (111.2, 84.1), turned to 90 degrees
Connections:
- J1 pad 01: HV_65-128_in -> GND
- J1 pad 03: unconnected-(J1-Pad03) -> GND
- J1 pad 04: unconnected-(J1-Pad04) -> GND
- J1 pad 05: unconnected-(J1-Pad05) -> GND
- J1 pad 06: unconnected-(J1-Pad06) -> GND
- J1 pad 07: unconnected-(J1-Pad07) -> GND
- J1 pad 08: unconnected-(J1-Pad08) -> GND
- J1 pad 09: unconnected-(J1-Pad09) -> GND
- J1 pad 10: unconnected-(J1-Pad10) -> GND
- J1 pad 11: unconnected-(J1-Pad11) -> GND
- J1 pad 12: unconnected-(J1-Pad12) -> GND
- J1 pad 13: unconnected-(J1-Pad13) -> GND
- J1 pad 14: unconnected-(J1-Pad14) -> GND
- J1 pad 47: unconnected-(J1-Pad47) -> GND
- J1 pad 48: unconnected-(J1-Pad48) -> GND
- J1 pad 49: unconnected-(J1-Pad49) -> GND
- J1 pad 50: unconnected-(J1-Pad50) -> GND
- J1 pad 51: unconnected-(J1-Pad51) -> GND
- J1 pad 52: unconnected-(J1-Pad52) -> GND
- J1 pad 53: unconnected-(J1-Pad53) -> GND
- J1 pad 54: unconnected-(J1-Pad54) -> GND
- J1 pad 55: unconnected-(J1-Pad55) -> GND
- J1 pad 56: unconnected-(J1-Pad56) -> GND
- J1 pad 57: unconnected-(J1-Pad57) -> GND
- J1 pad 58: unconnected-(J1-Pad58) -> GND
- J1 pad 60: unconnected-(J1-Pad60) -> GND
- J2 pad 01: HV_1-64_in -> GND
- J2 pad 02: HV_1-64_in -> GND
- J2 pad 03: unconnected-(J2-Pad03) -> GND
- J2 pad 04: unconnected-(J2-Pad04) -> GND
- J2 pad 05: unconnected-(J2-Pad05) -> GND
- J2 pad 06: unconnected-(J2-Pad06) -> GND
- J2 pad 07: unconnected-(J2-Pad07) -> GND
- J2 pad 08: unconnected-(J2-Pad08) -> GND
- J2 pad 09: unconnected-(J2-Pad09) -> GND
- J2 pad 10: unconnected-(J2-Pad10) -> GND
- J2 pad 11: unconnected-(J2-Pad11) -> GND
- J2 pad 12: unconnected-(J2-Pad12) -> GND
- J2 pad 13: unconnected-(J2-Pad13) -> GND
- J2 pad 14: unconnected-(J2-Pad14) -> GND
- J2 pad 47: unconnected-(J2-Pad47) -> GND
- J2 pad 48: unconnected-(J2-Pad48) -> GND
- J2 pad 49: unconnected-(J2-Pad49) -> GND
- J2 pad 50: unconnected-(J2-Pad50) -> GND
- J2 pad 51: unconnected-(J2-Pad51) -> GND
- J2 pad 52: unconnected-(J2-Pad52) -> GND
- J2 pad 53: unconnected-(J2-Pad53) -> GND
- J2 pad 54: unconnected-(J2-Pad54) -> GND
- J2 pad 55: unconnected-(J2-Pad55) -> GND
- J2 pad 56: unconnected-(J2-Pad56) -> GND
- J2 pad 57: unconnected-(J2-Pad57) -> GND
- J2 pad 58: unconnected-(J2-Pad58) -> GND
- J2 pad 59: unconnected-(J2-Pad59) -> HV_1-64_in
- J2 pad 60: unconnected-(J2-Pad60) -> GND
Routing:
- net Ch_2: track 17.0 -> 3.88 mm
- net Ch_62: track 16.0 -> 3.85 mm
- net Ch_6: track 15.7 -> 3.85 mm
- net Ch_60: track 15.5 -> 3.97 mm
- net Ch_58: track 14.7 -> 3.85 mm
- net Ch_10: track 14.3 -> 3.85 mm
- net Ch_56: track 14.2 -> 3.85 mm
- net Ch_54: track 13.7 -> 3.85 mm
- net Ch_14: track 13.2 -> 3.85 mm
- net Ch_52: track 12.9 -> 3.85 mm
- net Ch_50: track 12.7 -> 3.85 mm
- net Ch_18: track 12.6 -> 3.85 mm
- net Ch_46: track 12.2 -> 3.85 mm
- net Ch_22: track 12.0 -> 3.85 mm
- net Ch_48: track 11.9 -> 3.85 mm
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