File: SmallFiber/SiPM_Array_for_VMM3a_Rev-0/SiPM_Array_for_VMM3a_Rev-0.kicad_sch (KiCad schematic)
At the start: 21 parts, among them J1 ERM6-30-01.5-L-DV-A-K-TR, J2 ERM6-30-01.5-L-DV-A-K-TR

Commit message: .
Other:
- added sheet VoltageControl (VoltageControl.kicad_sch)
- moved on the sheet: C12, C13, C14, C15, C6, C7, C8, C9, H101, H102, H103, H104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

Commit message: .
Other:
- removed sheet VoltageControl
Changed lines of the file:
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@@
-		)
-	)
-	(sheet
-		(at 109.22 203.2)
-		(size 39.37 22.86)
-		(exclude_from_sim no)
-		(in_bom yes)
-		(on_board yes)
-		(dnp no)
-		(fields_autoplaced yes)
-		(stroke
-			(width 0.1524)
-			(type solid)
-		)
-		(fill
-			(color 0 0 0 0.0000)
-		)
-		(property "Sheetname" "VoltageControl"
-			(at 109.22 202.4884 0)
-			(effects
-				(font
-					(size 1.27 1.27)
-				)
-				(justify left bottom)
-			)
-		)
-		(property "Sheetfile" "VoltageControl.kicad_sch"
-			(at 109.22 226.6446 0)
-			(effects
-				(font
-					(size 1.27 1.27)
-				)
-				(justify left top)
-				(hide yes)
-			)
-		)
-		(instances
-			(project "SiPM_Array_for_VMM3a_Rev-0"
-				(path "/0fb97f82-6dac-4756-9e99-da1cf8056c45"
-					(page "2")
-				)
-			)
 		)
 	)
