File: FARICH_new_amplifier/FARICH_Amplifier_v0/FARICH_Amplifier_v0.kicad_pcb (KiCad board)
At the start: 4 copper layers, 15 parts

Commit message: .
Parts:
- removed C1, C3: 4.7n, Capacitor_SMD:C_0402_1005Metric
- removed C2: 100n, Capacitor_SMD:C_0402_1005Metric
- removed C4, C7: 10n, Capacitor_SMD:C_0402_1005Metric
- removed C5, C8, C9: 1p, Capacitor_SMD:C_0402_1005Metric
- removed C6: 2.7p, Capacitor_SMD:C_0402_1005Metric
- removed FB1: FerriteBead_Small, Inductor_SMD:L_0402_1005Metric
- removed L1: 560 nH, Inductor_SMD:L_0402_1005Metric
- removed R1, R3: 150, Resistor_SMD:R_0402_1005Metric
- removed R2: 8.2k, Resistor_SMD:R_0402_1005Metric
- removed U1: ~, FARICH_Amplifier_Library:SOT343F_NXP
- added C201: 4.7n, Capacitor_SMD:C_0201_0603Metric, F.Cu at (98.4, 60.2)
- added C202: 100n, Capacitor_SMD:C_0201_0603Metric, F.Cu at (97.8, 60.2)
- added C203: 4.7n, Capacitor_SMD:C_0201_0603Metric, F.Cu at (99.0, 60.2)
- added C204: 10n, Capacitor_SMD:C_0201_0603Metric, F.Cu at (94.3, 59.1)
- added C205: 1p, Capacitor_SMD:C_0201_0603Metric, F.Cu at (95.0, 59.7)
- added C206: 2.7p, Capacitor_SMD:C_0201_0603Metric, F.Cu at (98.1, 57.7)
- added C207: 10n, Capacitor_SMD:C_0201_0603Metric, F.Cu at (98.4, 59.2)
- added C208: 1p, Capacitor_SMD:C_0201_0603Metric, F.Cu at (99.1, 57.3)
- added C209: 1p, Capacitor_SMD:C_0201_0603Metric, F.Cu at (99.1, 58.5)
- added C210: 4.7n, Capacitor_SMD:C_0201_0603Metric, F.Cu at (105.1, 57.5)
- added C211: 100n, Capacitor_SMD:C_0201_0603Metric, F.Cu at (105.6, 57.5)
- added C212: 4.7n, Capacitor_SMD:C_0201_0603Metric, F.Cu at (104.5, 57.5)
- added C213: 10n, Capacitor_SMD:C_0201_0603Metric, F.Cu at (100.9, 56.3)
- added C214: 1p, Capacitor_SMD:C_0201_0603Metric, F.Cu at (101.6, 57.0)
- added C215: 2.7p, Capacitor_SMD:C_0201_0603Metric, F.Cu at (104.7, 54.9)
- added C216: 10n, Capacitor_SMD:C_0201_0603Metric, F.Cu at (105.1, 56.4)
- added C217: 1p, Capacitor_SMD:C_0201_0603Metric, F.Cu at (105.7, 54.6)
- added C218: 1p, Capacitor_SMD:C_0201_0603Metric, F.Cu at (105.7, 55.8)
- added FB201: FerriteBead_Small, Inductor_SMD:L_0201_0603Metric, F.Cu at (99.6, 59.5)
- added FB202: FerriteBead_Small, Inductor_SMD:L_0201_0603Metric, F.Cu at (106.2, 56.8)
- added L201: 560 nH, Inductor_SMD:L_0402_1005Metric, F.Cu at (97.3, 59.7)
- added L202: 560 nH, Inductor_SMD:L_0402_1005Metric, F.Cu at (103.9, 57.0)
- added R201: 150, Resistor_SMD:R_0201_0603Metric, F.Cu at (94.3, 57.7)
- added R202: 8.2k, Resistor_SMD:R_0201_0603Metric, F.Cu at (96.2, 59.2)
- added R203: 150, Resistor_SMD:R_0201_0603Metric, F.Cu at (99.1, 57.9)
- added R204: 150, Resistor_SMD:R_0201_0603Metric, F.Cu at (100.9, 55.0)
- added R205: 8.2k, Resistor_SMD:R_0201_0603Metric, F.Cu at (102.8, 56.5)
- added R206: 150, Resistor_SMD:R_0201_0603Metric, F.Cu at (105.7, 55.2)
- added U201: ~, FARICH_Amplifier_Library:SOT343F_NXP, F.Cu at (96.3, 58.0)
- added U202: ~, FARICH_Amplifier_Library:SOT343F_NXP, F.Cu at (102.9, 55.2)
Routing:
- net /Amplifier2/1_1V_filtered: track 0.00 -> 3.78 mm
- net /Amplifier/1_1V_filtered: track 0.00 -> 3.78 mm
- net Net-(U202-B): track 0.00 -> 3.69 mm
- net Net-(U201-B): track 0.00 -> 3.69 mm
- net Net-(U202-C): track 0.00 -> 2.68 mm
- net Net-(U201-C): track 0.00 -> 2.68 mm
- net /Amplifier2/1_1V: track 0.00 -> 1.94 mm
- net /Amplifier/1_1V: track 0.00 -> 1.94 mm
- net Ch_2_Out: track 0.00 -> 1.28 mm
- net Ch_1_Out: track 0.00 -> 1.28 mm
- net Ch_1_In: track 0.00 -> 0.71 mm
- net Ch_2_In: track 0.00 -> 0.71 mm
- net GND: vias 7 -> 0
- removed copper zone on F.Cu, net GND
