File: SmallFiber/S13552_64Ch_Adapter_BGA2803/BGA2803_amplifier.kicad_sch (KiCad schematic)
At the start: 7 parts

Commit message: .
Parts:
- renumbered R to R201, U to U201
Changed lines of the file:
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@@
 		(dnp no)
 		(fields_autoplaced yes)
-		(property "Reference" "#PWR"
+		(property "Reference" "#PWR0332"
 			(at 99.06 82.55 0)
 			(effects
@@
 				(path "/0fb97f82-6dac-4756-9e99-da1cf8056c45/2f31a830-26ac-403c-8419-3e8bc72676cb"
 					(reference "#PWR065")
+					(unit 1)
+				)
+				(path "/0fb97f82-6dac-4756-9e99-da1cf8056c45/303476a1-f3d7-4f09-8d8d-90f68a89488e"
+					(reference "#PWR0332")
 					(unit 1)
 				)
@@
 		(on_board yes)
 		(dnp no)
-		(property "Reference" "U"
+		(property "Reference" "U201"
 			(at 104.648 62.484 0)
 			(effects
@@
 				(path "/0fb97f82-6dac-4756-9e99-da1cf8056c45/2f31a830-26ac-403c-8419-3e8bc72676cb"
 					(reference "U13")
+					(unit 1)
+				)
+				(path "/0fb97f82-6dac-4756-9e99-da1cf8056c45/303476a1-f3d7-4f09-8d8d-90f68a89488e"
+					(reference "U201")
 					(unit 1)
 				)
@@
 		(dnp no)
 		(fields_autoplaced yes)
-		(property "Reference" "R"
+		(property "Reference" "R201"
 			(at 124.46 60.9599 0)
 			(effects
@@
 					(unit 1)
 				)
+				(path "/0fb97f82-6dac-4756-9e99-da1cf8056c45/303476a1-f3d7-4f09-8d8d-90f68a89488e"
+					(reference "R201")
+					(unit 1)
+				)

Commit message: .
Other:
- title: Hamamatsu S13552 carrier board -> Hamamatsu S13552 64 Channels Amplifier
Changed lines of the file:
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@@
 	(paper "A5")
 	(title_block
-		(title "Hamamatsu S13552 carrier board")
-		(rev "2")
+		(title "Hamamatsu S13552 64 Channels Amplifier")
+		(date "2025-03-25")
+		(rev "0")
 	)
 	(rectangle

Commit message: .
Other:
- note added: "FARICH Amplifier ref page_48: https://jspc29.x-matter.uni-frankfurt.de/trb/schematics/farich_system.pdf"
- note added: "PADIWA3 Amplifier ref page_4: https://jspc29.x-matter.uni-frankfurt.de/trb/schematics/PADIWA3-all.pdf"
- moved on the sheet: C3, C4, C5, C6, C7, R201, U201

Commit message: .
Other:
- note added: "Other ref: 1. W. Zhi et al 2024 JINST 19 P06011 DOI 10.1088/1748-0221/19/06/P06011 2. Joshua W Cates et al 2018 Phys. Med. Biol. 63 185022 DOI 10.1088/1361-6560/aadbcd 3. F. Simon NIM-A Volume 926, 11 May 2019, Pages 85-100 doi.org/10.1016/j.nima.2018.11.042"
Changed lines of the file:
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@@
 		)
 	)
+	(text "Other ref:\n1. W. Zhi et al 2024 JINST 19 P06011 \nDOI 10.1088/1748-0221/19/06/P06011\n2. Joshua W Cates et al 2018 Phys. Med. Biol. 63 185022\nDOI 10.1088/1361-6560/aadbcd\n3. F. Simon NIM-A Volume 926, 11 May 2019, Pages 85-100\ndoi.org/10.1016/j.nima.2018.11.042"
+		(exclude_from_sim no)
+		(at 17.526 120.65 0)
+		(effects
+			(font
+				(size 1.27 1.27)
+				(thickness 0.254)
+				(bold yes)
+			)
+			(justify left)
+		)
+	)
 	(text "PADIWA3 Amplifier\nref page_4: https://jspc29.x-matter.uni-frankfurt.de/trb/schematics/PADIWA3-all.pdf"
 		(exclude_from_sim no)
@@
 			"AAAAAAAAAAAAAAAAAAAAAAAAAAAAAAAAAAAAAAAAAAAAAAAAAAAAAAAAAAAAAAAAAAAAAAAAAAAA"
 			"AAAAAAAAAAAAAAAAAAAAAAAAAAAAAAAAAAAAAAAAAAAAAAAAAAAAAAAAAAAAAAAAAAAAAAAAAAAA"
-			"AAAAAAAAAAAAAAAAAAAAAAAAAAAAAAAAAA=="
+			"AAAAAAAAAAAAAAAAAAAAAAAAAAAAAAAAADYAeABwADgAQgBEADcARQBhAHIAYgBWAEUAcABXAHkA"
+			"dwBwAGoAaQBLAEQASgBzAEIARABiAFYAMQAvAFMAUwB2AFgAZQBCAGoATQBsAEIANwBWADIAMwBm"
+			"ADkAMwB6AHkASQBQAGcAVgBBAHMANgBHAFQAYQBNAEsAWgBGAFkAMwB0AGUAdwArAFAAZgBkAG0A"
+			"cABZADYAOQBCAGEAaQBMAFUAQQBCAHoAZAAwAFQAKwBuAGMAawBmAGUAdgBDADMAQwBBAG4AagAy"
+			"AE0AUQBhAG8AWAB6AHgAMgBQAHkANgArAGMAZAB3AG4AWABZAGgAMgBhAEYAQgB0AEcAdwBSAEIA"
+			"QQBDAGwAbwB5AEcATQBOAFoASwBFAHYATgBYAFAAQgBpAGcAKwBBAEcAVgBVAHgAbwBtAGcARwBS"
+			"AGgANQBwACsAdABHAFAAZgB0ADEAdgBuAFQASQB0ADAAYwA0AHMASgAvAEMAeQA3AGUAZAB1AHgA"
+			"ZgBFAEgAZQAxAEcAVwBSAHcAOQBrAFMAdwBzAHUARABiAEQAeQAvAGIAcgA5ADkASQBtAGoAaABi"
+			"AFoAcwBGAEIASABDAGoAawBHAHAARgBIAEMAbABmADAALwB1ADQAZABmAGUAOQBSAFQAKwB6AGUA"
+			"ZgAyAHoAVgBSADkAbABQAGEAZgA4AEMAQwBGADMASwBRAFMAUgAyAEMAZQBQAEIAVwBqAHMAagBE"
+			"ACsAcABzACsANwA1AEkAZgB4AGwALwArAEIAcQB3AFgATQB5AHkASAA2AFkAMwB1AE8AWAB0ADIA"
+			"KwBGADgAcwBuADkAbQBEADUAaABQADkAegBkAEQAbwBHAG4AYQBwAEEASwBRAGoANABjAFQAegBu"
+			"ADkATABxAEwAVwByAGoANwAwAGYASABHAFEANQBHAEEAawBIAEgAOQBjADgAZQBWAEEAeQBZAGkA"
+			"dgBQAE4ATgBLADIATQBNAHUAbgBUAEQATwBGAGsAbgA0AE4AUgBwAHoAUgBuAFQASAB1AFAANQBZ"
+			"ADkAZgBpAFIAZgBlACsAbAAyAC8ATABtAG0ARwBEADMALwBlAFAANQBSAGUAdQBjAEIAOQBMAE8A"
+			"SABWAGkARwBiAHMAdQBPAEQAZwBhAGcAMgBwAEMARwBGAHIAVQA1AGwAMgBRAEIAbwAzAEsAcAB1"
+			"ACsAZAB1AFoAZABkAGUAeABLAFkAcwBTAFAAMwBnADcALwAyAG8ATQBlAGMAaQBuAFMAaABZAEEA"
+			"egBoADkATABMAEoASgBrADgATQBIADYAYQBFAFMAUwA4AGgAZwBRAEEAQQBJAEEAQgBKAFIARQBG"
+			"AFUAWgB4ADcAcQBHAGMAKwBYAGIAYwB2AA=="
 		)
 	)
@@
 			"vwAAAABR7zVCu5WbwQAAgD9qaCK/WONFvwAAAABR7zVCu5WbwQAAAABqaCK/WONFvwAAAADvsjVC"
 			"CUWbwQAAgD9lWvG+vMVhvwAAAADvsjVCCUWbwQAAAABlWvG+vMVhvwAAAADWbzVCdA2bwQAAgD/n"
-			"npQ="
+			"npQAAAAAAAAAAAAAAAAAAAAAAAAAAAAAAAAAAAAAAAAAAAAAAAAAAAAAAAAAAAAAAAAAAAAAAAAA"
+			"AAAAAAAAAAAAAAAAAAAAAAAAAAAAAAAAAAAAAAAAAAAAAAAAAAAAAAAAAAAAAAAAAAAAAAAAAAAA"
+			"AAAAAAAAAAAAAAAAAAAAAAAAAAAAAAAAAAAAAAAAAAAAAAAAAAAAAAAAAAAAAAAAAAAAAAAAAAAA"
+			"AAAAAAAAAAAAAAAAAAAAAAAAAAAAAAAAAAAAAAAAAAAAAAAAAAAAAAAAAAAAAAAAAAAAAAAAAAAA"
+			"AAAAAAAAAAAAAAAAAAAAAAAAAAAAAAAAAAAAAAAAAAAAAAAAAAAAAAAAAAAAAAAAAAAAAAAAAAAA"
+			"AAAAAAAAAAAAAAAAAAAAAAAAAAAAAAAAAAAAAAAAAAAAAAAAAAAAAAAAAAAAAAAAAAAAAAAAAAAA"
+			"AAAAAAAAAAAAAAAAAAAAAAAAAAAAAAAAAAAAAAAAAAAAAAAAAAAAAAAAAAAAAAAAAAAAAAAAAAAA"
+			"AAAAAAAAAAAAAAAAAAAAAAAAAAAAAAAAAAAAAAAAAAAAAAAAAAAAAAAAAAAAAAAAAAAAAAAAAAAA"
+			"AAAAAAAAAAAAAAAAAAAAAAAAAAAAAAAAAAAAAAAAAAAAAAAAAAAAAAAAAAAAAAAAAAAAAAAAAAAA"
+			"AAAAAAAAAAAAAAAAAAAAAAAAAAAAAAAAAAAAAAAAAAAAAAAAAAAAAAAAAAAAAAAAAAAAAAAAAAAA"
+			"AAAAAAAAAAAAAAAAAAAAAAAAAAAAAAAAAAAAAAAAAAAAAAAAAAAAAAAAAAAAAAAAAAAAAAAAAAAA"
+			"AAAAAAAAAAAAAAAAAAAAAAAAAAAAAAAAAAAAAAAAAAAAAAAAAAAAAAAAAAAAAAAAAAAAAAAAAAAA"
+			"AAAAAAAAAAAAAAAAAAAAAAAAAAAAAAAAAAAAAAAAAAAAAAAAAAAAAAAAAAAAAAAAAAAAAAAAAAAA"
+			"AAAAAAAAAAAAAAAAAAAAAAAAAAAAAAAAAAAAAAAAAAAAAAAAAAAAAAAAAAAAAAAAAAAAAAAAAAAA"
+			"AAAAAAAAAAAAAAAAAAAAAAAAAAAAAAAAAAAAAAAAAAAAAAAAAAAAAAAAAAAAAAAAAAAAAAAAAAAA"
+			"AAAAAAAAAAAAAAAAAAAAAAAAAAAAAAAAAAAAAAAAAAAAAAAAAAAAAAAAAAAAAAAAAAAAAAAAAAAA"
+			"AAAAAAAAAAAAAAAAAAAAAAAAAAAAAAAAAAAAAAAAAAAAAAAAAAAAAAAAAAAAAAAAAAAAAAAAAAAA"
+			"AAAAAAAAAAAAAAAAAAAAAAAAAAAAAAAAAAAAAAAAAAAAAAAAAAAAAAAAAAAAAAAAAAAAAAAAAAAA"
+			"AA=="
 		)
 	)
