File: SmallFiber/Demo_board_bga2803/BGA2803_amplifier.kicad_sch (KiCad schematic)
At the start: 7 parts, among them U14 BGA2803

Commit message: .
Parts:
- renumbered C58 to C63, C59 to C64, C60 to C65, C61 to C66, C62 to C67, R16 to R17
