File: SmallFiber/Demo_board_bga2803/Demo_board_bga2803.kicad_sch (KiCad schematic)
At the start: 10 parts, among them J1 12401945E212A, U1 NCP1117-3.3_SOT223, U2 TLV1117LV12DCYR

Commit message: .
Parts:
- added J101, J103: Input_1, Connector_Coaxial:SMA_Amphenol_132289_EdgeMount, symbol Connector:Conn_Coaxial_Small
- added J102, J104: Output_1, Connector_Coaxial:SMA_Amphenol_132289_EdgeMount, symbol Connector:Conn_Coaxial_Small
- U2: footprint (none) -> Package_TO_SOT_SMD:SOT-223-3_TabPin2
Connections:
- net Amp_1/In: now also J101.1 (In)
- net Amp_1/Out: now also J102.1 (In)
- net GND: now also J101.2 (Ext), J102.2 (Ext), J103.2 (Ext), J104.2 (Ext)
- net +1V1: now reaches U2.2 (VO)
- new net Amp_2/In: J103.1 (In)
- new net Amp_2/Out: J104.1 (In)
Other:
- added sheet Amp_2 (BGA2803_amplifier.kicad_sch)

Commit message: .
Parts:
- removed L1: L_Iron_Small, symbol Device:L_Iron_Small
- removed U1: NCP1117-3.3_SOT223, Package_TO_SOT_SMD:SOT-223-3_TabPin2, symbol Regulator_Linear:NCP1117-3.3_SOT223
- removed U2: TLV1117LV12DCYR, Package_TO_SOT_SMD:SOT-223-3_TabPin2, symbol Regulator_Linear:TLV1117-15
- added A1, A2: MICROFC-10035-SMT-TR1, 0_lib:XDCR_MICROFC-10035-SMT-TR1, symbol 0_SiPM:MICROFC-10035-SMT-TR1
- added C11, C12: 10nF/50V, Capacitor_SMD:C_0603_1608Metric, symbol Device:C
- added D2: LED, LED_SMD:LED_0603_1608Metric, symbol Device:LED
- added J2, J5: sig_out, 0_lib:IPEX_20449-001E-03, symbol Connector:Conn_Coaxial_Small
- added J3: HV_Out, 0_lib:IPEX_20449-001E-03, symbol Connector:Conn_Coaxial_Small
- added J4: HV, 0_lib:IPEX_20449-001E-03, symbol Connector:Conn_Coaxial_Small
- added R10, R11, R2, R3: 10k, Resistor_SMD:R_0402_1005Metric, symbol Device:R
- added R4: 600, Resistor_SMD:R_0402_1005Metric, symbol Device:R
- added U1, U2: ~, Package_TO_SOT_SMD:SOT-23-5, symbol 0_USB-C:TPS7A2033PDBVR
- C1, C2: value C -> 1u; footprint (none) -> Capacitor_SMD:C_0402_1005Metric
- C3, C4: value 10u -> 1u; footprint (none) -> Capacitor_SMD:C_0402_1005Metric; Mnf. nr. TAJC106K035RNJ -> (none)
- D1: footprint (none) -> LED_SMD:LED_0603_1608Metric
- R1: value R -> 600; footprint (none) -> Resistor_SMD:R_0402_1005Metric
Connections:
- net +1V1: now also C4.1, D2.2 (A), U2.5 (Out)
- net +3V3: now also U1.5 (Out)
- net +5V: now also C1.1, R2.1, R3.1, U1.1 (In), U2.1 (In)
- net GND: now also C11.2, C12.2, J2.2 (Ext), J3.2 (Ext), J4.2 (Ext), J5.2 (Ext), R4.2, U1.2 (GND), U2.2 (GND); no longer J1.SH3_1 (SHIELD__2), J1.SH3_2 (SHIELD__3), J1.SH3_3 (SHIELD__4), J1.SH3_4 (SHIELD__5), J1.SH4_1 (SHIELD__6), J1.SH4_2 (SHIELD__7), J1.SH4_3 (SHIELD__8), J1.SH4_4 (SHIELD__9)
- new net: A1.1, J2.1 (In)
- new net: A1.3, C11.1, R10.2
- new net: R2.2, U1.3 (EN)
- new net: A2.1, J5.1 (In)
- new net: A2.3, C12.1, R11.2
- new net: J4.1 (In), R10.1, R11.1
- new net: R3.2, U2.3 (EN)
- new net: D2.1 (K), R4.1
- new net HV_PSU/HV: J3.1 (In)
- no-connect marks 16 -> 20
Other:
- added sheet HV_PSU (HV_PSU_33.75V.kicad_sch)
- moved on the sheet: D1, R1
