File: SmallFiber/S13552_64Ch_Adapter_BGA2803_V2/S13552_64Ch_Adapter_BGA2803_V2.kicad_sch (KiCad schematic)
At the start: 11 parts, among them J1 ERM6-30-01.5-L-DV-A-K-TR, J2 ERM6-30-01.5-L-DV-A-K-TR

Commit message: .
Connections:
- net GND: no longer J1.01, J1.03, J1.04, J1.05, J1.06, J1.07, J1.08, J1.09, J1.10, J1.11, J1.12, J1.13, J1.14, J1.47, J1.48, J1.49, J1.50, J1.51, J1.52, J1.53, J1.54, J1.55, J1.56, J1.57, J1.58, J1.59, J1.60, J2.01, J2.02, J2.03, J2.04, J2.05, J2.06, J2.07, J2.08, J2.09, J2.10, J2.11, J2.12, J2.13, J2.14, J2.47, J2.48, J2.49, J2.50, J2.51, J2.52, J2.53, J2.54, J2.55, J2.56, J2.57, J2.58, J2.60
- net out_Ch_64: now reaches J1.16
- net out_Ch_56: now reaches J1.18
- net out_Ch_48: now reaches J1.19
- net out_Ch_48: now also J1.22
- net out_Ch_58: now reaches J1.20
- net out_Ch_40: now reaches J1.23
- net out_Ch_52: now reaches J1.24
- net out_Ch_42: now reaches J1.26
- net out_Ch_34: now reaches J1.27
- net out_Ch_46: now reaches J1.28
- net out_Ch_32: now reaches J1.30
- net out_Ch_26: now reaches J1.31
- net out_Ch_38: now reaches J1.32
- net out_Ch_22: now reaches J1.34
- net out_Ch_20: now reaches J1.35
- net out_Ch_28: now reaches J1.36
- net out_Ch_12: now reaches J1.38
- net out_Ch_18: now reaches J1.40
- net out_Ch_6: now reaches J1.42
- net out_Ch_10: now reaches J1.44
- net out_Ch_2: now reaches J1.46
- new net out_Ch_4: J1.48
- new net out_Ch_62: J1.14
