File: SmallFiber/S13552_64Ch_Adapter_BGA2803_V2/S13552_64Ch_Adapter_BGA2803_V2.kicad_sch (KiCad schematic)
At the start: 11 parts, among them J1 ERM6-30-01.5-L-DV-A-K-TR, J2 ERM6-30-01.5-L-DV-A-K-TR

Commit message: .
Parts:
- added C323, C324, C325, C326, C327, C328, C329, C330, C331, C332, C333, C334, C335, C336, C337, C338, C339, C340, C341, C342: 100nF, Capacitor_SMD:C_0402_1005Metric, symbol Device:C
Connections:
- net GND: now also J1.01, J1.03, J1.04, J1.06, J1.08, J1.10, J1.12, J1.13, J1.43, J1.45, J1.50, J1.52, J1.54, J1.56, J1.57, J1.58, J1.59, J1.60, J2.01, J2.02, J2.03, J2.04, J2.05, J2.07, J2.09, J2.11, J2.16, J2.18, J2.48, J2.49, J2.51, J2.53, J2.55, J2.57, J2.58, J2.60, C323.2, C324.2, C325.2, C326.2, C327.2, C328.2, C329.2, C330.2, C331.2, C332.2, C333.2, C334.2, C335.2, C336.2, C337.2, C338.2, C339.2, C340.2, C341.2, C342.2
- net out_Ch_13: now also J2.44
- net out_Ch_15: now also J2.39
- net out_Ch_19: now also J2.42
- net out_Ch_21: now also J2.40
- net out_Ch_23: now also J2.35
- net out_Ch_25: now also J2.38
- net out_Ch_29: now also J2.36
- net out_Ch_3: now also J2.47
- net out_Ch_31: now also J2.34
- net out_Ch_33: now also J2.31
- net out_Ch_35: now also J2.32
- net out_Ch_39: now also J2.30
- net out_Ch_41: now also J2.28
- net out_Ch_43: now also J2.27
- net out_Ch_45: now also J2.26
- net out_Ch_48: no longer J1.22
- net out_Ch_49: now also J2.24
- net out_Ch_5: now also J2.46
- net out_Ch_51: now also J2.22
- net out_Ch_53: now also J2.23
- net out_Ch_57: now also J2.19
- net out_Ch_59: now also J2.20
- net out_Ch_63: now also J2.15
- net out_Ch_9: now also J2.43
- net +1V1: now reaches J1.05
- net +1V1: now also J1.07, J1.09, J1.11, J2.50, J2.52, J2.54, J2.56, C323.1, C324.1, C325.1, C326.1, C327.1, C328.1, C329.1, C330.1, C331.1, C332.1, C333.1, C334.1, C335.1, C336.1, C337.1, C338.1, C339.1, C340.1, C341.1, C342.1
- net +3V3: now reaches J1.47
- net +3V3: now also J1.49, J1.51, J1.53, J1.55, J2.06, J2.08, J2.10, J2.12, J2.14
- new net out_Ch_50: J1.22
Other:
- moved on the sheet: J2

Commit message: .
Parts:
- added FID1, FID2, FID3, FID4, FID5, FID6: Fiducial, Fiducial:Fiducial_0.5mm_Mask1mm, symbol Mechanical:Fiducial
