File: SmallFiber/S13552_64Ch_Adapter_BGA2803_V2/PCB_Stackup.kicad_sch (KiCad schematic)
At the start: 0 parts

Commit message: .
Changed lines of the file:
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@@
 	(text "PCB Stackup"
 		(exclude_from_sim no)
-		(at 31.242 100.838 0)
+		(at 31.242 105.41 0)
 		(effects
 			(font
@@
 		)
 		(column_widths 8.89 17.78)
-		(row_heights 2.54 2.54 2.54 2.54 2.54 2.54 2.54 2.54)
+		(row_heights 2.54 2.54 2.54 2.54 2.54 2.54 2.54 2.54 2.54 2.54)
 		(cells
 			(table_cell "Top"
@@
 				)
 			)
-			(table_cell "Power 3V3/1V1"
+			(table_cell "Power 3V3"
 				(exclude_from_sim no)
 				(at 26.67 87.63 0)
@@
 				(fill
 					(type color)
+					(color 255 122 120 1)
+				)
+				(effects
+					(font
+						(size 1.27 1.27)
+					)
+				)
+			)
+			(table_cell "1V1"
+				(exclude_from_sim no)
+				(at 26.67 92.71 0)
+				(size 17.78 2.54)
+				(margins 0.9525 0.9525 0.9525 0.9525)
+				(span 1 1)
+				(fill
+					(type color)
+					(color 255 122 120 1)
+				)
+				(effects
+					(font
+						(size 1.27 1.27)
+					)
+				)
+			)
+			(table_cell "Inner_7"
+				(exclude_from_sim no)
+				(at 17.78 95.25 0)
+				(size 8.89 2.54)
+				(margins 0.9525 0.9525 0.9525 0.9525)
+				(span 1 1)
+				(fill
+					(type color)
 					(color 12 255 191 1)
 				)
@@
 			(table_cell "Ground"
 				(exclude_from_sim no)
-				(at 26.67 92.71 0)
+				(at 26.67 95.25 0)
+				(size 17.78 2.54)
+				(margins 0.9525 0.9525 0.9525 0.9525)
+				(span 1 1)
+				(fill
+					(type color)
+					(color 12 255 191 1)
+				)
+				(effects
+					(font
+						(size 1.27 1.27)
+					)
+				)
+			)
+			(table_cell "Inner_8"
+				(exclude_from_sim no)
+				(at 17.78 97.79 0)
+				(size 8.89 2.54)
+				(margins 0.9525 0.9525 0.9525 0.9525)
+				(span 1 1)
+				(fill
+					(type color)
+					(color 12 255 191 1)
+				)
+				(effects
+					(font
+						(size 1.27 1.27)
+					)
+				)
+			)
+			(table_cell "Ground"
+				(exclude_from_sim no)
+				(at 26.67 97.79 0)
 				(size 17.78 2.54)
 				(margins 0.9525 0.9525 0.9525 0.9525)
@@
 			(table_cell "Bottom"
 				(exclude_from_sim no)
-				(at 17.78 95.25 0)
+				(at 17.78 100.33 0)
 				(size 8.89 2.54)
 				(margins 0.9525 0.9525 0.9525 0.9525)
@@
 			(table_cell "Signal"
 				(exclude_from_sim no)
-				(at 26.67 95.25 0)
+				(at 26.67 100.33 0)
 				(size 17.78 2.54)
 				(margins 0.9525 0.9525 0.9525 0.9525)
