File: HV_MPPC_Ballance/Prototype/HV_MPPC_Ballance_prototype/1_ch_ltc6090.kicad_sch (KiCad schematic)
At the start: 4 parts, among them U1 LTC6090CS8E-5-PBF

Commit message: .
Parts:
- added C11, C12: 100n/100V, Capacitor_SMD:C_0805_2012Metric, symbol Device:C
- added C13, C14: 100n, Capacitor_SMD:C_0603_1608Metric, symbol Device:C
- added C15: 100n/100V, Capacitor_SMD:C_0603_1608Metric, symbol Device:C
- R1: footprint (none) -> Resistor_SMD:R_0805_2012Metric
- R2, R3: footprint (none) -> Resistor_SMD:R_0603_1608Metric
- U1: footprint SO-8_S_LIT -> 0_lib:SO-8_S_LIT
Connections:
- net -5V: now also C13.1
- net DAC: now also C14.1
- net GND: now also C11.2, C12.2, C13.2, C14.2
- net HV_in: now also C12.1
- net Out: now also C11.1
- net at R2.1, R3.2, U1.2 (-IN): now also C15.1
- net at R1.1, R2.2, U1.6 (OUT): now also C15.2
Other:
- note added: "!in case of unstability populate this capacitor"
- moved on the sheet: R3
