File: HV_MPPC_Ballance/Prototype/HV_MPPC_Ballance_prototype/HV_MPPC_Ballance_prototype.kicad_sch (KiCad schematic)
At the start: 46 parts, among them J1 Conn_02x05_Odd_Even, J2 TPS7A2033PDBVR, J3 12401945E212A, J4 IPL1-102-01-X-D-RA-K, J5 IPL1-102-01-X-D-RA-K, J6 IPL1-102-01-X-D-RA-K, J7 IPL1-102-01-X-D-RA-K, J8 IPL1-102-01-X-D-RA-K, U2 MCP47FEB08-20E/ST, U9 ADP5600ACPZ-R7

Commit message: I2C Python communication
Python firmware for RP2040 to control the DAC via SPI, there is also an app with UI and monitoring.
Parts:
- U2: value MCP47FEB08-20E/ST -> MCP47FEB28
