File: Main_Board/Main_Board_REV_0/Microcontroller.kicad_sch (KiCad schematic)
At the start: 3 parts, among them J17 RJHSE538002, J18 430450200, J19 UJ20-C-R-G-TH-P14

Commit message: .
Parts:
- added J20: 60612202111307, symbol Connector:Conn_Coaxial_Small
Changed lines of the file:
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@@
 	(paper "A4")
+	(symbol
+		(lib_id "Connector:Conn_Coaxial_Small")
+		(at 72.39 170.18 0)
+		(unit 1)
+		(exclude_from_sim no)
+		(in_bom yes)
+		(on_board yes)
+		(dnp no)
+		(fields_autoplaced yes)
+		(property "Reference" "J20"
+			(at 71.8704 163.83 0)
+			(effects
+				(font
+					(size 1.27 1.27)
+				)
+			)
+		)
+		(property "Value" "60612202111307"
+			(at 71.8704 166.37 0)
+			(effects
+				(font
+					(size 1.27 1.27)
+				)
+			)
+		)
+		(property "Footprint" ""
+			(at 72.39 170.18 0)
+			(effects
+				(font
+					(size 1.27 1.27)
+				)
+				(hide yes)
+			)
+		)
+		(property "Datasheet" "~"
+			(at 72.39 170.18 0)
+			(effects
+				(font
+					(size 1.27 1.27)
+				)
+				(hide yes)
+			)
+		)
+		(property "Description" "small coaxial connector (BNC, SMA, SMB, SMC, Cinch/RCA, LEMO, ...)"
+			(at 72.39 170.18 0)
+			(effects
+				(font
+					(size 1.27 1.27)
+				)
+				(hide yes)
+			)
+		)
+		(pin "2"
+		)
+		(pin "1"
+		)
+		(instances
+			(project ""
+				(path "/7125c2d5-be96-492e-8b70-c56cceaf676d/2f51ce8a-6831-403a-819e-2c739fb15ce3"
+					(reference "J20")
+					(unit 1)
+				)
+			)
+		)
+	)
 	(symbol
 		(lib_id "0-lib:430450200")

Commit message: .
Parts:
- J20: footprint (none) -> 0-lib:60612202111307
Changed lines of the file:
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@@
 			)
 		)
-		(property "Footprint" ""
+		(property "Footprint" "0-lib:60612202111307"
 			(at 72.39 170.18 0)
 			(effects
