File: Main_Board/Main_Board_REV_0/Main_Board_REV_0.kicad_sch (KiCad schematic)
At the start: 73 parts, among them J1 ERF6-30-03.5-L-DV-A-K-TR, J10 ERF6-30-03.5-L-DV-A-K-TR, J11 ERF6-30-03.5-L-DV-A-K-TR, J12 ERF6-30-03.5-L-DV-A-K-TR, J13 ERF6-30-03.5-L-DV-A-K-TR, J14 ERF6-30-03.5-L-DV-A-K-TR, J15 ERF6-30-03.5-L-DV-A-K-TR, J16 ERF6-30-03.5-L-DV-A-K-TR, J17 1778764, J18 NCP1117LPST33T3G, J19 Conn_02x16_Odd_Even, J2 ERF6-30-03.5-L-DV-A-K-TR, J20 NCP1117LPST33T3G, J21 NCP1117LPST33T3G, J22 NCP1117LPST33T3G, J23 Amphenol_132289, J3 ERF6-30-03.5-L-DV-A-K-TR, J4 ERF6-30-03.5-L-DV-A-K-TR, J5 ERF6-30-03.5-L-DV-A-K-TR, J6 ERF6-30-03.5-L-DV-A-K-TR, J7 ERF6-30-03.5-L-DV-A-K-TR, J8 ERF6-30-03.5-L-DV-A-K-TR, J9 ERF6-30-03.5-L-DV-A-K-TR

Commit message: .
Parts:
- added TP14: 1V1_A3, TestPoint:TestPoint_Pad_1.0x1.0mm, symbol Connector:TestPoint
Connections:
- net 1V1_Cube_5 is gone; now on net 1V1_A3: J13.43, J13.44, J13.47, J13.48, J13.51, J13.52, J13.55, J13.56, J15.43, J15.44, J15.47, J15.48, J15.51, J15.52, J15.55, J15.56
- net Out_A1_Cube_1 is gone; now on net Ch_37_A2: J10.54
- net Out_A1_Cube_2 is gone; now on net Ch_36_A2: J12.54
- net Out_A1_Cube_5 is gone; now on net Ch_44_A4: J15.54
- net Out_A1_Cube_6 is gone; now on net Ch_37_A4: J16.54
- net Out_A2_Cube_1 is gone; now on net Ch_53_A2: J10.50
- net Out_A2_Cube_2 is gone; now on net Ch_40_A2: J12.50
- net Out_A2_Cube_5 is gone; now on net Ch_48_A4: J15.50
- net Out_A2_Cube_6 is gone; now on net Ch_53_A4: J16.50
- net Out_A3_Cube_1 is gone; now on net Ch_63_A2: J10.58
- net Out_A3_Cube_2 is gone; now on net Ch_34_A2: J12.58
- net Out_A3_Cube_5 is gone; now on net Ch_40_A4: J15.58
- net Out_A3_Cube_6 is gone; now on net Ch_43_A4: J16.58
- net Out_A4_Cube_1 is gone; now on net Ch_57_A2: J10.42
- net Out_A4_Cube_2 is gone; now on net Ch_54_A2: J12.42
- net Out_A4_Cube_5 is gone; now on net Ch_60_A4: J15.42
- net Out_A4_Cube_6 is gone; now on net Ch_57_A4: J16.42
- net Out_A5_Cube_5 is gone; now on net Ch_28_A3: J13.25
- net Out_A5_Cube_6 is gone; now on net Ch_63_A3: J14.25
- net Out_A6_Cube_1 is gone; now on net Ch_43_A2: J10.25
- net Out_A6_Cube_2 is gone; now on net Ch_28_A2: J12.25
- net Out_A6_Cube_5 is gone; now on net Ch_28_A4: J15.25
- net Out_A6_Cube_6 is gone; now on net Ch_31_A4: J16.25
- net Out_A7_Cube_1 is gone; now on net Ch_27_A2: J10.21
- net Out_A7_Cube_2 is gone; now on net Ch_12_A2: J12.21
- net Out_A7_Cube_5 is gone; now on net Ch_12_A4: J15.21
- net Out_A7_Cube_6 is gone; now on net Ch_29_A4: J16.21
- net Out_A8_Cube_1 is gone; now on net Ch_35_A2: J10.10
- net Out_A8_Cube_2 is gone; now on net Ch_32_A2: J12.10
- net Out_A8_Cube_5 is gone; now on net Ch_46_A4: J15.10
- net Out_A8_Cube_6 is gone; now on net Ch_41_A4: J16.10
- net Out_B1_Cube_1 is gone; now on net Ch_01_A2: J10.57
- net Out_B1_Cube_2 is gone; now on net Ch_14_A2: J12.57
- net Out_B1_Cube_5 is gone; now on net Ch_14_A4: J15.57
- net Out_B1_Cube_6 is gone; now on net Ch_01_A4: J16.57
- net Out_B2_Cube_1 is gone; now on net Ch_49_A2: J10.30
- net Out_B2_Cube_2 is gone; now on net Ch_58_A2: J12.30
- net Out_B2_Cube_5 is gone; now on net Ch_56_A4: J15.30
- net Out_B2_Cube_6 is gone; now on net Ch_61_A4: J16.30
- net Out_B3_Cube_1 is gone; now on net Ch_47_A2: J10.46
- net Out_B3_Cube_2 is gone; now on net Ch_44_A2: J12.46
- net Out_B3_Cube_5 is gone; now on net Ch_54_A4: J15.46
- net Out_B3_Cube_6 is gone; now on net Ch_47_A4: J16.46
- net Out_B4_Cube_1 is gone; now on net Ch_11_A2: J10.41
- net Out_B4_Cube_2 is gone; now on net Ch_26_A2: J12.41
- net Out_B4_Cube_5 is gone; now on net Ch_26_A4: J15.41
- net Out_B4_Cube_6 is gone; now on net Ch_11_A4: J16.41
- net Out_B5_Cube_1 is gone; now on net Ch_51_A2: J10.26
- net Out_B5_Cube_2 is gone; now on net Ch_50_A2: J12.26
- net Out_B5_Cube_5 is gone; now on net Ch_58_A4: J15.26
- net Out_B5_Cube_6 is gone; now on net Ch_59_A4: J16.26
- net Out_B6_Cube_1 is gone; now on net Ch_33_A2: J10.29
- net Out_B6_Cube_2 is gone; now on net Ch_22_A2: J12.29
- net Out_B6_Cube_5 is gone; now on net Ch_22_A4: J15.29
- net Out_B6_Cube_6 is gone; now on net Ch_33_A4: J16.29
- net Out_B7_Cube_1 is gone; now on net Ch_39_A2: J10.14
- net Out_B7_Cube_2 is gone; now on net Ch_46_A2: J12.14
- net Out_B7_Cube_5 is gone; now on net Ch_42_A4: J15.14
- net Out_B7_Cube_6 is gone; now on net Ch_45_A4: J16.14
- net Out_B8_Cube_1 is gone; now on net Ch_13_A2: J10.05
- net Out_B8_Cube_2 is gone; now on net Ch_02_A2: J12.05
- net Out_B8_Cube_5 is gone; now on net Ch_02_A4: J15.05
- net Out_B8_Cube_6 is gone; now on net Ch_13_A4: J16.05
- net Out_C1_Cube_1 is gone; now on net Ch_09_A2: J10.53
- net Out_C1_Cube_2 is gone; now on net Ch_16_A2: J12.53
- net Out_C1_Cube_5 is gone; now on net Ch_16_A4: J15.53
- net Out_C1_Cube_6 is gone; now on net Ch_09_A4: J16.53
- net Out_C2_Cube_1 is gone; now on net Ch_23_A2: J10.37
- net Out_C2_Cube_2 is gone; now on net Ch_30_A2: J12.37
- net Out_C2_Cube_5 is gone; now on net Ch_30_A4: J15.37
- net Out_C2_Cube_6 is gone; now on net Ch_23_A4: J16.37
- net Out_C3_Cube_1 is gone; now on net Ch_55_A2: J10.38
- net Out_C3_Cube_2 is gone; now on net Ch_48_A2: J12.38
- net Out_C3_Cube_5 is gone; now on net Ch_62_A4: J15.38
- net Out_C3_Cube_6 is gone; now on net Ch_55_A4: J16.38
- net Out_C4_Cube_1 is gone; now on net Ch_45_A2: J10.34
- net Out_C4_Cube_2 is gone; now on net Ch_56_A2: J12.34
- net Out_C4_Cube_5 is gone; now on net Ch_64_A4: J15.34
- net Out_C4_Cube_6 is gone; now on net Ch_63_A4: J16.34
- net Out_C5_Cube_1 is gone; now on net Ch_17_A2: J10.33
- net Out_C5_Cube_2 is gone; now on net Ch_38_A2: J12.33
- net Out_C5_Cube_5 is gone; now on net Ch_34_A4: J15.33
- net Out_C5_Cube_6 is gone; now on net Ch_17_A4: J16.33
- net Out_C6_Cube_1 is gone; now on net Ch_21_A2: J10.13
- net Out_C6_Cube_2 is gone; now on net Ch_06_A2: J12.13
- net Out_C6_Cube_5 is gone; now on net Ch_06_A4: J15.13
- net Out_C6_Cube_6 is gone; now on net Ch_21_A4: J16.13
- net Out_C7_Cube_1 is gone; now on net Ch_41_A2: J10.18
- net Out_C7_Cube_2 is gone; now on net Ch_42_A2: J12.18
- net Out_C7_Cube_5 is gone; now on net Ch_52_A4: J15.18
- net Out_C7_Cube_6 is gone; now on net Ch_49_A4: J16.18
- net Out_C8_Cube_1 is gone; now on net Ch_29_A2: J10.02
- net Out_C8_Cube_2 is gone; now on net Ch_62_A2: J12.02
- net Out_C8_Cube_5 is gone; now on net Ch_38_A4: J15.02
- net Out_C8_Cube_6 is gone; now on net Ch_35_A4: J16.02
- net Out_D1_Cube_1 is gone; now on net Ch_03_A2: J10.59
- net Out_D1_Cube_2 is gone; now on net Ch_08_A2: J12.59
- net Out_D1_Cube_5 is gone; now on net Ch_08_A4: J15.59
- net Out_D1_Cube_6 is gone; now on net Ch_03_A4: J16.59
- net Out_D2_Cube_1 is gone; now on net Ch_07_A2: J10.49
- net Out_D2_Cube_2 is gone; now on net Ch_20_A2: J12.49
- net Out_D2_Cube_5 is gone; now on net Ch_20_A4: J15.49
- net Out_D2_Cube_6 is gone; now on net Ch_07_A4: J16.49
- net Out_D3_Cube_1 is gone; now on net Ch_15_A2: J10.45
- net Out_D3_Cube_2 is gone; now on net Ch_24_A2: J12.45
- net Out_D3_Cube_5 is gone; now on net Ch_24_A4: J15.45
- net Out_D3_Cube_6 is gone; now on net Ch_15_A4: J16.45
- net Out_D4_Cube_1 is gone; now on net Ch_61_A2: J10.60
- net Out_D4_Cube_2 is gone; now on net Ch_60_A2: J12.60
- net Out_D4_Cube_5 is gone; now on net Ch_36_A4: J15.60
- net Out_D4_Cube_6 is gone; now on net Ch_27_A4: J16.60
- net Out_D5_Cube_1 is gone; now on net Ch_25_A2: J10.17
- net Out_D5_Cube_2 is gone; now on net Ch_18_A2: J12.17
- net Out_D5_Cube_5 is gone; now on net Ch_18_A4: J15.17
- net Out_D5_Cube_6 is gone; now on net Ch_25_A4: J16.17
- net Out_D6_Cube_1 is gone; now on net Ch_05_A2: J10.01
- net Out_D6_Cube_2 is gone; now on net Ch_04_A2: J12.01
- net Out_D6_Cube_5 is gone; now on net Ch_04_A4: J15.01
- net Out_D6_Cube_6 is gone; now on net Ch_05_A4: J16.01
- net Out_D7_Cube_1 is gone; now on net Ch_19_A2: J10.09
- net Out_D7_Cube_2 is gone; now on net Ch_10_A2: J12.09
- net Out_D7_Cube_5 is gone; now on net Ch_10_A4: J15.09
- net Out_D7_Cube_6 is gone; now on net Ch_19_A4: J16.09
- net Out_D8_Cube_1 is gone; now on net Ch_31_A2: J10.06
- net Out_D8_Cube_2 is gone; now on net Ch_64_A2: J12.06
- net Out_D8_Cube_5 is gone; now on net Ch_32_A4: J15.06
- net Out_D8_Cube_6 is gone; now on net Ch_39_A4: J16.06
- net Out_E1_Cube_5 is gone; now on net Ch_64_A3: J13.38
- net Out_E1_Cube_6 is gone; now on net Ch_55_A3: J14.38
- net Out_E2_Cube_5 is gone; now on net Ch_48_A3: J13.50
- net Out_E2_Cube_6 is gone; now on net Ch_53_A3: J14.50
- net Out_E3_Cube_5 is gone; now on net Ch_54_A3: J13.46
- net Out_E3_Cube_6 is gone; now on net Ch_47_A3: J14.46
- net Out_E4_Cube_5 is gone; now on net Ch_34_A3: J13.37
- net Out_E4_Cube_6 is gone; now on net Ch_23_A3: J14.37
- net Out_E5_Cube_5 is gone; now on net Ch_50_A3: J13.22
- net Out_E5_Cube_6 is gone; now on net Ch_59_A3: J14.22
- net Out_E6_Cube_5 is gone; now on net Ch_62_A3: J13.34
- net Out_E6_Cube_6 is gone; now on net Ch_49_A3: J14.34
- net Out_E7_Cube_5 is gone; now on net Ch_38_A3: J13.02
- net Out_E7_Cube_6 is gone; now on net Ch_31_A3: J14.02
- net Out_E8_Cube_5 is gone; now on net Ch_04_A3: J13.01
- net Out_E8_Cube_6 is gone; now on net Ch_05_A3: J14.01
- net Out_F1_Cube_5 is gone; now on net Ch_40_A3: J13.58
- net Out_F1_Cube_6 is gone; now on net Ch_43_A3: J14.58
- net Out_F2_Cube_5 is gone; now on net Ch_36_A3: J13.60
- net Out_F2_Cube_6 is gone; now on net Ch_27_A3: J14.60
- net Out_F3_Cube_5 is gone; now on net Ch_30_A3: J13.33
- net Out_F3_Cube_6 is gone; now on net Ch_17_A3: J14.33
- net Out_F4_Cube_5 is gone; now on net Ch_60_A3: J13.42
- net Out_F4_Cube_6 is gone; now on net Ch_57_A3: J14.42
- net Out_F5_Cube_5 is gone; now on net Ch_52_A3: J13.18
- net Out_F5_Cube_6 is gone; now on net Ch_45_A3: J14.18
- net Out_F6_Cube_5 is gone; now on net Ch_42_A3: J13.14
- net Out_F6_Cube_6 is gone; now on net Ch_41_A3: J14.14
- net Out_F7_Cube_5 is gone; now on net Ch_46_A3: J13.10
- net Out_F7_Cube_6 is gone; now on net Ch_39_A3: J14.10
- net Out_F8_Cube_5 is gone; now on net Ch_18_A3: J13.17
- net Out_F8_Cube_6 is gone; now on net Ch_25_A3: J14.17
- net Out_G1_Cube_5 is gone; now on net Ch_44_A3: J13.54
- net Out_G1_Cube_6 is gone; now on net Ch_37_A3: J14.54
- net Out_G2_Cube_5 is gone; now on net Ch_22_A3: J13.29
- net Out_G2_Cube_6 is gone; now on net Ch_33_A3: J14.29
- net Out_G3_Cube_5 is gone; now on net Ch_14_A3: J13.57
- net Out_G3_Cube_6 is gone; now on net Ch_01_A3: J14.57
- net Out_G4_Cube_5 is gone; now on net Ch_24_A3: J13.45
- net Out_G4_Cube_6 is gone; now on net Ch_15_A3: J14.45
- net Out_G5_Cube_5 is gone; now on net Ch_58_A3: J13.26
- net Out_G5_Cube_6 is gone; now on net Ch_61_A3: J14.26
- net Out_G6_Cube_5 is gone; now on net Ch_56_A3: J13.30
- net Out_G6_Cube_6 is gone; now on net Ch_51_A3: J14.30
- net Out_G7_Cube_5 is gone; now on net Ch_06_A3: J13.13
- net Out_G7_Cube_6 is gone; now on net Ch_21_A3: J14.13
- net Out_G8_Cube_5 is gone; now on net Ch_10_A3: J13.09
- net Out_G8_Cube_6 is gone; now on net Ch_19_A3: J14.09
- net Out_H1_Cube_5 is gone; now on net Ch_20_A3: J13.49
- net Out_H1_Cube_6 is gone; now on net Ch_07_A3: J14.49
- net Out_H2_Cube_5 is gone; now on net Ch_16_A3: J13.53
- net Out_H2_Cube_6 is gone; now on net Ch_09_A3: J14.53
- net Out_H3_Cube_5 is gone; now on net Ch_26_A3: J13.41
- net Out_H3_Cube_6 is gone; now on net Ch_11_A3: J14.41
- net Out_H4_Cube_5 is gone; now on net Ch_08_A3: J13.59
- net Out_H4_Cube_6 is gone; now on net Ch_03_A3: J14.59
- net Out_H5_Cube_5 is gone; now on net Ch_12_A3: J13.21
- net Out_H5_Cube_6 is gone; now on net Ch_29_A3: J14.21
- net Out_H6_Cube_1 is gone; now on net Ch_59_A2: J10.22
- net Out_H6_Cube_2 is gone; now on net Ch_52_A2: J12.22
- net Out_H6_Cube_5 is gone; now on net Ch_50_A4: J15.22
- net Out_H6_Cube_6 is gone; now on net Ch_51_A4: J16.22
- net Out_H7_Cube_5 is gone; now on net Ch_02_A3: J13.05
- net Out_H7_Cube_6 is gone; now on net Ch_13_A3: J14.05
- net Out_H8_Cube_5 is gone; now on net Ch_32_A3: J13.06
- net Out_H8_Cube_6 is gone; now on net Ch_35_A3: J14.06
- net 1V1_A1: now also J3.05, J3.07, J3.09, J3.11; no longer J2.50, J2.52, J2.54, J2.56
- net 1V1_A3: now also J7.05, J7.07, J7.09, J7.11, TP14.1; no longer J6.50, J6.52, J6.54, J6.56
- net GND: no longer H1.1, H10.1, H11.1, H12.1, H13.1, H14.1, H15.1, H16.1, H2.1, H3.1, H4.1, H5.1, H6.1, H7.1, H8.1, H9.1
- removed net 1V1_A2: J3.05, J3.07, J3.09, J3.11, J4.50, J4.52, J4.54, J4.56
- removed net 1V1_A4: J7.05, J7.07, J7.09, J7.11, J8.50, J8.52, J8.54, J8.56
- net 4->5V renamed 4-5V
- no-connect marks 36 -> 52
Other:
- title: Fiber - Main Board -> Fibers Main Board

Commit message: .
Parts:
- removed J23: Amphenol_132289, Connector_Coaxial:SMA_Amphenol_132289_EdgeMount, symbol Connector:Conn_Coaxial_Small
- added J24: 92_SMA-50-0-10/111_NE, 0-lib:HUBER_SUHNER_92_SMA-50-0-10_111_NE, symbol Connector:Conn_Coaxial_Small
Connections:
- net GND: now also J24.2 (Ext)
- net HV_In: now also J24.1 (In)
Other:
- note added: "BACK VIEW"
- note added: "Connectors"
- note added: "TOP VIEW"
- moved on the sheet: C1, C10, C11, C12, C13, C14, C15, C16, C17, C18, C19, C2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
