File: Main_Board/Main_Board_REV_0/_autosave-Main_Board_REV_0.kicad_sch (KiCad schematic)
At the start: 74 parts, among them J1 ERF6-30-03.5-L-DV-A-K-TR, J10 ERF6-30-03.5-L-DV-A-K-TR, J11 ERF6-30-03.5-L-DV-A-K-TR, J12 ERF6-30-03.5-L-DV-A-K-TR, J13 ERF6-30-03.5-L-DV-A-K-TR, J14 ERF6-30-03.5-L-DV-A-K-TR, J15 ERF6-30-03.5-L-DV-A-K-TR, J16 ERF6-30-03.5-L-DV-A-K-TR, J17 1778764, J18 NCP1117LPST33T3G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

Commit message: .
Other:
- note added: "BACK VIEW"
- note added: "Connectors"
- note added: "TOP VIEW"
- moved on the sheet: C1, C10, C11, C12, C13, C14, C15, C16, C17, C18, C19, C2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
