File: HV_MPPC_Ballance/Prototype/STM32_RS485_I2C/1_ch_ltc6090.kicad_sch (KiCad schematic)
At the start: 9 parts, among them U4 LTC6090CS8E-5-PBF

Commit message: .
Other:
- title: (none) -> HV Control
Changed lines of the file:
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@@
 	(generator_version "9.0")
 	(paper "A4")
+	(title_block
+		(title "HV Control")
+	)
 	(text "!in case of unstability populate this capacitor"
 		(exclude_from_sim no)
