File: HV_MPPC_Ballance/Prototype/STM32_RS485_I2C/STM32_RS485_I2C.kicad_sch (KiCad schematic)
At the start: 0 parts

Commit message: .
Other:
- added sheet Untitled Sheet (1_ch_ltc6090.kicad_sch)
Changed lines of the file:
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@@
 	(paper "A4")
+	(sheet
+		(at 165.1 50.8)
+		(size 41.91 22.86)
+		(exclude_from_sim no)
+		(in_bom yes)
+		(on_board yes)
+		(dnp no)
+		(fields_autoplaced yes)
+		(stroke
+			(width 0.1524)
+			(type solid)
+		)
+		(fill
+			(color 0 0 0 0.0000)
+		)
+		(property "Sheetname" "Untitled Sheet"
+			(at 165.1 50.0884 0)
+			(effects
+				(font
+					(size 1.27 1.27)
+				)
+				(justify left bottom)
+			)
+		)
+		(property "Sheetfile" "1_ch_ltc6090.kicad_sch"
+			(at 165.1 74.2446 0)
+			(effects
+				(font
+					(size 1.27 1.27)
+				)
+				(justify left top)
+			)
+		)
+		(instances
+			(project "STM32_RS485_I2C"
+				(path "/b57b15c3-de3f-4cb9-ac5a-185df551189c"
+					(page "3")
+				)
+			)
+		)
+	)
 	(sheet
 		(at 66.04 36.83)

Commit message: .
Other:
- sheet Untitled Sheet renamed HV Control
Changed lines of the file:
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@@
 	(paper "A4")
 	(sheet
-		(at 165.1 50.8)
-		(size 41.91 22.86)
+		(at 105.41 25.4)
+		(size 24.13 6.35)
 		(exclude_from_sim no)
 		(in_bom yes)
 		(on_board yes)
 		(dnp no)
-		(fields_autoplaced yes)
 		(stroke
 			(width 0.1524)
@@
 			(color 0 0 0 0.0000)
 		)
-		(property "Sheetname" "Untitled Sheet"
-			(at 165.1 50.0884 0)
+		(property "Sheetname" "HV Control"
+			(at 106.68 29.972 0)
 			(effects
 				(font
-					(size 1.27 1.27)
+					(size 2.54 2.54)
+					(thickness 0.254)
+					(bold yes)
 				)
 				(justify left bottom)
@@
 		)
 		(property "Sheetfile" "1_ch_ltc6090.kicad_sch"
-			(at 165.1 74.2446 0)
+			(at 105.41 48.8446 0)
 			(effects
 				(font
@@
 				)
 				(justify left top)
+				(hide yes)
 			)
 		)
@@
 	)
 	(sheet
-		(at 66.04 36.83)
-		(size 50.8 82.55)
+		(at 17.78 36.83)
+		(size 35.56 11.43)
 		(exclude_from_sim no)
 		(in_bom yes)
@@
 		)
 		(property "Sheetname" "Microcontroller"
-			(at 76.2 80.264 0)
+			(at 20.32 44.196 0)
 			(effects
 				(font
@@
 		)
 		(property "Sheetfile" "STM32L476RET6.kicad_sch"
-			(at 66.04 119.9646 0)
+			(at 17.78 119.9646 0)
 			(effects
 				(font

Commit message: .
Other:
- company: (none) -> TU Darmstadt
- title: (none) -> STM32 HV Control via RS485

Commit message: .
Changed lines of the file:
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@@
 	(sheet
 		(at 17.78 36.83)
-		(size 35.56 11.43)
+		(size 35.56 24.13)
 		(exclude_from_sim no)
 		(in_bom yes)
@@
 		)
 		(property "Sheetname" "Microcontroller"
-			(at 20.32 44.196 0)
+			(at 20.32 50.038 0)
 			(effects
 				(font

Commit message: .
Other:
- added sheet Power (Power.kicad_sch)
- added sheet RS485 (rs485.kicad_sch)
- sheet HV Control ports: added DAC, HV_in, Out; removed none
- sheet Microcontroller ports: added RX, RX_Enable, SCL, SDA, TX, TX_Enable; removed none
Changed lines of the file:
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@@
 	)
 	(sheet
-		(at 100.33 38.1)
-		(size 24.13 6.35)
+		(at 134.62 38.1)
+		(size 34.29 6.35)
 		(exclude_from_sim no)
 		(in_bom yes)
@@
 		)
 		(property "Sheetname" "HV Control"
-			(at 101.6 42.672 0)
+			(at 141.986 43.18 0)
 			(effects
 				(font
@@
 		)
 		(property "Sheetfile" "1_ch_ltc6090.kicad_sch"
-			(at 100.33 61.5446 0)
-			(effects
-				(font
-					(size 1.27 1.27)
-				)
-				(justify left top)
-				(hide yes)
+			(at 134.62 61.5446 0)
+			(effects
+				(font
+					(size 1.27 1.27)
+				)
+				(justify left top)
+				(hide yes)
+			)
+		)
+		(pin "DAC" input
+			(at 134.62 43.18 180)
+			(effects
+				(font
+					(size 1.27 1.27)
+				)
+				(justify left)
+			)
+		)
+		(pin "HV_in" input
+			(at 134.62 39.37 180)
+			(effects
+				(font
+					(size 1.27 1.27)
+				)
+				(justify left)
+			)
+		)
+		(pin "Out" output
+			(at 168.91 41.91 0)
+			(effects
+				(font
+					(size 1.27 1.27)
+				)
+				(justify right)
 			)
 		)
@@
 	)
 	(sheet
-		(at 17.78 36.83)
-		(size 35.56 24.13)
+		(at 24.13 34.29)
+		(size 45.72 16.51)
 		(exclude_from_sim no)
 		(in_bom yes)
@@
 		)
 		(property "Sheetname" "Microcontroller"
-			(at 20.32 50.038 0)
+			(at 25.908 44.958 0)
 			(effects
 				(font
@@
 		)
 		(property "Sheetfile" "STM32L476RET6.kicad_sch"
-			(at 17.78 119.9646 0)
-			(effects
-				(font
-					(size 1.27 1.27)
-				)
-				(justify left top)
-				(hide yes)
+			(at 24.13 117.4246 0)
+			(effects
+				(font
+					(size 1.27 1.27)
+				)
+				(justify left top)
+				(hide yes)
+			)
+		)
+		(pin "RX" input
+			(at 69.85 46.99 0)
+			(effects
+				(font
+					(size 1.27 1.27)
+				)
+				(justify right)
+			)
+		)
+		(pin "RX_Enable" output
+			(at 69.85 49.53 0)
+			(effects
+				(font
+					(size 1.27 1.27)
+				)
+				(justify right)
+			)
+		)
+		(pin "SCL" output
+			(at 69.85 35.56 0)
+			(effects
+				(font
+					(size 1.27 1.27)
+				)
+				(justify right)
+			)
+		)
+		(pin "SDA" bidirectional
+			(at 69.85 38.1 0)
+			(effects
+				(font
+					(size 1.27 1.27)
+				)
+				(justify right)
+			)
+		)
+		(pin "TX" output
+			(at 69.85 41.91 0)
+			(effects
+				(font
+					(size 1.27 1.27)
+				)
+				(justify right)
+			)
+		)
+		(pin "TX_Enable" output
+			(at 69.85 44.45 0)
+			(effects
+				(font
+					(size 1.27 1.27)
+				)
+				(justify right)
 			)
 		)
@@
 				)
 			)
+		)
+	)
+	(sheet
+		(at 24.13 76.2)
+		(size 41.91 27.94)
+		(exclude_from_sim no)
+		(in_bom yes)
+		(on_board yes)
+		(dnp no)
+		(fields_autoplaced yes)
+		(stroke
+			(width 0.1524)
+			(type solid)
+		)
+		(fill
+			(color 0 0 0 0.0000)
+		)
+		(property "Sheetname" "Power"
+			(at 24.13 75.4884 0)
+			(effects
+				(font
+					(size 1.27 1.27)
+				)
+				(justify left bottom)
+			)
+		)
+		(property "Sheetfile" "Power.kicad_sch"
+			(at 24.13 104.7246 0)
+			(effects
+				(font
+					(size 1.27 1.27)
+				)
+				(justify left top)
+				(hide yes)
+			)
+		)
+		(instances
+			(project "STM32_RS485_I2C"
+				(path "/b57b15c3-de3f-4cb9-ac5a-185df551189c"
+					(page "4")
+				)
+			)
+		)
+	)
+	(sheet
+		(at 100.33 76.2)
+		(size 64.77 33.02)
+		(exclude_from_sim no)
+		(in_bom yes)
+		(on_board yes)
+		(dnp no)
+		(fields_autoplaced yes)
+		(stroke
+			(width 0.1524)
+			(type solid)
+		)
+		(fill
+			(color 0 0 0 0.0000)
+		)
+		(property "Sheetname" "RS485"
+			(at 100.33 75.4884 0)
+			(effects
+				(font
+					(size 1.27 1.27)
+				)
+				(justify left bottom)
+			)
+		)
+		(property "Sheetfile" "rs485.kicad_sch"
+			(at 100.33 109.8046 0)
+			(effects
+				(font
+					(size 1.27 1.27)
+				)
+				(justify left top)
+				(hide yes)
+			)
+		)
+		(instances
+			(project "STM32_RS485_I2C"
+				(path "/b57b15c3-de3f-4cb9-ac5a-185df551189c"
+					(page "5")
+				)
+			)
