File: HV_MPPC_Ballance/Prototype/STM32_RS485_I2C/Power.kicad_sch (KiCad schematic)
At the start: 24 parts, among them J2 430450200, U1 TPS7A2033PDBVR, U3 ADP5600ACPZ-R7, U5 TPS7A2033PDBVR, U6 TPS7A2033PDBVR

Commit message: .
Parts:
- removed J2: 430450200, 0_lib:0430450200, symbol 0-lib:430450200
- added J19: Conn_02x16_Odd_Even, Connector_PinSocket_2.54mm:PinSocket_2x16_P2.54mm_Vertical, symbol Connector_Generic:Conn_02x16_Odd_Even
Changed lines of the file:
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@@
 	(wire
 		(pts
-			(xy 147.32 34.29) (xy 147.32 35.56)
-		)
-		(stroke
-			(width 0)
-			(type default)
-		)
-	)
-	(wire
-		(pts
 			(xy 27.94 53.34) (xy 27.94 54.61)
 		)
@@
 	(wire
 		(pts
-			(xy 147.32 31.75) (xy 148.59 31.75)
-		)
-		(stroke
-			(width 0)
-			(type default)
-		)
-	)
-	(wire
-		(pts
 			(xy 67.31 87.63) (xy 67.31 88.9)
 		)
@@
 	(wire
 		(pts
-			(xy 147.32 30.48) (xy 147.32 31.75)
-		)
-		(stroke
-			(width 0)
-			(type default)
-		)
-	)
-	(wire
-		(pts
 			(xy 22.86 135.89) (xy 22.86 137.16)
 		)
@@
 	(wire
 		(pts
-			(xy 148.59 34.29) (xy 147.32 34.29)
-		)
-		(stroke
-			(width 0)
-			(type default)
-		)
-	)
-	(wire
-		(pts
 			(xy 34.29 144.78) (xy 36.83 144.78)
 		)
@@
 	)
 	(symbol
+		(lib_id "Connector_Generic:Conn_02x16_Odd_Even")
+		(at 160.02 54.61 0)
+		(mirror y)
+		(unit 1)
+		(exclude_from_sim no)
+		(in_bom yes)
+		(on_board yes)
+		(dnp no)
+		(property "Reference" "J19"
+			(at 158.75 30.48 0)
+			(effects
+				(font
+					(size 1.27 1.27)
+				)
+			)
+		)
+		(property "Value" "Conn_02x16_Odd_Even"
+			(at 158.75 33.02 0)
+			(effects
+				(font
+					(size 1.27 1.27)
+				)
+			)
+		)
+		(property "Footprint" "Connector_PinSocket_2.54mm:PinSocket_2x16_P2.54mm_Vertical"
+			(at 160.02 54.61 0)
+			(effects
+				(font
+					(size 1.27 1.27)
+				)
+				(hide yes)
+			)
+		)
+		(property "Datasheet" "~"
+			(at 160.02 54.61 0)
+			(effects
+				(font
+					(size 1.27 1.27)
+				)
+				(hide yes)
+			)
+		)
+		(property "Description" "Generic connector, double row, 02x16, odd/even pin numbering scheme (row 1 odd numbers, row 2 even numbers), script generated (kicad-library-utils/schlib/autogen/connector/)"
+			(at 160.02 54.61 0)
+			(effects
+				(font
+					(size 1.27 1.27)
+				)
+				(hide yes)
+			)
+		)
+		(pin "28"
+		)
+		(pin "24"
+		)
+		(pin "22"
+		)
+		(pin "26"
+		)
+		(pin "30"
+		)
+		(pin "32"
+		)
+		(pin "27"
+		)
+		(pin "19"
+		)
+		(pin "21"
+		)
+		(pin "25"
+		)
+		(pin "5"
+		)
+		(pin "9"
+		)
+		(pin "23"
+		)
+		(pin "7"
+		)
+		(pin "11"
+		)
+		(pin "29"
+		)
+		(pin "15"
+		)
+		(pin "1"
+		)
+		(pin "13"
+		)
+		(pin "17"
+		)
+		(pin "3"
+		)
+		(pin "31"
+		)
+		(pin "10"
+		)
+		(pin "8"
+		)
+		(pin "12"
+		)
+		(pin "6"
+		)
+		(pin "4"
+		)
+		(pin "14"
+		)
+		(pin "2"
+		)
+		(pin "18"
+		)
+		(pin "20"
+		)
+		(pin "16"
+		)
+		(instances
+			(project "STM32_RS485_I2C"
+				(path "/b57b15c3-de3f-4cb9-ac5a-185df551189c/32f012e1-7e21-437e-ab00-df9acbe51353"
+					(reference "J19")
+					(unit 1)
+				)
+			)
+		)
+	)
+	(symbol
 		(lib_id "Connector:TestPoint")
 		(at 77.47 77.47 0)
@@
 	)
 	(symbol
-		(lib_id "0-lib:430450200")
-		(at 148.59 31.75 0)
-		(unit 1)
-		(exclude_from_sim no)
-		(in_bom yes)
-		(on_board yes)
-		(dnp no)
-		(fields_autoplaced yes)
-		(property "Reference" "J2"
-			(at 162.56 31.7499 0)
-			(effects
-				(font
-					(size 1.524 1.524)
-				)
-				(justify left)
-			)
-		)
-		(property "Value" "430450200"
-			(at 162.56 34.2899 0)
-			(effects
-				(font
-					(size 1.524 1.524)
-				)
-				(justify left)
-			)
-		)
-		(property "Footprint" "0_lib:0430450200"
-			(at 148.59 31.75 0)
-			(effects
-				(font
-					(size 1.27 1.27)
-					(italic yes)
-				)
-				(hide yes)
-			)
-		)
-		(property "Datasheet" "https://www.molex.com/en-us/products/part-detail-pdf/430450200?display=pdf"
-			(at 148.59 31.75 0)
-			(effects
-				(font
-					(size 1.27 1.27)
-					(italic yes)
-				)
-				(hide yes)
-			)
-		)
-		(property "Description" ""
-			(at 148.59 31.75 0)
-			(effects
-				(font
-					(size 1.27 1.27)
-				)
-				(hide yes)
-			)
-		)
-		(pin "2"
-		)
-		(pin "1"
-		)
-		(instances
-			(project ""
-				(path "/b57b15c3-de3f-4cb9-ac5a-185df551189c/32f012e1-7e21-437e-ab00-df9acbe51353"
-					(reference "J2")
-					(unit 1)
-				)
-			)
-		)
-	)
-	(symbol
 		(lib_id "0-lib:ADP5600ACPZ-R7")
 		(at 36.83 124.46 0)
@@
 	)
 	(symbol
-		(lib_id "power:GND")
-		(at 147.32 35.56 0)
-		(unit 1)
-		(exclude_from_sim no)
-		(in_bom yes)
-		(on_board yes)
-		(dnp no)
-		(fields_autoplaced yes)
-		(property "Reference" "#PWR037"
-			(at 147.32 41.91 0)
-			(effects
-				(font
-					(size 1.27 1.27)
-				)
-				(hide yes)
-			)
-		)
-		(property "Value" "GND"
-			(at 147.32 40.64 0)
-			(effects
-				(font
-					(size 1.27 1.27)
-				)
-				(hide yes)
-			)
-		)
-		(property "Footprint" ""
-			(at 147.32 35.56 0)
-			(effects
-				(font
-					(size 1.27 1.27)
-				)
-				(hide yes)
-			)
-		)
-		(property "Datasheet" ""
-			(at 147.32 35.56 0)
-			(effects
-				(font
-					(size 1.27 1.27)
-				)
-				(hide yes)
-			)
-		)
-		(property "Description" "Power symbol creates a global label with name \"GND\" , ground"
-			(at 147.32 35.56 0)
-			(effects
-				(font
-					(size 1.27 1.27)
-				)
-				(hide yes)
-			)
-		)
-		(pin "1"
-		)
-		(instances
-			(project "STM32_RS485_I2C"
-				(path "/b57b15c3-de3f-4cb9-ac5a-185df551189c/32f012e1-7e21-437e-ab00-df9acbe51353"
-					(reference "#PWR037")
-					(unit 1)
-				)
-			)
-		)
-	)
-	(symbol
 		(lib_id "power:+5V")
 		(at 22.86 127 0)
@@
 					(unit 1)
 				)
-			)
-		)
-	)
-	(symbol
-		(lib_id "power:+5V")
-		(at 147.32 30.48 0)
-		(unit 1)
-		(exclude_from_sim no)
-		(in_bom yes)
-		(on_board yes)
-		(dnp no)
-		(fields_autoplaced yes)
-		(property "Reference" "#PWR029"
-			(at 147.32 34.29 0)
-			(effects
-				(font
-					(size 1.27 1.27)
-				)
-				(hide yes)
-			)
-		)
-		(property "Value" "+5V"
-			(at 147.32 25.4 0)
-			(effects
-				(font
-					(size 1.27 1.27)
-				)
-			)
-		)
-		(property "Footprint" ""
-			(at 147.32 30.48 0)
-			(effects
-				(font
-					(size 1.27 1.27)
-				)
-				(hide yes)
-			)
-		)
-		(property "Datasheet" ""
-			(at 147.32 30.48 0)
-			(effects
-				(font
-					(size 1.27 1.27)
-				)
-				(hide yes)
-			)
-		)
-		(property "Description" "Power symbol creates a global label with name \"+5V\""
-			(at 147.32 30.48 0)
-			(effects
-				(font
-					(size 1.27 1.27)
-				)
-				(hide yes)
-			)
-		)
-		(pin "1"
-		)
-		(instances
-			(project "STM32_RS485_I2C"
-				(path "/b57b15c3-de3f-4cb9-ac5a-185df551189c/32f012e1-7e21-437e-ab00-df9acbe51353"
-					(reference "#PWR029")
-					(unit 1)
-				)
